File: hw/power_input.kicad_sch (KiCad schematic)
At the start: 0 parts

Commit message: Draw the power_input sheet, and a generator for the nine after it
hw/schlib.py is the reusable piece: a minimal KiCad 7 schematic writer
that places symbols, wires them, labels nets and exposes hierarchical
pins. Symbol definitions are copied out of the installed libraries into
each sheet's own (lib_symbols) block, which is what KiCad expects.

Generated rather than hand-drawn because almost no component value on
these sheets is a free choice -- nearly every one traces to a check in
sim/blocks/ or a tag in docs/bom_requirements.md. A hand-drawn sheet
holds those as text nobody re-derives, and they drift the moment a
simulation moves, which has already happened three times with the
reverse-battery FET's voltage class alone. Each part now carries its
source in a hidden field, so the value and the reason for it travel
together. Eeschema can still edit these freely; the generator refuses to
overwrite a sheet that has content.

power_input is the first sheet. Stage order is spec sec.4 -- EMI filter,
fuse, TVS, reverse-battery FET, negative clamp -- and the EMI filter is
emi_filter.cir element for element: 22 uH, 4.7 uF, 0.5 uH damped by
120 R, 100 nF, and the 1 uF/2R2 damping leg.

Two gates are deliberately left on named nets with nothing driving them.
VBAT_REV_GATE wants the ideal-diode controller whose turn-off time is
load-bearing and unsourced; NCLAMP_GATE wants the comparator whose
propagation delay is the last unmodelled term in negative_pulses.cir.
Neither pinout can be drawn without choosing a part. ERC will report
both, correctly -- that is the sheet reporting an open decision, and the
note on the page says so to whoever opens it next.

Three bugs found by checking the exported netlist rather than the plot,
which is the point of checking the netlist:

The rotation helper had 90 and 270 the other way round. Nothing
complained -- parts looked placed, wires met their endpoints, the page
plotted fine -- and the only symptom was the negative clamp Schottky
coming ou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
Parts:
- added C1: 4.7uF, symbol Device:C
- added C2: 100nF, symbol Device:C
- added C3: 1uF, symbol Device:C
- added D1: SMCJ43CA, symbol Device:D_TVS
- added D2: 60V 20A, symbol Device:D_Schottky
- added F1: 20A, symbol Device:Fuse
- added L1: 22uH, symbol Device:L
- added L2: 0.5uH, symbol Device:L
- added Q1: 100V N-ch, symbol Device:Q_NMOS_GSD
- added Q2: 40V 5mOhm N-ch, symbol Device:Q_NMOS_GSD
- added R1: 120R, symbol Device:R
- added R2: 2R2, symbol Device:R
Connections:
- new net: C3.2, R2.1
- new net: C1.1, L1.2, L2.1, R1.1
- new net: F1.2, L1.1
- new net GND: C1.2, C2.2, D1.1 (A1), D2.2 (A), Q2.2 (S), R2.2
- new net NCLAMP_GATE: Q2.1 (G)
- new net VBAT_CLAMPED: C2.1, C3.1, D1.2 (A2), L2.2, Q1.2 (S), R1.2
- new net VBAT_IN: F1.1
- new net VBAT_PROT: D2.1 (K), Q1.3 (D), Q2.3 (D)
- new net VBAT_REV_GATE: Q1.1 (G)
Other:
- note added: "OPEN -- two gates on this sheet are intentionally undriven, and ERC will report them: VBAT_REV_GATE ideal-diode controller for Q1. No part chosen. Its turn-off time is load-bearing (reverse_battery.cir models it with none) but nothing sources that number yet. NCLAMP_GATE comparator for Q2, sensing VIN against -0.1 V. No part chosen. Its propagation delay is the last unmodelled term in negative_pu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"
- note added: "Stage order is spec sec.4: EMI filter -> fuse -> TVS -> reverse-battery FET -> buck VIN. EMI filter values are emi_filter.cir element for element. Every part carries its source in a hidden Source field."

Commit message: Draw the mcu sheet, and choose the supervisor part
The S32K148 with all 144 pins wired, the TPS3850G33 watching its rail,
the inverting stage that turns the supervisor's active-low RESET into an
active-high GATE_KILL for the driver sheets, mcu_pdn.cir's decoupling
network, and the debug header. A2 rather than A3: six 25-pin units plus
a supervisor, a header and eleven decoupling parts do not fit A3 without
stacking, and a schematic whose parts overlap is one nobody reads.

THE SUPERVISOR IS NOW A PART, NOT A CLASS. Memo 11 had TPS3850 CONFIRMED
on its electricals but recommended it as "TPS3850-class", and the pinout
was never captured. Both are settled here from the retrieved datasheet
(TI SBVS301B, Table 5-1 and Figure 5-1), and the variant is chosen
rather than assumed. The nomenclature table gives G = thresholds at +/-4%
of nominal and H = +/-7%; with the part's own +/-0.8% accuracy that puts
the worst-case undervoltage trip at 3.143 V for G33 against 3.044 V for
H33. The supervisor exists to assert BEFORE the S32K148's own LVD, whose
maximum is 3.0 V, so G33 clears it by 143 mV and H33 by 44 mV -- close
enough that the two could fire in either order, and a supervisor that
might lose the race to the thing it supervises is not doing its job. The
cost is a tighter window the rail must live inside, 3.143-3.459 V, which
is now a constraint on the rails sheet.

THE PIN MAP HAD A GAP, and this sheet is what found it. Section 1.8 said
outright that "the only MCU pin in this interface is RESET_b". True of
the kill path, which deliberately involves no MCU pin -- and wrong about
the watchdog, which is not a passive monitor. The MCU has to present a
falling edge on WDI inside every window or the part resets the board on
a timer. A supervisor topology with no pin to kick it guarantees a reset
loop. PTE0 (WDT_KICK) and PTE1 (WDT_FAULT) are added, both free GPIO-HD,
both PE=0/PS=0 at reset, taking the map from 37 committed signals to 39.
WDO is worth its own pin because it ass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
Other:
- note added: "OPEN -- two gates on this sheet are intentionally undriven, and ERC will report them:\n VBAT_REV_GATE ideal-diode controller for Q1. No part chosen. Its turn-off time is load-bearing\n (reverse_battery.cir models it with none) but nothing sources that number yet.\n NCLAMP_GATE comparator for Q2, sensing VIN against -0.1 V. No part chosen. Its propagation\n delay is the last unmodelled term in neg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"
- note added: "Stage order is spec sec.4: EMI filter -> fuse -> TVS -> reverse-battery FET -> buck VIN.\nEMI filter values are emi_filter.cir element for element. Every part carries its source in a hidden Source field."
- note removed: "OPEN -- two gates on this sheet are intentionally undriven, and ERC will report them: VBAT_REV_GATE ideal-diode controller for Q1. No part chosen. Its turn-off time is load-bearing (reverse_battery.cir models it with none) but nothing sources that number yet. NCLAMP_GATE comparator for Q2, sensing VIN against -0.1 V. No part chosen. Its propagation delay is the last unmodelled term in negative_pu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"
- note removed: "Stage order is spec sec.4: EMI filter -> fuse -> TVS -> reverse-battery FET -> buck VIN. EMI filter values are emi_filter.cir element for element. Every part carries its source in a hidden Source field."
Changed lines of the file:
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@@
     (effects (font (size 1.27 1.27)) (justify left bottom))
   )
-  (text "OPEN -- two gates on this sheet are intentionally undriven, and ERC will report them:\n  VBAT_REV_GATE   ideal-diode controller for Q1. No part chosen. Its turn-off time is load-bearing\n                  (reverse_battery.cir models it with none) but nothing sources that number yet.\n  NCLAMP_GATE     comparator for Q2, sensing VIN against -0.1 V. No part chosen. Its propagation\n                  delay is the last unmodelled term in negative_pulses.cir -- VIN sits at the\n                  Schottky's -0.53 V for exactly that long before the clamp engages.\nNeither pinout can be drawn without choosing a part, and this project does not guess parts into copper." (at 30 150 0)
+  (text "OPEN -- two gates on this sheet are intentionally undriven, and ERC will report them:\\n  VBAT_REV_GATE   ideal-diode controller for Q1. No part chosen. Its turn-off time is load-bearing\\n                  (reverse_battery.cir models it with none) but nothing sources that number yet.\\n  NCLAMP_GATE     comparator for Q2, sensing VIN against -0.1 V. No part chosen. Its propagation\\n                  delay is the last unmodelled term in negative_pulses.cir -- VIN sits at the\\n                  Schottky's -0.53 V for exactly that long before the clamp engages.\\nNeither pinout can be drawn without choosing a part, and this project does not guess parts into copper." (at 30 150 0)
     (effects (font (size 1.6 1.6)) (justify left))
   )
-  (text "Stage order is spec sec.4: EMI filter -> fuse -> TVS -> reverse-battery FET -> buck VIN.\nEMI filter values are emi_filter.cir element for element. Every part carries its source in a hidden Source field." (at 30 175 0)
+  (text "Stage order is spec sec.4: EMI filter -> fuse -> TVS -> reverse-battery FET -> buck VIN.\\nEMI filter values are emi_filter.cir element for element. Every part carries its source in a hidden Source field." (at 30 175 0)
     (effects (font (size 1.6 1.6)) (justify left))
   )
