File: hw/rails.kicad_sch (KiCad schematic)
At the start: 0 parts

Commit message: Draw the rails sheet, and settle the buck the suite had already ruled on
LM5164 to 5 V, TLV767-Q1 to 3V3, one PTC per sensor group, and the
ratiometric monitor divider. Values are buck_preregulator.cir's and
sensor_rail.cir's; the configuration values around the buck are derived
from the datasheet rather than picked, and are written up in
docs/bom_requirements.md.

THE BUCK WAS A CONTRADICTION THE REPOSITORY WAS ALREADY CARRYING.
Research memo 07 sec.4 selected a 60 V TPS54360B-Q1, reasoning it beat a
42 V part for load-dump margin. That was correct when written. The
input-protection work then raised the TVS standoff to 43 V so the
suppressor stops conducting during a NORMAL clamped dump -- and a higher
standoff clamps higher, putting the ISO 7637-2 pulse 2a clamp at 73.3 V.
transient_clamp.cir has carried a PASSING check reading "60 V-class
parts are NO LONGER viable downstream" ever since.

So the BOM named a part that fails the first pulse 2a event, while every
rating check in the suite was written against the LM5164's own -0.3 V /
100 V VIN limits. Both statements sat in the repository for days. Only
the executable one knew, because nothing compares a netlist check against
a prose table, and it surfaced only when someone had to draw the buck and
needed a pinout. Memo 07's rows are now struck through in place with the
reasoning, rather than quietly edited.

RON deserves a line of its own. The datasheet's tON table is linear in
RON/VIN, and solving it for 400 kHz at 5 V out gives 31.4 k at BOTH 13.5 V
and 40 V -- the VIN feedforward is what holds the frequency fixed. That
independently reproduces buck_preregulator.cir's own gate timings, 925 ns
and 312.5 ns. The netlist got them from D = Vout/Vin; the datasheet gets
them from RON; they agree.

The 3V3 LDO was listed as representative with "class pricing, not
fetched". Choosing the supervisor made its accuracy load-bearing --
outside 3.143-3.459 V the board resets itself -- so TLV767-Q1 replaces
it at 1% over load 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
Parts:
- added C1: 4.7uF/100V, symbol Device:C
- added C2: 2.2nF/50V X7R, symbol Device:C
- added C3: 47uF/10mOhm, symbol Device:C
- added C4: 100nF, symbol Device:C
- added C5: 1uF, symbol Device:C
- added C6: 10uF, symbol Device:C
- added F1, F2, F3: 3.0R 200mA, symbol Device:Polyfuse
- added L1: 33uH, symbol Device:L
- added R1: 75k, symbol Device:R
- added R2: 24.9k, symbol Device:R
- added R3: 31.6k, symbol Device:R
- added R4: 100k, symbol Device:R
- added R5: 38.3k, symbol Device:R
- added R6: 12.1k, symbol Device:R
- added R7: 10k, symbol Device:R
- added R8: 15k, symbol Device:R
- added U1: LM5164, Package_SO:SOIC-8-1EP_3.9x4.9mm_P1.27mm_EP2.29x3mm, symbol ecu25kva:LM5164
- added U2: TLV76733, Package_SON:VSON-8-1EP_3x3mm_P0.65mm_EP1.65x2.4mm, symbol ecu25kva:TLV76733
Connections:
- new net: R1.2, R2.1, U1.3 (EN/UVLO)
- new net: R3.1, U1.4 (RON)
- new net 3V3_MCU: C6.1, U2.1 (OUT), U2.3 (SNS)
- new net 5V_MAIN: C3.1, C4.1, C5.1, F1.1, F2.1, F3.1, L1.2, R4.2, R5.1, R7.1, U2.5 (EN), U2.8 (IN)
- new net 5V_SENSOR_A: F1.2
- new net 5V_SENSOR_B: F2.2
- new net 5V_SENSOR_C: F3.2
- new net BST: C2.1, U1.7 (BST)
- new net FB_5V: R5.2, R6.1, U1.5 (FB)
- new net GND: C1.2, C3.2, C4.2, C5.2, C6.2, R2.2, R3.2, R6.2, R8.2, U1.1 (GND), U2.4 (GND), U2.6 (GND)
- new net PGOOD_5V: R4.1, U1.6 (PGOOD)
- new net SENSOR_5V_MON: R7.2, R8.1
- new net SW: C2.2, L1.1, U1.8 (SW)
- new net VBAT_PROT: C1.1, R1.1, U1.2 (VIN)
Other:
- note added: "PGOOD_5V is brought out and left unassigned. The LM5164 asserts it open-drain; the pin map has no channel for it. Available, not wired to anything -- shown rather than hidden."
- note added: "RATIOMETRIC MONITOR, a limitation worth stating: the divider taps 5V_MAIN, upstream of the PTCs. Each group's own PTC drops about 50 mA x 3.0 ohm = 150 mV, which is 3% of the rail and is NOT captured by a measurement taken before it. Correct for the regulator's drift, not for the protection element's. Moving the tap downstream would fix one group and leave the other two wrong, so the tap stays co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"
- note added: "TWO PARTS CHOSEN HERE, both replacing research memo 07 entries that were marked representative rather than chosen: LM5164 memo 07 sec.4 names a 60 V TPS54360B-Q1. transient_clamp.cir now carries a PASSING check that reads "60 V-class parts are NO LONGER viable downstream" -- raising the TVS standoff to 43 V, so the part stops conducting during a NORMAL clamped dump, put the pulse 2a clamp at 73.3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"
- title: Buck pre-regulator, 3V3 and 5V_SENSOR rails -> Rails: buck, 3V3 LDO, 5V sensor distribution
