File: hw/rails.kicad_sch (KiCad schematic)
At the start: 20 parts, among them U1 LM5164, U2 TLV76733

Commit message: Wire the root sheet: the project has a netlist for the first time
Ten sheets each passed their own netlist and the project had none. The
root sheet's ten sheet symbols carried NO hierarchical pins, so a net
name appearing on two sheets was two nets and nothing compared them --
the cross-sheet audit in the last commit was a name comparison, not a
connectivity check.

Each symbol now carries one pin per net its child exports, read OUT of
the child rather than declared in a second list that could drift: 162
pins across the ten, each with a stub and a label. Two labels with the
same name are one net, which is how 162 pins connect without routing
162 wires across a page nobody could read.

Exporting it found the other half of the same problem immediately.
kicad-cli reported annotation errors: every sheet generator allocated
R1, C1, U1 from its own counter, so ten sheets had ten parts called R1.
schlib.REF_BASE gives each sheet its own hundred -- KiCad's own
sheet-number x 100 convention, applied at generation time instead of by
a hand pass in Eeschema. 196 components, no duplicate reference.

hw/check_netlist.py is the gate, and the counterpart to sim/run_sim.py:
that one guards the component values, this one guards the connectivity.
Same rule -- an exemption is not a pass. Every single-pin net is listed
with its reason, and a net that STOPS being single-pin fails the check
until it is removed from the list. An open item that quietly closes is
as much a drift as one that quietly opens.

  196 components, every reference unique
  113 named nets carrying two or more pins
   18 named nets reaching one pin, each a recorded open item
      GND 134 pins, 3V3_MCU 27, VBAT_PROT 12 -- all spanning the project

The root sheet carries those eighteen on the page itself, grouped by
what they wait on, so a reader does not have to run a script to find
which ends are loose.

Full set plots to docs/pdf/ECU-Schematics.pdf, 11 pages.

Two rendering bugs fixed: sheet pin names and their stu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
Parts:
- removed C1: 4.7uF/100V, symbol Device:C
- removed C2: 2.2nF/50V X7R, symbol Device:C
- removed C3: 47uF/10mOhm, symbol Device:C
- removed C4: 100nF, symbol Device:C
- removed C5: 1uF, symbol Device:C
- removed C6: 10uF, symbol Device:C
- removed F1, F2, F3: 3.0R 200mA, symbol Device:Polyfuse
- removed L1: 33uH, symbol Device:L
- removed R1: 75k, symbol Device:R
- removed R2: 24.9k, symbol Device:R
- removed R3: 31.6k, symbol Device:R
- removed R4: 100k, symbol Device:R
- removed R5: 38.3k, symbol Device:R
- removed R6: 12.1k, symbol Device:R
- removed R7: 10k, symbol Device:R
- removed R8: 15k, symbol Device:R
- removed U1: LM5164, Package_SO:SOIC-8-1EP_3.9x4.9mm_P1.27mm_EP2.29x3mm, symbol ecu25kva:LM5164
- removed U2: TLV76733, Package_SON:VSON-8-1EP_3x3mm_P0.65mm_EP1.65x2.4mm, symbol ecu25kva:TLV76733
- added C201: 4.7uF/100V, symbol Device:C
- added C202: 2.2nF/50V X7R, symbol Device:C
- added C203: 47uF/10mOhm, symbol Device:C
- added C204: 100nF, symbol Device:C
- added C205: 1uF, symbol Device:C
- added C206: 10uF, symbol Device:C
- added F201, F202, F203: 3.0R 200mA, symbol Device:Polyfuse
- added L201: 33uH, symbol Device:L
- added R201: 75k, symbol Device:R
- added R202: 24.9k, symbol Device:R
- added R203: 31.6k, symbol Device:R
- added R204: 100k, symbol Device:R
- added R205: 38.3k, symbol Device:R
- added R206: 12.1k, symbol Device:R
- added R207: 10k, symbol Device:R
- added R208: 15k, symbol Device:R
- added U201: LM5164, Package_SO:SOIC-8-1EP_3.9x4.9mm_P1.27mm_EP2.29x3mm, symbol ecu25kva:LM5164
- added U202: TLV76733, Package_SON:VSON-8-1EP_3x3mm_P0.65mm_EP1.65x2.4mm, symbol ecu25kva:TLV76733
Connections:
- net 3V3_MCU: now also C206.1, U202.1 (OUT), U202.3 (SNS)
- net 5V_MAIN: now also C203.1, C204.1, C205.1, F201.1, F202.1, F203.1, L201.2, R204.2, R205.1, R207.1, U202.5 (EN), U202.8 (IN)
- net 5V_SENSOR_A: now also F201.2
- net 5V_SENSOR_B: now also F202.2
- net 5V_SENSOR_C: now also F203.2
- net BST: now also C202.1, U201.7 (BST)
- net FB_5V: now also R205.2, R206.1, U201.5 (FB)
- net GND: now also C201.2, C203.2, C204.2, C205.2, C206.2, R202.2, R203.2, R206.2, R208.2, U201.1 (GND), U202.4 (GND), U202.6 (GND)
- net PGOOD_5V: now also R204.1, U201.6 (PGOOD)
- net SENSOR_5V_MON: now also R207.2, R208.1
- net SW: now also C202.2, L201.1, U201.8 (SW)
- net VBAT_PROT: now also C201.1, R201.1, U201.2 (VIN)
- new net: R203.1, U201.4 (RON)
- new net: R201.2, R202.1, U201.3 (EN/UVLO)
Changed lines of the file:
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@@
   (symbol (lib_id "ecu25kva:LM5164") (at 150.0 85.0 0) (unit 1)
     (in_bom yes) (on_board yes) (fields_autoplaced)
-    (property "Reference" "U1" (id 0) (at 150.0 79.92 0)
+    (property "Reference" "U201" (id 0) (at 150.0 79.92 0)
       (effects (font (size 1.27 1.27)))
     )
@@
   (symbol (lib_id "power:GND") (at 150.0 102.78 0) (unit 1)
     (in_bom yes) (on_board yes) (fields_autoplaced)
-    (property "Reference" "#PWR1" (id 0) (at 150.0 97.7 0)
+    (property "Reference" "#PWR201" (id 0) (at 150.0 97.7 0)
       (effects (font (size 1.27 1.27)) hide)
     )
@@
   (symbol (lib_id "Device:C") (at 60.0 101.19 0) (unit 1)
     (in_bom yes) (on_board yes) (fields_autoplaced)
-    (property "Reference" "C1" (id 0) (at 60.0 96.11 0)
+    (property "Reference" "C201" (id 0) (at 60.0 96.11 0)
       (effects (font (size 1.27 1.27)))
     )
@@
   (symbol (lib_id "power:GND") (at 60.0 112.62 0) (unit 1)
     (in_bom yes) (on_board yes) (fields_autoplaced)
-    (property "Reference" "#PWR2" (id 0) (at 60.0 107.54 0)
+    (property "Reference" "#PWR202" (id 0) (at 60.0 107.54 0)
       (effects (font (size 1.27 1.27)) hide)
     )
@@
   (symbol (lib_id "Device:R") (at 86.0 97.19 0) (unit 1)
     (in_bom yes) (on_board yes) (fields_autoplaced)
-    (property "Reference" "R1" (id 0) (at 86.0 92.11 0)
+    (property "Reference" "R201" (id 0) (at 86.0 92.11 0)
       (effects (font (size 1.27 1.27)))
     )
@@
   (symbol (lib_id "Device:R") (at 86.0 115.19 0) (unit 1)
     (in_bom yes) (on_board yes) (fields_autoplaced)
-    (property "Reference" "R2" (id 0) (at 86.0 110.11 0)
+    (property "Reference" "R202" (id 0) (at 86.0 110.11 0)
       (effects (font (size 1.27 1.27)))
     )
@@
   (symbol (lib_id "power:GND") (at 86.0 126.62 0) (unit 1)
     (in_bom yes) (on_board yes) (fields_autoplaced)
-    (property "Reference" "#PWR3" (id 0) (at 86.0 121.54 0)
+    (property "Reference" "#PWR203" (id 0) (at 86.0 121.54 0)
       (effects (font (size 1.27 1.27)) hide)
     )
@@
   (symbol (lib_id "Device:R") (at 120.0 112.27 0) (unit 1)
     (in_bom yes) (on_board yes) (fields_autoplaced)
-    (property "Reference" "R3" (id 0) (at 120.0 107.19 0)
+    (property "Reference" "R203" (id 0) (at 120.0 107.19 0)
       (effects (font (size 1.27 1.27)))
     )
@@
   (symbol (lib_id "power:GND") (at 120.0 123.7 0) (unit 1)
     (in_bom yes) (on_board yes) (fields_autoplaced)
-    (property "Reference" "#PWR4" (id 0) (at 120.0 118.62 0)
+    (property "Reference" "#PWR204" (id 0) (at 120.0 118.62 0)
       (effects (font (size 1.27 1.27)) hide)
     )
@@
   (symbol (lib_id "Device:R") (at 180.48 101.27 0) (unit 1)
     (in_bom yes) (on_board yes) (fields_autoplaced)
-    (property "Reference" "R4" (id 0) (at 180.48 96.19 0)
+    (property "Reference" "R204" (id 0) (at 180.48 96.19 0)
       (effects (font (size 1.27 1.27)))
     )
@@
   (symbol (lib_id "Device:C") (at 210.0 56.0 0) (unit 1)
     (in_bom yes) (on_board yes) (fields_autoplaced)
-    (property "Reference" "C2" (id 0) (at 210.0 50.92 0)
+    (property "Reference" "C202" (id 0) (at 210.0 50.92 0)
       (effects (font (size 1.27 1.27)))
     )
@@
   (symbol (lib_id "Device:L") (at 284.0 85.0 90) (unit 1)
     (in_bom yes) (on_board yes) (fields_autoplaced)
-    (property "Reference" "L1" (id 0) (at 284.0 79.92 0)
+    (property "Reference" "L201" (id 0) (at 284.0 79.92 0)
       (effects (font (size 1.27 1.27)))
     )
@@
   (symbol (lib_id "Device:C") (at 310.0 107.0 0) (unit 1)
     (in_bom yes) (on_board yes) (fields_autoplaced)
-    (property "Reference" "C3" (id 0) (at 310.0 101.92 0)
+    (property "Reference" "C203" (id 0) (at 310.0 101.92 0)
       (effects (font (size 1.27 1.27)))
     )
@@
   (symbol (lib_id "power:GND") (at 310.0 118.43 0) (unit 1)
     (in_bom yes) (on_board yes) (fields_autoplaced)
-    (property "Reference" "#PWR5" (id 0) (at 310.0 113.35000000000001 0)
+    (property "Reference" "#PWR205" (id 0) (at 310.0 113.35000000000001 0)
       (effects (font (size 1.27 1.27)) hide)
     )
@@
   (symbol (lib_id "Device:C") (at 332.0 107.0 0) (unit 1)
     (in_bom yes) (on_board yes) (fields_autoplaced)
-    (property "Reference" "C4" (id 0) (at 332.0 101.92 0)
+    (property "Reference" "C204" (id 0) (at 332.0 101.92 0)
       (effects (font (size 1.27 1.27)))
     )
@@
   (symbol (lib_id "power:GND") (at 332.0 118.43 0) (unit 1)
     (in_bom yes) (on_board yes) (fields_autoplaced)
-    (property "Reference" "#PWR6" (id 0) (at 332.0 113.35000000000001 0)
+    (property "Reference" "#PWR206" (id 0) (at 332.0 113.35000000000001 0)
       (effects (font (size 1.27 1.27)) hide)
     )
@@
   (symbol (lib_id "Device:R") (at 380.0 101.0 0) (unit 1)
     (in_bom yes) (on_board yes) (fields_autoplaced)
-    (property "Reference" "R5" (id 0) (at 380.0 95.92 0)
+    (property "Reference" "R205" (id 0) (at 380.0 95.92 0)
       (effects (font (size 1.27 1.27)))
     )
@@
   (symbol (lib_id "Device:R") (at 380.0 119.0 0) (unit 1)
     (in_bom yes) (on_board yes) (fields_autoplaced)
-    (property "Reference" "R6" (id 0) (at 380.0 113.92 0)
+    (property "Reference" "R206" (id 0) (at 380.0 113.92 0)
       (effects (font (size 1.27 1.27)))
     )
@@
   (symbol (lib_id "power:GND") (at 380.0 130.43 0) (unit 1)
     (in_bom yes) (on_board yes) (fields_autoplaced)
-    (property "Reference" "#PWR7" (id 0) (at 380.0 125.35000000000001 0)
+    (property "Reference" "#PWR207" (id 0) (at 380.0 125.35000000000001 0)
       (effects (font (size 1.27 1.27)) hide)
     )
@@
   (symbol (lib_id "ecu25kva:TLV76733") (at 170.0 200.0 0) (unit 1)
     (in_bom yes) (on_board yes) (fields_autoplaced)
-    (property "Reference" "U2" (id 0) (at 170.0 194.92 0)
+    (property "Reference" "U202" (id 0) (at 170.0 194.92 0)
       (effects (font (size 1.27 1.27)))
     )
@@
   (symbol (lib_id "power:GND") (at 167.46 224.13 0) (unit 1)
     (in_bom yes) (on_board yes) (fields_autoplaced)
-    (property "Reference" "#PWR8" (id 0) (at 167.46 219.04999999999998 0)
+    (property "Reference" "#PWR208" (id 0) (at 167.46 219.04999999999998 0)
       (effects (font (size 1.27 1.27)) hide)
     )
@@
   (symbol (lib_id "Device:C") (at 90.0 216.19 0) (unit 1)
     (in_bom yes) (on_board yes) (fields_autoplaced)
-    (property "Reference" "C5" (id 0) (at 90.0 211.10999999999999 0)
+    (property "Reference" "C205" (id 0) (at 90.0 211.10999999999999 0)
       (effects (font (size 1.27 1.27)))
     )
@@
   (symbol (lib_id "power:GND") (at 90.0 227.62 0) (unit 1)
     (in_bom yes) (on_board yes) (fields_autoplaced)
-    (property "Reference" "#PWR9" (id 0) (at 90.0 222.54 0)
+    (property "Reference" "#PWR209" (id 0) (at 90.0 222.54 0)
       (effects (font (size 1.27 1.27)) hide)
     )
@@
   (symbol (lib_id "Device:C") (at 235.0 218.19 0) (unit 1)
     (in_bom yes) (on_board yes) (fields_autoplaced)
-    (property "Reference" "C6" (id 0) (at 235.0 213.10999999999999 0)
+    (property "Reference" "C206" (id 0) (at 235.0 213.10999999999999 0)
       (effects (font (size 1.27 1.27)))
     )
@@
   (symbol (lib_id "power:GND") (at 235.0 229.62 0) (unit 1)
     (in_bom yes) (on_board yes) (fields_autoplaced)
-    (property "Reference" "#PWR10" (id 0) (at 235.0 224.54 0)
+    (property "Reference" "#PWR210" (id 0) (at 235.0 224.54 0)
       (effects (font (size 1.27 1.27)) hide)
     )
@@
   (symbol (lib_id "Device:Polyfuse") (at 110.0 318.0 0) (unit 1)
     (in_bom yes) (on_board yes) (fields_autoplaced)
-    (property "Reference" "F1" (id 0) (at 110.0 312.92 0)
+    (property "Reference" "F201" (id 0) (at 110.0 312.92 0)
       (effects (font (size 1.27 1.27)))
     )
@@
   (symbol (lib_id "Device:Polyfuse") (at 170.0 318.0 0) (unit 1)
     (in_bom yes) (on_board yes) (fields_autoplaced)
-    (property "Reference" "F2" (id 0) (at 170.0 312.92 0)
+    (property "Reference" "F202" (id 0) (at 170.0 312.92 0)
       (effects (font (size 1.27 1.27)))
     )
@@
   (symbol (lib_id "Device:Polyfuse") (at 230.0 318.0 0) (unit 1)
     (in_bom yes) (on_board yes) (fields_autoplaced)
-    (property "Reference" "F3" (id 0) (at 230.0 312.92 0)
+    (property "Reference" "F203" (id 0) (at 230.0 312.92 0)
       (effects (font (size 1.27 1.27)))
     )
@@
   (symbol (lib_id "Device:R") (at 440.0 316.0 0) (unit 1)
     (in_bom yes) (on_board yes) (fields_autoplaced)
-    (property "Reference" "R7" (id 0) (at 440.0 310.92 0)
+    (property "Reference" "R207" (id 0) (at 440.0 310.92 0)
       (effects (font (size 1.27 1.27)))
     )
@@
   (symbol (lib_id "Device:R") (at 440.0 334.0 0) (unit 1)
     (in_bom yes) (on_board yes) (fields_autoplaced)
-    (property "Reference" "R8" (id 0) (at 440.0 328.92 0)
+    (property "Reference" "R208" (id 0) (at 440.0 328.92 0)
       (effects (font (size 1.27 1.27)))
     )
@@
   (symbol (lib_id "power:GND") (at 440.0 345.43 0) (unit 1)
     (in_bom yes) (on_board yes) (fields_autoplaced)
-    (property "Reference" "#PWR11" (id 0) (at 440.0 340.35 0)
-      (effects (font (size 1.27 1.27)) hide)
-    )
+    (property "Reference" "#PWR211" (id 0) (at 440.0 340.35 0)
+      (effects (font (size 1.27 1.27)) hide)
+    )

Commit message: Check the project netlist, and fix the three things it caught
hw/check_netlist.py grew the two checks that found them, so neither can
come back quietly. It is the counterpart to sim/run_sim.py: that one
guards the component values, this one guards the connectivity.

5V_MAIN WAS FOUR NETS. The buck's 5 V output is a board rail -- both CAN
transceivers' VCC, the five difference amplifiers and the discrete
inputs' pull-ups run off it -- and it was a LOCAL label on every one of
those sheets. A local label stops at its sheet's edge, so three of the
four copies had no regulator on them. Each sheet's own netlist was
correct, which is exactly why ten clean per-sheet netlists never found
it. rails now exports it as a hierarchical label.

3V3_MCU WAS THREE. Same mechanism on can (both transceivers' VIO) and
speed_inputs, where the comparator's supply, both upper clamp diodes and
the bias divider sat on a five-pin net with no rail attached.

New check: any sheet-local net whose name shadows a project-wide net
name fails. That is the exact shape of both defects.

FIVE SUPPLY PINS HAD NO DECOUPLING CAPACITOR. The difference amplifiers
on sensors_analog were the only undecoupled supply pins on the board. No
simulation block was ever going to say so -- sensor_differential.cir
models an ideal amplifier with no supply pin at all. 100 nF each, at the
pin.

New check: walk every power_in pin in the project netlist and ask
whether a capacitor sits on the same net. 22 supply pins, all covered.
One documented exemption, the LM5164's BST pin, whose bootstrap
capacitor IS the net.

Gate now: 201 components with unique references, 108 named nets carrying
two or more pins, 18 reaching one and each a recorded open item, GND 139
pins, 3V3_MCU 36, 5V_MAIN 28, VBAT_PROT 12.

Schematic set re-plotted: docs/pdf/ECU-Schematics.pdf, 11 pages.
Suite still 24/24.

Co-Authored-By: Claude Opus 5 <noreply@anthropic.com>
Changed lines of the file:
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@@
   (junction (at 356.0 85.0) (diameter 0) (color 0 0 0 0)
   )
-  (label "5V_MAIN" (at 356.0 85.0 0)
-    (effects (font (size 1.27 1.27)) (justify left bottom))
+  (hierarchical_label "5V_MAIN" (shape output) (at 356.0 85.0 0)
+    (effects (font (size 1.27 1.27)) (justify left))
   )
   (symbol (lib_id "Device:R") (at 380.0 101.0 0) (unit 1)
