File: hw/rails.kicad_sch (KiCad schematic)
At the start: 41 parts, among them Q201 IPD90N10S4-06, U201 LM5164, U202 TLV76733, U203 TPS48110, U204 TPS7B4253, U205 TPS7B4253, U206 TPS7B4253

Commit message: Draw the four missing land patterns: SMPD, WE-PD 1050, DGX0019A, DDA0008J
Each comes from the maker's recommended layout, written in KiCad 7
format by gen_footprints.py:
- Vishay SMPD (doc 95604) for D408-D414: tab = cathode = pad 1, both
  leads = anode = pad 2, matching Device:D
- Wurth WE-PD 1050 for L201: 3.5 x 2.0 pads, 7.0 inner gap
- TI DGX0019A for U203: 0.5 mm pitch, position 16 empty
- TI DDA0008J for U204-U206: 2.95 x 4.9 thermal copper with a
  2.6 x 3.2 solder-mask-defined opening, which no stock variant has

The installed KiCad 10 stock library is newer than KiCad 7 can open, so
the two renumbered stock copies are skipped rather than rewritten.
363 of 365 components now have a footprint; J1001 (Bosch drawing) and
D806 (trip-loop clamp) remain.
Parts:
- L201: footprint (none) -> ecu25kva:L_Wuerth_WE-PD-1050; Chosen Wurth WE-PD 1050, 33 uH, Isat 2.9 A typ, IR 2.5 A, 79 mOhm max, AEC-Q200 Grade 1. No WE-PD land pattern in KiCad 7 -- drawn in phase 3 from the Wurth drawing -> Wurth WE-PD 1050, 33 uH, Isat 2.9 A typ, IR 2.5 A, 79 mOhm max, AEC-Q200 Grade 1. No WE-PD 1050 land pattern in KiCad 7 -- drawn from the Wurth drawing (gen_footprints.py)
- U203: footprint (none) -> ecu25kva:TI_DGX0019A_VSSOP-19_3x5.1mm_P0.5mm
- U204, U205, U206: footprint (none) -> ecu25kva:TI_DDA0008J_HSOIC-8_EP2.95x4.9_Mask2.6x3.2
Changed lines of the file:
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@@
       (effects (font (size 1.27 1.27)))
     )
-    (property "Footprint" "" (id 2) (at 284.0 85.0 0)
+    (property "Footprint" "ecu25kva:L_Wuerth_WE-PD-1050" (id 2) (at 284.0 85.0 0)
       (effects (font (size 1.27 1.27)) hide)
     )
@@
       (effects (font (size 1.27 1.27)) hide)
     )
-    (property "Chosen" "Wurth WE-PD 1050, 33 uH, Isat 2.9 A typ, IR 2.5 A, 79 mOhm max, AEC-Q200 Grade 1. No WE-PD land pattern in KiCad 7 -- drawn in phase 3 from the Wurth drawing" (id 6) (at 284.0 85.0 0)
+    (property "Chosen" "Wurth WE-PD 1050, 33 uH, Isat 2.9 A typ, IR 2.5 A, 79 mOhm max, AEC-Q200 Grade 1. No WE-PD 1050 land pattern in KiCad 7 -- drawn from the Wurth drawing (gen_footprints.py)" (id 6) (at 284.0 85.0 0)
       (effects (font (size 1.27 1.27)) hide)
     )
@@
       (effects (font (size 1.27 1.27)))
     )
-    (property "Footprint" "" (id 2) (at 120.0 318.0 0)
+    (property "Footprint" "ecu25kva:TI_DGX0019A_VSSOP-19_3x5.1mm_P0.5mm" (id 2) (at 120.0 318.0 0)
       (effects (font (size 1.27 1.27)) hide)
     )
@@
       (effects (font (size 1.27 1.27)))
     )
-    (property "Footprint" "" (id 2) (at 300.0 318.0 0)
+    (property "Footprint" "ecu25kva:TI_DDA0008J_HSOIC-8_EP2.95x4.9_Mask2.6x3.2" (id 2) (at 300.0 318.0 0)
       (effects (font (size 1.27 1.27)) hide)
     )
@@
       (effects (font (size 1.27 1.27)))
     )
-    (property "Footprint" "" (id 2) (at 370.0 318.0 0)
+    (property "Footprint" "ecu25kva:TI_DDA0008J_HSOIC-8_EP2.95x4.9_Mask2.6x3.2" (id 2) (at 370.0 318.0 0)
       (effects (font (size 1.27 1.27)) hide)
     )
@@
       (effects (font (size 1.27 1.27)))
     )
-    (property "Footprint" "" (id 2) (at 440.0 318.0 0)
-      (effects (font (size 1.27 1.27)) hide)
-    )
+    (property "Footprint" "ecu25kva:TI_DDA0008J_HSOIC-8_EP2.95x4.9_Mask2.6x3.2" (id 2) (at 440.0 318.0 0)
+      (effects (font (size 1.27 1.27)) hide)
+    )
