File: hw/discrete_io.kicad_sch (KiCad schematic)
At the start: 0 parts

Commit message: Draw the discrete I/O sheet; the trip sense needed an ADC, not a GPIO
Six input channels and two relay drivers, from discrete_input.cir,
trip_module_sense.cir and relay_driver.cir.

THE PIN MAP HAD THE TRIP SENSE ON A GPIO. trip_module_sense.cir designs
a three-state supervised loop and checks all three bands with real
margin -- healthy 2.863-2.954 V, tripped 0.310-2.068 V, wire fault
0.000 V. A GPIO reads two states. It separates healthy from not-healthy
and nothing else, which throws away exactly the distinction the 1.2 MOhm
bleed resistor exists to create: a supervised loop that cannot tell a
trip from a cut wire is an unsupervised loop with extra parts in it.

PTD6 is not ADC-capable, and neither is any other pin in pinmap sec.1.4 --
correct for those channels, wrong for this one. The channel moves to
PTB0 (ADC0_SE4), free, bonded out at package pin 78, Hi-Z with no pull
at reset. PTD6 returns to the spare pool. pinmap.md carries the
correction and the band table; the mcu sheet follows.

That row previously read "placeholder pin only -- front-end is
undesigned". The front-end has since been designed, and designing it
invalidated the pin class. Nothing rechecked the assignment against the
block that superseded it.

The rest of the sheet:

The 47k/68k/220nF/3.0V front-end is used unchanged on all six inputs.
The two whose switch is a contact to ground rather than a feed get a 10k
pull-up BEFORE the 47k, so a battery short on the harness still meets
the clamp chain rather than the pull-up -- an open contact then sits at
2.72 V, under the zener knee, reading high without the clamp conducting.

Relay FETs are 100 V class. Coil current is only 84 mA, so Rds(on) is
not the constraint; the drain sitting on VBAT_PROT is. Their gate
pulldowns are 10k rather than the 470 ohm supervisor.cir sized for the
six driver gates, and the difference is reasoned rather than copied:
that figure came from Miller coupling at Crss = 500 pF on a node
swinging to a 100 V boost rail, where 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
Parts:
- added C1, C2, C3, C4, C5, C6: 220nF, symbol Device:C
- added D1, D2, D3, D4, D5, D6: 3.0V, symbol Device:D_Zener
- added D7, D8: 100V 1A fast, symbol Device:D
- added Q1, Q2: 100V logic-level N-ch, symbol Device:Q_NMOS_GSD
- added R1, R11, R13, R3, R5, R8: 47k, symbol Device:R
- added R10, R15, R16, R7: 10k, symbol Device:R
- added R12, R14, R2, R4, R6, R9: 68k, symbol Device:R
Connections:
- new net 5V_MAIN: R10.1, R7.1
- new net GND: C1.2, C2.2, C3.2, C4.2, C5.2, C6.2, D1.2 (A), D2.2 (A), D3.2 (A), D4.2 (A), D5.2 (A), D6.2 (A), Q1.2 (S), Q2.2 (S), R12.2, R14.2, R15.2, R16.2, R2.2, R4.2, R6.2, R9.2
- new net IN_AUDIO_ABORT: C1.1, D1.1 (K), R1.2, R2.1
- new net IN_AUDIO_ABORT_H: R1.1
- new net IN_IGNITION: C3.1, D3.1 (K), R5.2, R6.1
- new net IN_IGNITION_H: R5.1
- new net IN_OVERRIDE_SS: C2.1, D2.1 (K), R3.2, R4.1
- new net IN_OVERRIDE_SS_H: R3.1
- new net RLY_BUZZER: Q2.1 (G), R16.1
- new net RLY_BUZZER_OUT: D8.2 (A), Q2.3 (D)
- new net RLY_MAIN: Q1.1 (G), R15.1
- new net RLY_MAIN_OUT: D7.2 (A), Q1.3 (D)
- new net SW_COOLANT: C4.1, D4.1 (K), R8.2, R9.1
- new net SW_COOLANT_C: R7.2, R8.1
- new net SW_DROOP: C5.1, D5.1 (K), R11.2, R12.1
- new net SW_DROOP_C: R10.2, R11.1
- new net TRIP_LOOP: R13.1
- new net TRIP_SENSE: C6.1, D6.1 (K), R13.2, R14.1
- new net VBAT_PROT: D7.1 (K), D8.1 (K)
Other:
- note added: "ECU pin 20 -- audio abort, active high -> PTD11"
- note added: "ECU pin 23 -- droop switch, contact to ground -> PTD7"
- note added: "ECU pin 24 -- override start/stop, active high -> PTD12"
- note added: "ECU pin 43 -- coolant switch, contact to ground -> PTD5"
- note added: "ECU pin 50 -- main relay, low side <- PTD13"
- note added: "ECU pin 69 -- buzzer relay, low side <- PTD14"
- note added: "ECU pin 71 -- ignition, active high -> PTD16"
- note added: "NEW pin -- supervised trip loop -> PTB0 (ADC0_SE4), not PTD6"
- note added: "TRIP SENSE MOVES FROM PTD6 TO PTB0 (ADC0_SE4). docs/pinmap.md assigns it as a GPIO input; trip_module_sense.cir designs a THREE-STATE supervised loop and checks the three bands with real margins -- healthy 2.863-2.954 V, tripped 0.310-2.068 V, wire fault 0.000 V. A GPIO reads two states. It separates healthy from not-healthy and nothing else, which discards exactly the distinction the bleed resis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"
- note added: "WHY THE SAME FRONT-END ON EVERY CHANNEL. The 47k/68k/220nF/3.0V chain is discrete_input.cir's, and it is used unchanged on all six inputs -- including the two whose switch is a contact to ground rather than a feed. Those two get a 10k pull-up BEFORE the 47k, so a battery short on the harness still meets the clamp chain rather than the pull-up. An open contact then leaves the divider at 2.72 V, un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"
- title: Switch inputs, trip-module sense, relay drivers -> Discrete I/O: switch inputs, trip loop, relay drivers
