File: hw/discrete_io.kicad_sch (KiCad schematic)
At the start: 32 parts, among them Q801 100V logic-level N-ch, Q802 100V logic-level N-ch

Commit message: Clamp GATE_KILL at 12 V and buffer the relay gates to 5 V
Choosing the small-signal FETs found two gate-drive errors.

GATE_KILL is pulled to VBAT_PROT so the kill path survives a 3V3
brownout, but only FET gates load it, so it followed the rail to
73.3 V on pulse 2a -- 3.7x a +/-20 V Vgs rating. A BZX84-C12-Q now
holds it at 12.7 V (13.7 V hot); transient_clamp checks the margin,
the zener current and the pullup dissipation.

The relay FETs were driven straight from 3.3 V GPIOs, with a note
claiming full enhancement at 3.0 V. No 100 V automotive small-signal
FET checked (PMV280ENEA, DMN10H220LQ, BSS123N) is specified below
Vgs = 4.5 V. An SN74AHCT1G125-Q1 on 5V_MAIN now drives each gate,
with a 100k input pulldown for reset; relay_driver checks overdrive
and drop.

Parts: 2N7002BK for the nine kill FETs and the reset inverter,
PMV280ENEA for the relay FETs. Also fixes the diagonal VBAT_PROT wire
to both relay flyback diodes.

24/24 sim blocks, netlist gate passing, 43 of 297 parts with footprints.
Parts:
- added C807, C808: 100nF, symbol Device:C
- added R817: 100k, symbol Device:R
- added R818: 10k, symbol Device:R
- added U801, U802: SN74AHCT1G125-Q1, Package_TO_SOT_SMD:SOT-23-5, symbol ecu25kva:AHCT1G125
- Q801, Q802: value 100V logic-level N-ch -> PMV280ENEA; footprint (none) -> Package_TO_SOT_SMD:SOT-23; MPN (none) -> PMV280ENEA; Source relay_driver.cir S1 (Ron 50 mOhm) -> relay_driver.cir S1 (Ron 50 mOhm); Nexperia PMV280ENEA data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; Vgs Fully enhanced at 3.0 V, driven straight from the GPIO -> Driven at 4.4 V min by the AHCT buffer: Rds(on) 432 mOhm ma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
- R815: value 10k -> 100k; Note 10k, NOT the 470 ohm supervisor.cir sized for the six drive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 -> (none); Source gate pulldown -- PTD13/PTD14 are Hi-Z with no pull at reset -> input pulldown -- relay OFF from reset until firmware drive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
Connections:
- net 5V_MAIN: now also C807.1, C808.1, U801.5 (VCC), U802.5 (VCC)
- net GND: now also C807.2, C808.2, R817.2, R818.2, U801.1 (~{OE}), U801.3 (GND), U802.1 (~{OE}), U802.3 (GND)
- net RLY_BUZZER: now also R817.1, U802.2 (A); no longer Q802.1 (G), R816.1
- net RLY_MAIN: now also U801.2 (A); no longer Q801.1 (G)
- new net: Q802.1 (G), R818.1, U802.4 (Y)
- new net: Q801.1 (G), R816.1, U801.4 (Y)

Commit message: Choose the diodes; the boost VDD clamp was 10 V over its pin rating
Part numbers for 27 diodes, each against a retrieved datasheet, applied
through one table (schlib.CHOSEN) keyed by symbol and class value, so
the class stays on the part as a field:
  VS-16EDH02HM3 x7   injector recirculation / blocking / freewheel
  VS-2EMH02HM3       boost diode
  VS-1EMH02HM3 x8    bootstrap and relay flyback
  VS-3ECH02HM3       metering freewheel
  SS20PH102HM3       negative-clamp backstop Schottky
  SMCJ43CA-HM3, SMAJ48CA-HE3, BZX84-C12-Q x2, BZX84-C13-Q, BZG03C36-HM3

The TPS40210 VDD clamp had been checked as an ideal 43.0 V source
behind 47 ohm. The real part in that class (40-46 V, +0.12 %/K, 45 ohm)
puts 61.9 V on a 52 V pin at 125 C, and its 40 V minimum conducts on
the load dump it was chosen to avoid. Now 220 ohm -- which the chosen
switch's gate charge allows -- and a 36 V zener: 46.6 V worst case with
tolerance, tempco and impedance, 33 mA on the dump. 39 V was tried
first; the transient_clamp rail table rejected it at 1.05x. The old
design stays as a pinned check.

TO-277A and SOT-23 zeners put the cathode on pad 3. gen_footprints.py
derives renumbered copies into lib/ecu25kva.pretty (new fp-lib-table).
The GATE_KILL zener, footprinted in the previous commit with the stock
SOT-23, had been reversed.

Left open as LOWV-CLAMP: the 15 zeners at 3.0 and 3.3 V. At tens of uA
a sub-5 V zener's knee is soft -- the datasheet allows 10 uA at 1 V --
and the model's sharp-knee zener hides it.

24/24 sim blocks, netlist gate passing, 74 of 297 parts with footprints.
Parts:
- D807, D808: value 100V 1A fast -> VS-1EMH02HM3; footprint (none) -> Diode_SMD:D_SMA; Chosen (none) -> The bootstrap diode's part: 200 V covers the 100 V class, a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; Class (none) -> 100V 1A fast; MPN (none) -> VS-1EMH02HM3
Changed lines of the file:
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@@
       (effects (font (size 1.27 1.27)))
     )
-    (property "Value" "100V 1A fast" (id 1) (at 90.0 242.08 0)
-      (effects (font (size 1.27 1.27)))
-    )
-    (property "Footprint" "" (id 2) (at 90.0 237.0 0)
+    (property "Value" "VS-1EMH02HM3" (id 1) (at 90.0 242.08 0)
+      (effects (font (size 1.27 1.27)))
+    )
+    (property "Footprint" "Diode_SMD:D_SMA" (id 2) (at 90.0 237.0 0)
       (effects (font (size 1.27 1.27)) hide)
     )
@@
       (effects (font (size 1.27 1.27)) hide)
     )
-    (property "Source" "relay_driver.cir D1" (id 4) (at 90.0 237.0 0)
-      (effects (font (size 1.27 1.27)) hide)
-    )
-    (property "Note" "Without it, interrupting 84 mA in a 1.2 H coil has nowhere to go -- relay_driver.cir's second branch is that case. Cathode to battery." (id 5) (at 90.0 237.0 0)
-      (effects (font (size 1.27 1.27)) hide)
-    )
-    (property "Vr" "100 V class, per transient_clamp's rail rating" (id 6) (at 90.0 237.0 0)
+    (property "MPN" "VS-1EMH02HM3" (id 4) (at 90.0 237.0 0)
+      (effects (font (size 1.27 1.27)) hide)
+    )
+    (property "Class" "100V 1A fast" (id 5) (at 90.0 237.0 0)
+      (effects (font (size 1.27 1.27)) hide)
+    )
+    (property "Chosen" "The bootstrap diode's part: 200 V covers the 100 V class, and one part number beats two" (id 6) (at 90.0 237.0 0)
+      (effects (font (size 1.27 1.27)) hide)
+    )
+    (property "Source" "relay_driver.cir D1" (id 7) (at 90.0 237.0 0)
+      (effects (font (size 1.27 1.27)) hide)
+    )
+    (property "Note" "Without it, interrupting 84 mA in a 1.2 H coil has nowhere to go -- relay_driver.cir's second branch is that case. Cathode to battery." (id 8) (at 90.0 237.0 0)
+      (effects (font (size 1.27 1.27)) hide)
+    )
+    (property "Vr" "100 V class, per transient_clamp's rail rating" (id 9) (at 90.0 237.0 0)
       (effects (font (size 1.27 1.27)) hide)
     )
@@
       (effects (font (size 1.27 1.27)))
     )
-    (property "Value" "100V 1A fast" (id 1) (at 290.0 242.08 0)
-      (effects (font (size 1.27 1.27)))
-    )
-    (property "Footprint" "" (id 2) (at 290.0 237.0 0)
+    (property "Value" "VS-1EMH02HM3" (id 1) (at 290.0 242.08 0)
+      (effects (font (size 1.27 1.27)))
+    )
+    (property "Footprint" "Diode_SMD:D_SMA" (id 2) (at 290.0 237.0 0)
       (effects (font (size 1.27 1.27)) hide)
     )
@@
       (effects (font (size 1.27 1.27)) hide)
     )
-    (property "Source" "relay_driver.cir D1" (id 4) (at 290.0 237.0 0)
-      (effects (font (size 1.27 1.27)) hide)
-    )
-    (property "Note" "Without it, interrupting 84 mA in a 1.2 H coil has nowhere to go -- relay_driver.cir's second branch is that case. Cathode to battery." (id 5) (at 290.0 237.0 0)
-      (effects (font (size 1.27 1.27)) hide)
-    )
-    (property "Vr" "100 V class, per transient_clamp's rail rating" (id 6) (at 290.0 237.0 0)
-      (effects (font (size 1.27 1.27)) hide)
-    )
+    (property "MPN" "VS-1EMH02HM3" (id 4) (at 290.0 237.0 0)
+      (effects (font (size 1.27 1.27)) hide)
+    )
+    (property "Class" "100V 1A fast" (id 5) (at 290.0 237.0 0)
+      (effects (font (size 1.27 1.27)) hide)
+    )
+    (property "Chosen" "The bootstrap diode's part: 200 V covers the 100 V class, and one part number beats two" (id 6) (at 290.0 237.0 0)
+      (effects (font (size 1.27 1.27)) hide)
+    )
+    (property "Source" "relay_driver.cir D1" (id 7) (at 290.0 237.0 0)
+      (effects (font (size 1.27 1.27)) hide)
+    )
+    (property "Note" "Without it, interrupting 84 mA in a 1.2 H coil has nowhere to go -- relay_driver.cir's second branch is that case. Cathode to battery." (id 8) (at 290.0 237.0 0)
+      (effects (font (size 1.27 1.27)) hide)
+    )
+    (property "Vr" "100 V class, per transient_clamp's rail rating" (id 9) (at 290.0 237.0 0)
+      (effects (font (size 1.27 1.27)) hide)
+    )

Commit message: Package every resistor and capacitor from the voltage across it
hw/assign_passives.py sizes all 188 chip R and C from a per-net table
of continuous and peak voltage (73.3 V pulse 2a, 104 V boost, bootstrap
domains riding on the bank nodes), against Vishay CRCW e3 resistor
ratings (Umax with 1.09x margin, power derated to 0.588x at a 105 C
board) and KEMET's automotive X7R waterfall (parsed by x-coordinate;
the text layout misreads its columns). schlib.place() applies the map
by ref and value; check_netlist fails on any unpackaged R or C.

Found along the way:
- 4.7 uF at 100 V is not in automotive X7R. The EMI filter C1, buck
  input and boost input are now 2 x 2.2 uF 100 V 1210; emi_filter.cir
  models the pair and its cold corner was re-pinned (0.6 dB worse).
- The twelve 470 ohm gate pulldowns need 2010: 0.31 W each at 100%
  duty. Recorded; 1k may now be possible against the real Crss.
- Local labels at 180 degrees were justified in the wrong frame on
  every sheet -- the bug fixed for hierarchical labels earlier -- so
  their text sat across their own wire. Fixed in schlib.label().

Internal nodes whose voltage matters now carry names (FB_BOOST_MID,
CAN1_SPLIT, ...); auto-names like Net-(R407-Pad2) move when parts are
added ahead of them.

24/24 sim blocks, netlist gate passing, 264 of 302 parts footprinted.
Parts:
- C801, C802, C803, C804, C805, C806, C807, C808: footprint (none) -> Capacitor_SMD:C_0603_1608Metric
- R801, R803, R805, R807, R808, R810, R811, R813: footprint (none) -> Resistor_SMD:R_0805_2012Metric
- R802, R804, R806, R809, R812, R814, R815, R816, R817, R818: footprint (none) -> Resistor_SMD:R_0603_1608Metric
Connections:
- net RLY_BUZZER_G: now reaches Q802.1 (G), R818.1, U802.4 (Y)
- net RLY_MAIN_G: now reaches Q801.1 (G), R816.1, U801.4 (Y)
Changed lines of the file:
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@@
       (effects (font (size 1.27 1.27)))
     )
-    (property "Footprint" "" (id 2) (at 74.0 60.0 0)
+    (property "Footprint" "Resistor_SMD:R_0805_2012Metric" (id 2) (at 74.0 60.0 0)
       (effects (font (size 1.27 1.27)) hide)
     )
@@
       (effects (font (size 1.27 1.27)))
     )
-    (property "Footprint" "" (id 2) (at 94.0 78.0 0)
+    (property "Footprint" "Resistor_SMD:R_0603_1608Metric" (id 2) (at 94.0 78.0 0)
       (effects (font (size 1.27 1.27)) hide)
     )
@@
       (effects (font (size 1.27 1.27)))
     )
-    (property "Footprint" "" (id 2) (at 110.0 78.0 0)
+    (property "Footprint" "Capacitor_SMD:C_0603_1608Metric" (id 2) (at 110.0 78.0 0)
       (effects (font (size 1.27 1.27)) hide)
     )
@@
       (effects (font (size 1.27 1.27)))
     )
-    (property "Footprint" "" (id 2) (at 74.0 120.0 0)
+    (property "Footprint" "Resistor_SMD:R_0805_2012Metric" (id 2) (at 74.0 120.0 0)
       (effects (font (size 1.27 1.27)) hide)
     )
@@
       (effects (font (size 1.27 1.27)))
     )
-    (property "Footprint" "" (id 2) (at 94.0 138.0 0)
+    (property "Footprint" "Resistor_SMD:R_0603_1608Metric" (id 2) (at 94.0 138.0 0)
       (effects (font (size 1.27 1.27)) hide)
     )
@@
       (effects (font (size 1.27 1.27)))
     )
-    (property "Footprint" "" (id 2) (at 110.0 138.0 0)
+    (property "Footprint" "Capacitor_SMD:C_0603_1608Metric" (id 2) (at 110.0 138.0 0)
       (effects (font (size 1.27 1.27)) hide)
     )
@@
       (effects (font (size 1.27 1.27)))
     )
-    (property "Footprint" "" (id 2) (at 74.0 180.0 0)
+    (property "Footprint" "Resistor_SMD:R_0805_2012Metric" (id 2) (at 74.0 180.0 0)
       (effects (font (size 1.27 1.27)) hide)
     )
@@
       (effects (font (size 1.27 1.27)))
     )
-    (property "Footprint" "" (id 2) (at 94.0 198.0 0)
+    (property "Footprint" "Resistor_SMD:R_0603_1608Metric" (id 2) (at 94.0 198.0 0)
       (effects (font (size 1.27 1.27)) hide)
     )
@@
       (effects (font (size 1.27 1.27)))
     )
-    (property "Footprint" "" (id 2) (at 110.0 198.0 0)
+    (property "Footprint" "Capacitor_SMD:C_0603_1608Metric" (id 2) (at 110.0 198.0 0)
       (effects (font (size 1.27 1.27)) hide)
     )
@@
       (effects (font (size 1.27 1.27)))
     )
-    (property "Footprint" "" (id 2) (at 336.0 42.0 0)
+    (property "Footprint" "Resistor_SMD:R_0805_2012Metric" (id 2) (at 336.0 42.0 0)
       (effects (font (size 1.27 1.27)) hide)
     )
@@
       (effects (font (size 1.27 1.27)))
     )
-    (property "Footprint" "" (id 2) (at 354.0 60.0 0)
+    (property "Footprint" "Resistor_SMD:R_0805_2012Metric" (id 2) (at 354.0 60.0 0)
       (effects (font (size 1.27 1.27)) hide)
     )
@@
       (effects (font (size 1.27 1.27)))
     )
-    (property "Footprint" "" (id 2) (at 374.0 78.0 0)
+    (property "Footprint" "Resistor_SMD:R_0603_1608Metric" (id 2) (at 374.0 78.0 0)
       (effects (font (size 1.27 1.27)) hide)
     )
@@
       (effects (font (size 1.27 1.27)))
     )
-    (property "Footprint" "" (id 2) (at 390.0 78.0 0)
+    (property "Footprint" "Capacitor_SMD:C_0603_1608Metric" (id 2) (at 390.0 78.0 0)
       (effects (font (size 1.27 1.27)) hide)
     )
@@
       (effects (font (size 1.27 1.27)))
     )
-    (property "Footprint" "" (id 2) (at 336.0 102.0 0)
+    (property "Footprint" "Resistor_SMD:R_0805_2012Metric" (id 2) (at 336.0 102.0 0)
       (effects (font (size 1.27 1.27)) hide)
     )
@@
       (effects (font (size 1.27 1.27)))
     )
-    (property "Footprint" "" (id 2) (at 354.0 120.0 0)
+    (property "Footprint" "Resistor_SMD:R_0805_2012Metric" (id 2) (at 354.0 120.0 0)
       (effects (font (size 1.27 1.27)) hide)
     )
@@
       (effects (font (size 1.27 1.27)))
     )
-    (property "Footprint" "" (id 2) (at 374.0 138.0 0)
+    (property "Footprint" "Resistor_SMD:R_0603_1608Metric" (id 2) (at 374.0 138.0 0)
       (effects (font (size 1.27 1.27)) hide)
     )
@@
       (effects (font (size 1.27 1.27)))
     )
-    (property "Footprint" "" (id 2) (at 390.0 138.0 0)
+    (property "Footprint" "Capacitor_SMD:C_0603_1608Metric" (id 2) (at 390.0 138.0 0)
       (effects (font (size 1.27 1.27)) hide)
     )
@@
       (effects (font (size 1.27 1.27)))
     )
-    (property "Footprint" "" (id 2) (at 354.0 180.0 0)
+    (property "Footprint" "Resistor_SMD:R_0805_2012Metric" (id 2) (at 354.0 180.0 0)
       (effects (font (size 1.27 1.27)) hide)
     )
@@
       (effects (font (size 1.27 1.27)))
     )
-    (property "Footprint" "" (id 2) (at 374.0 198.0 0)
+    (property "Footprint" "Resistor_SMD:R_0603_1608Metric" (id 2) (at 374.0 198.0 0)
       (effects (font (size 1.27 1.27)) hide)
     )
@@
       (effects (font (size 1.27 1.27)))
     )
-    (property "Footprint" "" (id 2) (at 390.0 198.0 0)
+    (property "Footprint" "Capacitor_SMD:C_0603_1608Metric" (id 2) (at 390.0 198.0 0)
       (effects (font (size 1.27 1.27)) hide)
     )
@@
   (junction (at 101.84 265.92) (diameter 0) (color 0 0 0 0)
   )
+  (label "RLY_MAIN_G" (at 112.0 265.92 180)
+    (effects (font (size 1.27 1.27)) (justify right bottom))
+  )
   (wire (pts (xy 91.68 265.92) (xy 91.68 296.4))
     (stroke (width 0) (type default))
@@
       (effects (font (size 1.27 1.27)))
     )
-    (property "Footprint" "" (id 2) (at 63.74000000000001 273.54 0)
+    (property "Footprint" "Capacitor_SMD:C_0603_1608Metric" (id 2) (at 63.74000000000001 273.54 0)
       (effects (font (size 1.27 1.27)) hide)
     )
@@
   )
   (label "5V_MAIN" (at 51.04 269.73 180)
-    (effects (font (size 1.27 1.27)) (justify left bottom))
+    (effects (font (size 1.27 1.27)) (justify right bottom))
   )
   (wire (pts (xy 61.2 296.4) (xy 51.04 296.4))
@@
       (effects (font (size 1.27 1.27)))
     )
-    (property "Footprint" "" (id 2) (at 51.040000000000006 312.40000000000003 0)
+    (property "Footprint" "Resistor_SMD:R_0603_1608Metric" (id 2) (at 51.040000000000006 312.40000000000003 0)
       (effects (font (size 1.27 1.27)) hide)
     )
@@
       (effects (font (size 1.27 1.27)))
     )
-    (property "Footprint" "" (id 2) (at 101.84 281.92 0)
+    (property "Footprint" "Resistor_SMD:R_0603_1608Metric" (id 2) (at 101.84 281.92 0)
       (effects (font (size 1.27 1.27)) hide)
     )
@@
   (junction (at 301.84 265.92) (diameter 0) (color 0 0 0 0)
   )
+  (label "RLY_BUZZER_G" (at 312.0 265.92 180)
+    (effects (font (size 1.27 1.27)) (justify right bottom))
+  )
   (wire (pts (xy 291.68 265.92) (xy 291.68 296.4))
     (stroke (width 0) (type default))
@@
       (effects (font (size 1.27 1.27)))
     )
-    (property "Footprint" "" (id 2) (at 263.74 273.54 0)
+    (property "Footprint" "Capacitor_SMD:C_0603_1608Metric" (id 2) (at 263.74 273.54 0)
       (effects (font (size 1.27 1.27)) hide)
     )
@@
   )
   (label "5V_MAIN" (at 251.04 269.73 180)
-    (effects (font (size 1.27 1.27)) (justify left bottom))
+    (effects (font (size 1.27 1.27)) (justify right bottom))
   )
   (wire (pts (xy 261.2 296.4) (xy 251.04 296.4))
@@
       (effects (font (size 1.27 1.27)))
     )
-    (property "Footprint" "" (id 2) (at 251.04 312.40000000000003 0)
+    (property "Footprint" "Resistor_SMD:R_0603_1608Metric" (id 2) (at 251.04 312.40000000000003 0)
       (effects (font (size 1.27 1.27)) hide)
     )
@@
       (effects (font (size 1.27 1.27)))
     )
-    (property "Footprint" "" (id 2) (at 301.84 281.92 0)
-      (effects (font (size 1.27 1.27)) hide)
-    )
+    (property "Footprint" "Resistor_SMD:R_0603_1608Metric" (id 2) (at 301.84 281.92 0)
+      (effects (font (size 1.27 1.27)) hide)
+    )
