File: hw/discrete_io.kicad_sch (KiCad schematic)
At the start: 38 parts, among them Q801 PMV280ENEA, Q802 PMV280ENEA, U801 SN74AHCT1G125-Q1, U802 SN74AHCT1G125-Q1

Commit message: Replace the discrete-input clamps with NPN buffers
LOWV-CLAMP, discrete half. The five switch inputs (pins 20/24/71 and
the contact-to-ground 43/23) clamped a 6-40 V input to ~3.0 V
continuously, which no clamp does inside the pad's ratings: a 3.0 V
zener has a soft knee at uA, a BAV199 rail clamp parks the pad at
3.9 V, and an LM4040-class reference draws ~35 uA of bias below
breakdown (TI SNOS633N Fig. 5-4) -- more than the cranking-dip input
could supply.

Each input is now 10k into an NPN base (4.7k + 4.7 uF to ground,
BAV199-Q lower diode against reverse battery), PMBT3904-Q collector to
the pad with 10k to 3V3_MCU. The pad only ever sees 0..3.3 V. Logic is
inverted; pinmap.md records it.

discrete_input.cir is rewritten and checked at the worst corners, not
typical: hFE 30 (datasheet min 60, halved for -40 C) still pulls the
pad to 0.03 V from a 6 V input; a typical part at 125 C stays off below
1.3 V; the base holds -1.05 V on -24 V reverse battery against a 6 V
VEBO; one edge through a 5-chatter bounce. The input resistor is 10k,
not 100k, for 1.1 mA of contact wetting current at 12 V -- 0.11 mA lets
non-gold contacts oxidise open in the field.

Failure modes (transistor open -> stuck inactive, C-E short -> stuck
active) are recorded on the sheet for the firmware plausibility spec.
The trip loop keeps its analog clamp: its healthy band is the clamp
level.

24/24 sim blocks, netlist gate passing, 202 R/C packaged.
Parts:
- removed D801, D802, D803, D804, D805: 3.0V, symbol Device:D_Zener
- removed Q801, Q802: PMV280ENEA, Package_TO_SOT_SMD:SOT-23, symbol Device:Q_NMOS_GSD
- added D801, D802, D803, D804, D805: BAV199-Q, Package_TO_SOT_SMD:SOT-23, symbol ecu25kva:BAV199
- added Q801, Q802, Q803, Q804, Q805: PMBT3904-Q, Package_TO_SOT_SMD:SOT-23, symbol Device:Q_NPN_BEC
- added Q806, Q807: PMV280ENEA, Package_TO_SOT_SMD:SOT-23, symbol Device:Q_NMOS_GSD
- added R819: 68k, Resistor_SMD:R_0603_1608Metric, symbol Device:R
- added R820, R822: 100k, Resistor_SMD:R_0603_1608Metric, symbol Device:R
- added R821, R823: 10k, Resistor_SMD:R_0603_1608Metric, symbol Device:R
- C801, C802, C803, C804, C805: value 220nF -> 4.7uF; footprint Capacitor_SMD:C_0603_1608Metric -> Capacitor_SMD:C_0805_2012Metric; Note 68k * 220 nF = 15 ms, long against contact bounce and short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 -> (10k || 4.7k) x 4.7 uF = 15 ms debounce; Source discrete_input.cir C1 -- debounce and EMI -> discrete_input.cir C1
- R801, R811: value 47k -> 10k; Note Sets the zener's worst-case sink current: (40 - 3) / 47k = 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 -> 10k, not 100k: 1.1 mA of wetting current through a closed c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; Source discrete_input.cir R5 -> discrete_input.cir R1
- R802, R812: value 68k -> 4.7k; Note With the 47k above, a 115k divider -- but the zener is what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 -> Holds the base off: a harness floating at 1 V reads inactiv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; Source discrete_input.cir R6 -> discrete_input.cir R2
- R803, R813: value 47k -> 10k; footprint Resistor_SMD:R_0805_2012Metric -> Resistor_SMD:R_0603_1608Metric; Note Sets the zener's worst-case sink current: (40 - 3) / 47k = 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 -> Pad pull-up to its own rail -- the pad sees 0..3.3 V and no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; Source discrete_input.cir R5 -> discrete_input.cir Rpu
- R804: value 68k -> 10k; footprint Resistor_SMD:R_0603_1608Metric -> Resistor_SMD:R_0805_2012Metric; Note With the 47k above, a 115k divider -- but the zener is what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 -> 10k, not 100k: 1.1 mA of wetting current through a closed c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; Source discrete_input.cir R6 -> discrete_input.cir R1
- R805, R808: value 47k -> 4.7k; footprint Resistor_SMD:R_0805_2012Metric -> Resistor_SMD:R_0603_1608Metric; Note Sets the zener's worst-case sink current: (40 - 3) / 47k = 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 -> Holds the base off: a harness floating at 1 V reads inactiv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; Source discrete_input.cir R5 -> discrete_input.cir R2
- R806, R809: value 68k -> 10k; Note With the 47k above, a 115k divider -- but the zener is what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 -> Pad pull-up to its own rail -- the pad sees 0..3.3 V and no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; Source discrete_input.cir R6 -> discrete_input.cir Rpu
- R807: Note Open contact leaves the divider at 5 * 115/125 * 68/115 = 2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 -> 10k, not 100k: 1.1 mA of wetting current through a closed c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; Source pull-up for a switch-to-ground contact (pinmap sec.1.4) -> discrete_input.cir R1
- R810: Note Open contact leaves the divider at 5 * 115/125 * 68/115 = 2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 -> Contact open: 5 V through this and the 10k input resistor s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
- R814: value 68k -> 10k; footprint Resistor_SMD:R_0603_1608Metric -> Resistor_SMD:R_0805_2012Metric; Note With the 47k above, a 115k divider -- but the zener is what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 -> Contact open: 5 V through this and the 10k input resistor s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; Source discrete_input.cir R6 -> pull-up for a switch-to-ground contact (pinmap sec.1.4)
- R815: value 100k -> 10k; footprint Resistor_SMD:R_0603_1608Metric -> Resistor_SMD:R_0805_2012Metric; Note (none) -> 10k, not 100k: 1.1 mA of wetting current through a closed c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; Source input pulldown -- relay OFF from reset until firmware drive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 -> discrete_input.cir R1
- R816: value 10k -> 4.7k; Note 10k, NOT the 470 ohm supervisor.cir sized for the six drive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 -> Holds the base off: a harness floating at 1 V reads inactiv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; Source gate pulldown -- PTD13/PTD14 are Hi-Z with no pull at reset -> discrete_input.cir R2
- R817: value 100k -> 10k; Note (none) -> Pad pull-up to its own rail -- the pad sees 0..3.3 V and no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; Source input pulldown -- relay OFF from reset until firmware drive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 -> discrete_input.cir Rpu
- R818: value 10k -> 47k; footprint Resistor_SMD:R_0603_1608Metric -> Resistor_SMD:R_0805_2012Metric; Note 10k, NOT the 470 ohm supervisor.cir sized for the six drive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 -> Sets the zener's worst-case sink current: (40 - 3) / 47k = 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; Source gate pulldown -- PTD13/PTD14 are Hi-Z with no pull at reset -> discrete_input.cir R5
Connections:
- net 5V_MAIN: now also R814.1; no longer R807.1
- net GND: now also R805.2, R808.2, D801.1 (A1), D802.1 (A1), D803.1 (A1), D804.1 (A1), D805.1 (A1), Q801.2 (E), Q802.2 (E), Q803.2 (E), Q804.2 (E), Q805.2 (E), Q806.2 (S), Q807.2 (S), R819.2, R820.2, R821.2, R822.2, R823.2; no longer R804.2, R806.2, R809.2, R814.2, R815.2, R817.2, R818.2
- net IN_AUDIO_ABORT: now also R803.2, Q801.3 (C); no longer C801.1, R801.2, R802.1
- net IN_IGNITION: now also R809.2, Q803.3 (C); no longer C803.1, R805.2, R806.1
- net IN_IGNITION_H: now also R807.1; no longer R805.1
- net IN_OVERRIDE_SS: now also R806.2, Q802.3 (C); no longer C802.1, R803.2, R804.1
- net IN_OVERRIDE_SS_H: now also R804.1; no longer R803.1
- net RLY_BUZZER: now also R822.1; no longer R817.1
- net RLY_BUZZER_G: now also Q807.1 (G), R823.1; no longer R818.1
- net RLY_BUZZER_OUT: now also Q807.3 (D)
- net RLY_MAIN: now also R820.1; no longer R815.1
- net RLY_MAIN_G: now also Q806.1 (G), R821.1; no longer R816.1
- net RLY_MAIN_OUT: now also Q806.3 (D)
- net SW_COOLANT: now also R813.2, Q804.3 (C); no longer C804.1, R808.2, R809.1
- net SW_COOLANT_C: now also R810.2, R811.1; no longer R807.2, R808.1
- net SW_DROOP: now also R817.2, Q805.3 (C); no longer C805.1, R811.2, R812.1
- net SW_DROOP_C: now also R814.2, R815.1; no longer R810.2, R811.1
- net TRIP_LOOP: now also R818.1; no longer R813.1
- net TRIP_SENSE: now also R818.2, R819.1; no longer R813.2, R814.1
- new net 3V3_MCU: R803.1, R806.1, R809.1, R813.1, R817.1
- new net IN_AUDIO_ABORT_B: C801.1, D801.3 (COM), Q801.1 (B), R801.2, R802.1
- new net IN_IGNITION_B: C803.1, D803.3 (COM), Q803.1 (B), R807.2, R808.1
- new net IN_OVERRIDE_SS_B: C802.1, D802.3 (COM), Q802.1 (B), R804.2, R805.1
- new net SW_COOLANT_B: C804.1, D804.3 (COM), Q804.1 (B), R811.2, R812.1
- new net SW_DROOP_B: C805.1, D805.3 (COM), Q805.1 (B), R815.2, R816.1
Other:
- note added: "ECU pin 20 -- audio abort, active high -> PTD11 INVERTED: pad LOW = input active"
- note added: "ECU pin 23 -- droop switch, contact to ground -> PTD7 INVERTED: pad LOW = input active"
- note added: "ECU pin 24 -- override start/stop, active high -> PTD12 INVERTED: pad LOW = input active"
- note added: "ECU pin 43 -- coolant switch, contact to ground -> PTD5 INVERTED: pad LOW = input active"
- note added: "ECU pin 71 -- ignition, active high -> PTD16 INVERTED: pad LOW = input active"
- note added: "THE FIVE SWITCH INPUTS ARE NPN BUFFERS, NOT CLAMPS (22 Sep 2026, LOWV-CLAMP). The 47k/68k/3.0 V-zener front end needed a clamp that conducts CONTINUOUSLY over 6-40 V, and none fits the pad's ratings: a 3.0 V zener leaks at uA (soft knee), a rail clamp parks the pad at 3.9 V, a shunt reference draws 35 uA of bias the cranking-dip input cannot supply. Here the pad sees only its own 10k pull-up or a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"
- note removed: "ECU pin 20 -- audio abort, active high -> PTD11"
- note removed: "ECU pin 23 -- droop switch, contact to ground -> PTD7"
- note removed: "ECU pin 24 -- override start/stop, active high -> PTD12"
- note removed: "ECU pin 43 -- coolant switch, contact to ground -> PTD5"
- note removed: "ECU pin 71 -- ignition, active high -> PTD16"
- note removed: "WHY THE SAME FRONT-END ON EVERY CHANNEL. The 47k/68k/220nF/3.0V chain is discrete_input.cir's, and it is used unchanged on all six inputs -- including the two whose switch is a contact to ground rather than a feed. Those two get a 10k pull-up BEFORE the 47k, so a battery short on the harness still meets the clamp chain rather than the pull-up. An open contact then leaves the divider at 2.72 V, un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"
