File: hw/mcu.kicad_sch (KiCad schematic)
At the start: 0 parts

Commit message: Draw the mcu sheet, and choose the supervisor part
The S32K148 with all 144 pins wired, the TPS3850G33 watching its rail,
the inverting stage that turns the supervisor's active-low RESET into an
active-high GATE_KILL for the driver sheets, mcu_pdn.cir's decoupling
network, and the debug header. A2 rather than A3: six 25-pin units plus
a supervisor, a header and eleven decoupling parts do not fit A3 without
stacking, and a schematic whose parts overlap is one nobody reads.

THE SUPERVISOR IS NOW A PART, NOT A CLASS. Memo 11 had TPS3850 CONFIRMED
on its electricals but recommended it as "TPS3850-class", and the pinout
was never captured. Both are settled here from the retrieved datasheet
(TI SBVS301B, Table 5-1 and Figure 5-1), and the variant is chosen
rather than assumed. The nomenclature table gives G = thresholds at +/-4%
of nominal and H = +/-7%; with the part's own +/-0.8% accuracy that puts
the worst-case undervoltage trip at 3.143 V for G33 against 3.044 V for
H33. The supervisor exists to assert BEFORE the S32K148's own LVD, whose
maximum is 3.0 V, so G33 clears it by 143 mV and H33 by 44 mV -- close
enough that the two could fire in either order, and a supervisor that
might lose the race to the thing it supervises is not doing its job. The
cost is a tighter window the rail must live inside, 3.143-3.459 V, which
is now a constraint on the rails sheet.

THE PIN MAP HAD A GAP, and this sheet is what found it. Section 1.8 said
outright that "the only MCU pin in this interface is RESET_b". True of
the kill path, which deliberately involves no MCU pin -- and wrong about
the watchdog, which is not a passive monitor. The MCU has to present a
falling edge on WDI inside every window or the part resets the board on
a timer. A supervisor topology with no pin to kick it guarantees a reset
loop. PTE0 (WDT_KICK) and PTE1 (WDT_FAULT) are added, both free GPIO-HD,
both PE=0/PS=0 at reset, taking the map from 37 committed signals to 39.
WDO is worth its own pin because it ass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
Parts:
- added C1, C2: 10nF, symbol Device:C
- added C10, C11, C12, C3, C4, C5, C6, C7, C8, C9: 100nF, symbol Device:C
- added C13: 150uF, symbol Device:C_Polarized
- added J1: SWD/JTAG, Connector_PinHeader_1.27mm:PinHeader_2x05_P1.27mm_Vertical, symbol Connector:Conn_ARM_JTAG_SWD_10
- added Q1: 60V logic-level N-ch, symbol Device:Q_NMOS_GSD
- added R1, R2: 10k, symbol Device:R
- added R3, R4: 0R, symbol Device:R
- added R5: 47k, symbol Device:R
- added U1: S32K148_144LQFP, Package_QFP:LQFP-144_20x20mm_P0.5mm, symbol ecu25kva:S32K148_144LQFP
- added U2: TPS3850G33, Package_SON:VSON-10-1EP_3x3mm_P0.5mm_EP1.2x2mm, symbol ecu25kva:TPS3850G33
Connections:
- new net: R3.1, U2.3 (SET0)
- new net: C2.1, U2.2 (CWD)
- new net: C1.1, U2.4 (CRST)
- new net: R4.1, U2.6 (SET1)
- new net 3V3_MCU: C10.1, C11.1, C12.1, C13.1, C3.1, C4.1, C5.1, C6.1, C7.1, C8.1, C9.1, J1.1 (VTref), R1.1, R2.1, U1.11 (VDD), U1.124 (VDD), U1.13 (VDDA), U1.14 (VREFH), U1.32 (VDD), U1.51 (VDD), U1.67 (VDD), U1.91 (VDD), U2.1 (VDD), U2.10 (SENSE)
- new net BARO: U1.88 (PTD18)
- new net BOOST_P: U1.113 (PTA1)
- new net BOOST_T: U1.104 (PTA3)
- new net CAM_EDGE: U1.63 (PTB3)
- new net CAN1_RX: U1.9 (PTE4)
- new net CAN1_TX: U1.8 (PTE5)
- new net CAN2_RX: U1.118 (PTC6)
- new net CAN2_TX: U1.117 (PTC7)
- new net COOLANT_T: U1.85 (PTA6)
- new net CRANK_EDGE: U1.68 (PTB2)
- new net EGR_IN1: U1.111 (PTB8)
- new net EGR_IN2: U1.109 (PTB9)
- new net EGR_POS: U1.120 (PTA15)
- new net GATE_KILL: Q1.3 (D), R5.2
- new net GND: C1.2, C10.2, C11.2, C12.2, C13.2, C2.2, C3.2, C4.2, C5.2, C6.2, C7.2, C8.2, C9.2, J1.3 (GND), J1.5 (GND), J1.9 (GNDDetect), Q1.2 (S), R3.2, R4.2, U1.12 (VSS), U1.123 (VSS), U1.15 (VREFL), U1.16 (VSS), U1.31 (VSS), U1.50 (VSS), U1.66 (VSS), U1.90 (VSS), U2.5 (GND)
- new net INJ_HS_A: U1.53 (PTC0)
- new net INJ_HS_B: U1.52 (PTC1)
- new net INJ_LS_1: U1.43 (PTC2)
- new net INJ_LS_2: U1.41 (PTB4)
- new net INJ_LS_3: U1.42 (PTC3)
- new net IN_AUDIO_ABORT: U1.48 (PTD11)
- new net IN_IGNITION: U1.28 (PTD16)
- new net IN_OVERRIDE_SS: U1.47 (PTD12)
- new net ISNS_EGR: U1.99 (PTD22)
- new net ISNS_INJ_A: U1.59 (PTC15)
- new net ISNS_INJ_B: U1.89 (PTD19)
- new net ISNS_MU: U1.57 (PTC16)
- new net JTAG_TCK: J1.4 (SWCLK/TCK), U1.140 (PTC4[PD])
- new net JTAG_TDI: J1.8 (NC/TDI), U1.139 (PTC5[PU])
- new net JTAG_TMS: J1.2 (SWDIO/TMS), U1.142 (PTA4[PU])
- new net MU_PWM: U1.49 (PTD10)
- new net OIL_P: U1.83 (PTA7)
- new net RAIL_P: U1.119 (PTA16)
- new net RLY_BUZZER: U1.34 (PTD14)
- new net RLY_MAIN: U1.35 (PTD13)
- new net SENSOR_5V_MON: U1.61 (PTC14)
- new net SW_COOLANT: U1.46 (PTD5)
- new net SW_DROOP: U1.44 (PTD7)
- new net TRIP_SENSE: U1.45 (PTD6)
- new net VBAT_PROT: R5.1
- new net V_BAT_1R_SNS: U1.115 (PTA0)
- new net V_BAT_2R_SNS: U1.105 (PTA2)
- new net WDT_FAULT: J1.10 (~{RESET}), Q1.1 (G), R1.2, R2.2, U1.137 (PTE1), U1.141 (PTA5[PU]), U2.8 (~WDO), U2.9 (~RESET)
- new net WDT_KICK: U1.138 (PTE0), U2.7 (WDI)
Other:
- note added: "PIN MAP ADDITIONS MADE ON THIS SHEET -- both are gaps in docs/pinmap.md, not changes to it: PTE0 WDT_KICK MCU -> TPS3850 WDI. pinmap.md assigns 37 signals and none of them services the external watchdog, but memo 11's topology requires the MCU to kick it. A window watchdog nobody feeds resets the board on a timer. PTE1 WDT_FAULT TPS3850 WDO -> MCU, so firmware can tell a watchdog trip from a rail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"
- note added: "SUPERVISOR CHOICE -- TPS3850G33, from the datasheet's own nomenclature table (G = thresholds at +/-4% of nominal, H = +/-7%) and its +/-0.8% accuracy spec: G33 UV 3.168 V nom, 3.143 V worst-low | H33 UV 3.069 V nom, 3.044 V worst-low The supervisor has to assert BEFORE the MCU's own LVD (3.0 V max) and above the 2.97 V correctness floor. G33 clears LVD by 143 mV worst case; H33 by 44 mV, close en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"
- note added: "SWO/TDO left open -- see note"
- title: S32K148, supervisor and fail-safe gating -> MCU, supervisor and debug

Commit message: Draw the discrete I/O sheet; the trip sense needed an ADC, not a GPIO
Six input channels and two relay drivers, from discrete_input.cir,
trip_module_sense.cir and relay_driver.cir.

THE PIN MAP HAD THE TRIP SENSE ON A GPIO. trip_module_sense.cir designs
a three-state supervised loop and checks all three bands with real
margin -- healthy 2.863-2.954 V, tripped 0.310-2.068 V, wire fault
0.000 V. A GPIO reads two states. It separates healthy from not-healthy
and nothing else, which throws away exactly the distinction the 1.2 MOhm
bleed resistor exists to create: a supervised loop that cannot tell a
trip from a cut wire is an unsupervised loop with extra parts in it.

PTD6 is not ADC-capable, and neither is any other pin in pinmap sec.1.4 --
correct for those channels, wrong for this one. The channel moves to
PTB0 (ADC0_SE4), free, bonded out at package pin 78, Hi-Z with no pull
at reset. PTD6 returns to the spare pool. pinmap.md carries the
correction and the band table; the mcu sheet follows.

That row previously read "placeholder pin only -- front-end is
undesigned". The front-end has since been designed, and designing it
invalidated the pin class. Nothing rechecked the assignment against the
block that superseded it.

The rest of the sheet:

The 47k/68k/220nF/3.0V front-end is used unchanged on all six inputs.
The two whose switch is a contact to ground rather than a feed get a 10k
pull-up BEFORE the 47k, so a battery short on the harness still meets
the clamp chain rather than the pull-up -- an open contact then sits at
2.72 V, under the zener knee, reading high without the clamp conducting.

Relay FETs are 100 V class. Coil current is only 84 mA, so Rds(on) is
not the constraint; the drain sitting on VBAT_PROT is. Their gate
pulldowns are 10k rather than the 470 ohm supervisor.cir sized for the
six driver gates, and the difference is reasoned rather than copied:
that figure came from Miller coupling at Crss = 500 pF on a node
swinging to a 100 V boost rail, where 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
Connections:
- net TRIP_SENSE: now also U1.78 (PTB0); no longer U1.45 (PTD6)
Changed lines of the file:
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@@
     (effects (font (size 1.27 1.27)) (justify left))
   )
-  (wire (pts (xy 64.52 230.73) (xy 41.66 230.73))
+  (wire (pts (xy 239.52 61.49) (xy 216.66 61.49))
     (stroke (width 0) (type default))
   )
-  (hierarchical_label "TRIP_SENSE" (shape input) (at 41.66 230.73 180)
+  (hierarchical_label "TRIP_SENSE" (shape input) (at 216.66 61.49 180)
     (effects (font (size 1.27 1.27)) (justify left))
   )
