File: hw/mcu.kicad_sch (KiCad schematic)
At the start: 22 parts, among them J1 SWD/JTAG, Q1 60V logic-level N-ch, U1 S32K148_144LQFP, U2 TPS3850G33

Commit message: Draw the connector; the power ground turns out to have no pin
Sheet 10 of 10. Not a circuit -- the harness boundary, and its job is to
be checkable against the machine: every pin the wiring diagram shows
wired to the net whichever sheet owns that signal already named, and
every pin it does not show left visibly empty.

41 of 94 pins wired, 53 left empty, every pin accounted for exactly once
in the netlist.

THE FINDING. GP3.8703.C4.pdf shows pin 21 as the battery positive feed
and shows no battery negative anywhere on the ECU connector. That is a
gap in the source rather than a contradiction in it -- the document is a
field troubleshooting diagram and its own scope note says it omits
"power grounds, unused pins and internal-only pins". It is still a gap
that stops a board: every other sheet in this project returns to GND,
the injector low sides carry 18 A into it, and at this boundary that net
has nowhere to go. It cannot be closed by choosing. Fifty pins have no
established function and several are certainly grounds -- a 94-way
connector feeding an 18 A injector stage does not have one return -- but
a wrong ground pin is not a rework, it is a harness that has to be
remade. Same for TRIP_LOOP, which is a NEW signal not on the OEM diagram
at all and needs one of the same fifty.

CONN_ECU_94 carries pin count and pin numbers, which are facts read off
page 4, and no footprint, because no part number is known. Pin names are
the diagram's own signal names where it shows the pin and blank where it
does not. Same treatment the op-amps and the comparator get.

Two distinctions the sheet makes explicit: pins 34 and 36 are SHARED
sensor returns and therefore signals, carried into difference amplifiers
on sensors_analog; pin 08 is rail pressure's dedicated return, with
nothing to reject, so it is simply ground here.

CROSS-SHEET AUDIT. 83 hierarchical net names across the ten sheets, 73
appearing on two or more. All ten that appear on only one sheet are
explained by an open it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
Changed lines of the file:
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@@
   )
   (hierarchical_label "V_BAT_1R_SNS" (shape input) (at 41.66 62.76 180)
-    (effects (font (size 1.27 1.27)) (justify left))
+    (effects (font (size 1.27 1.27)) (justify right))
   )
   (wire (pts (xy 64.52 67.84) (xy 41.66 67.84))
@@
   )
   (hierarchical_label "V_BAT_2R_SNS" (shape input) (at 41.66 67.84 180)
-    (effects (font (size 1.27 1.27)) (justify left))
+    (effects (font (size 1.27 1.27)) (justify right))
   )
   (wire (pts (xy 64.52 65.3) (xy 41.66 65.3))
@@
   )
   (hierarchical_label "BOOST_P" (shape input) (at 41.66 65.3 180)
-    (effects (font (size 1.27 1.27)) (justify left))
+    (effects (font (size 1.27 1.27)) (justify right))
   )
   (wire (pts (xy 64.52 70.38) (xy 41.66 70.38))
@@
   )
   (hierarchical_label "BOOST_T" (shape input) (at 41.66 70.38 180)
-    (effects (font (size 1.27 1.27)) (justify left))
+    (effects (font (size 1.27 1.27)) (justify right))
   )
   (wire (pts (xy 64.52 78.0) (xy 41.66 78.0))
@@
   )
   (hierarchical_label "COOLANT_T" (shape input) (at 41.66 78.0 180)
-    (effects (font (size 1.27 1.27)) (justify left))
+    (effects (font (size 1.27 1.27)) (justify right))
   )
   (wire (pts (xy 125.48 67.84) (xy 148.34 67.84))
@@
   )
   (hierarchical_label "OIL_P" (shape input) (at 41.66 80.54 180)
-    (effects (font (size 1.27 1.27)) (justify left))
+    (effects (font (size 1.27 1.27)) (justify right))
   )
   (wire (pts (xy 125.48 70.38) (xy 148.34 70.38))
@@
   )
   (hierarchical_label "CRANK_EDGE" (shape input) (at 216.66 66.57 180)
-    (effects (font (size 1.27 1.27)) (justify left))
+    (effects (font (size 1.27 1.27)) (justify right))
   )
   (wire (pts (xy 239.52 69.11) (xy 216.66 69.11))
@@
   )
   (hierarchical_label "CAM_EDGE" (shape input) (at 216.66 69.11 180)
-    (effects (font (size 1.27 1.27)) (justify left))
+    (effects (font (size 1.27 1.27)) (justify right))
   )
   (wire (pts (xy 414.52 62.76) (xy 391.66 62.76))
@@
   )
   (hierarchical_label "INJ_HS_A" (shape output) (at 391.66 62.76 180)
-    (effects (font (size 1.27 1.27)) (justify left))
+    (effects (font (size 1.27 1.27)) (justify right))
   )
   (wire (pts (xy 414.52 65.3) (xy 391.66 65.3))
@@
   )
   (hierarchical_label "INJ_HS_B" (shape output) (at 391.66 65.3 180)
-    (effects (font (size 1.27 1.27)) (justify left))
+    (effects (font (size 1.27 1.27)) (justify right))
   )
   (wire (pts (xy 414.52 67.84) (xy 391.66 67.84))
@@
   )
   (hierarchical_label "INJ_LS_1" (shape output) (at 391.66 67.84 180)
-    (effects (font (size 1.27 1.27)) (justify left))
+    (effects (font (size 1.27 1.27)) (justify right))
   )
   (wire (pts (xy 414.52 70.38) (xy 391.66 70.38))
@@
   )
   (hierarchical_label "INJ_LS_3" (shape output) (at 391.66 70.38 180)
-    (effects (font (size 1.27 1.27)) (justify left))
+    (effects (font (size 1.27 1.27)) (justify right))
   )
   (wire (pts (xy 239.52 71.65) (xy 216.66 71.65))
@@
   )
   (hierarchical_label "INJ_LS_2" (shape output) (at 216.66 71.65 180)
-    (effects (font (size 1.27 1.27)) (justify left))
+    (effects (font (size 1.27 1.27)) (justify right))
   )
   (wire (pts (xy 64.52 240.89) (xy 41.66 240.89))
@@
   )
   (hierarchical_label "MU_PWM" (shape output) (at 41.66 240.89 180)
-    (effects (font (size 1.27 1.27)) (justify left))
+    (effects (font (size 1.27 1.27)) (justify right))
   )
   (wire (pts (xy 239.52 81.81) (xy 216.66 81.81))
@@
   )
   (hierarchical_label "EGR_IN1" (shape output) (at 216.66 81.81 180)
-    (effects (font (size 1.27 1.27)) (justify left))
+    (effects (font (size 1.27 1.27)) (justify right))
   )
   (wire (pts (xy 239.52 84.35) (xy 216.66 84.35))
@@
   )
   (hierarchical_label "EGR_IN2" (shape output) (at 216.66 84.35 180)
-    (effects (font (size 1.27 1.27)) (justify left))
+    (effects (font (size 1.27 1.27)) (justify right))
   )
   (wire (pts (xy 64.52 228.19) (xy 41.66 228.19))
@@
   )
   (hierarchical_label "SW_COOLANT" (shape input) (at 41.66 228.19 180)
-    (effects (font (size 1.27 1.27)) (justify left))
+    (effects (font (size 1.27 1.27)) (justify right))
   )
   (wire (pts (xy 64.52 233.27) (xy 41.66 233.27))
@@
   )
   (hierarchical_label "SW_DROOP" (shape input) (at 41.66 233.27 180)
-    (effects (font (size 1.27 1.27)) (justify left))
+    (effects (font (size 1.27 1.27)) (justify right))
   )
   (wire (pts (xy 64.52 243.43) (xy 41.66 243.43))
@@
   )
   (hierarchical_label "IN_AUDIO_ABORT" (shape input) (at 41.66 243.43 180)
-    (effects (font (size 1.27 1.27)) (justify left))
+    (effects (font (size 1.27 1.27)) (justify right))
   )
   (wire (pts (xy 64.52 245.97) (xy 41.66 245.97))
@@
   )
   (hierarchical_label "IN_OVERRIDE_SS" (shape input) (at 41.66 245.97 180)
-    (effects (font (size 1.27 1.27)) (justify left))
+    (effects (font (size 1.27 1.27)) (justify right))
   )
   (wire (pts (xy 125.48 220.57) (xy 148.34 220.57))
@@
   )
   (hierarchical_label "TRIP_SENSE" (shape input) (at 216.66 61.49 180)
-    (effects (font (size 1.27 1.27)) (justify left))
+    (effects (font (size 1.27 1.27)) (justify right))
   )
   (wire (pts (xy 64.52 248.51) (xy 41.66 248.51))
@@
   )
   (hierarchical_label "RLY_MAIN" (shape output) (at 41.66 248.51 180)
-    (effects (font (size 1.27 1.27)) (justify left))
+    (effects (font (size 1.27 1.27)) (justify right))
   )
   (wire (pts (xy 125.48 215.49) (xy 148.34 215.49))
@@
   )
   (hierarchical_label "CAN1_RX" (shape input) (at 216.66 228.19 180)
-    (effects (font (size 1.27 1.27)) (justify left))
+    (effects (font (size 1.27 1.27)) (justify right))
   )
   (wire (pts (xy 239.52 230.73) (xy 216.66 230.73))
@@
   )
   (hierarchical_label "CAN1_TX" (shape output) (at 216.66 230.73 180)
-    (effects (font (size 1.27 1.27)) (justify left))
+    (effects (font (size 1.27 1.27)) (justify right))
   )
   (wire (pts (xy 414.52 78.0) (xy 391.66 78.0))
@@
   )
   (hierarchical_label "CAN2_RX" (shape input) (at 391.66 78.0 180)
-    (effects (font (size 1.27 1.27)) (justify left))
+    (effects (font (size 1.27 1.27)) (justify right))
   )
   (wire (pts (xy 414.52 80.54) (xy 391.66 80.54))
@@
   )
   (hierarchical_label "CAN2_TX" (shape output) (at 391.66 80.54 180)
-    (effects (font (size 1.27 1.27)) (justify left))
+    (effects (font (size 1.27 1.27)) (justify right))
   )
   (wire (pts (xy 64.52 75.46) (xy 41.66 75.46))
@@
   )
   (hierarchical_label "3V3_MCU" (shape input) (at 267.92 384.84 180)
-    (effects (font (size 1.27 1.27)) (justify left))
+    (effects (font (size 1.27 1.27)) (justify right))
   )
   (wire (pts (xy 267.92 384.84) (xy 273.0 384.84))

Commit message: Wire the root sheet: the project has a netlist for the first time
Ten sheets each passed their own netlist and the project had none. The
root sheet's ten sheet symbols carried NO hierarchical pins, so a net
name appearing on two sheets was two nets and nothing compared them --
the cross-sheet audit in the last commit was a name comparison, not a
connectivity check.

Each symbol now carries one pin per net its child exports, read OUT of
the child rather than declared in a second list that could drift: 162
pins across the ten, each with a stub and a label. Two labels with the
same name are one net, which is how 162 pins connect without routing
162 wires across a page nobody could read.

Exporting it found the other half of the same problem immediately.
kicad-cli reported annotation errors: every sheet generator allocated
R1, C1, U1 from its own counter, so ten sheets had ten parts called R1.
schlib.REF_BASE gives each sheet its own hundred -- KiCad's own
sheet-number x 100 convention, applied at generation time instead of by
a hand pass in Eeschema. 196 components, no duplicate reference.

hw/check_netlist.py is the gate, and the counterpart to sim/run_sim.py:
that one guards the component values, this one guards the connectivity.
Same rule -- an exemption is not a pass. Every single-pin net is listed
with its reason, and a net that STOPS being single-pin fails the check
until it is removed from the list. An open item that quietly closes is
as much a drift as one that quietly opens.

  196 components, every reference unique
  113 named nets carrying two or more pins
   18 named nets reaching one pin, each a recorded open item
      GND 134 pins, 3V3_MCU 27, VBAT_PROT 12 -- all spanning the project

The root sheet carries those eighteen on the page itself, grouped by
what they wait on, so a reader does not have to run a script to find
which ends are loose.

Full set plots to docs/pdf/ECU-Schematics.pdf, 11 pages.

Two rendering bugs fixed: sheet pin names and their stu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
Parts:
- removed C1, C2: 10nF, symbol Device:C
- removed C10, C11, C12, C3, C4, C5, C6, C7, C8, C9: 100nF, symbol Device:C
- removed C13: 150uF, symbol Device:C_Polarized
- removed J1: SWD/JTAG, Connector_PinHeader_1.27mm:PinHeader_2x05_P1.27mm_Vertical, symbol Connector:Conn_ARM_JTAG_SWD_10
- removed Q1: 60V logic-level N-ch, symbol Device:Q_NMOS_GSD
- removed R1, R2: 10k, symbol Device:R
- removed R3, R4: 0R, symbol Device:R
- removed R5: 47k, symbol Device:R
- removed U1: S32K148_144LQFP, Package_QFP:LQFP-144_20x20mm_P0.5mm, symbol ecu25kva:S32K148_144LQFP
- removed U2: TPS3850G33, Package_SON:VSON-10-1EP_3x3mm_P0.5mm_EP1.2x2mm, symbol ecu25kva:TPS3850G33
- added C301, C302: 10nF, symbol Device:C
- added C303, C304, C305, C306, C307, C308, C309, C310, C311, C312: 100nF, symbol Device:C
- added C313: 150uF, symbol Device:C_Polarized
- added J301: SWD/JTAG, Connector_PinHeader_1.27mm:PinHeader_2x05_P1.27mm_Vertical, symbol Connector:Conn_ARM_JTAG_SWD_10
- added Q301: 60V logic-level N-ch, symbol Device:Q_NMOS_GSD
- added R301, R302: 10k, symbol Device:R
- added R303, R304: 0R, symbol Device:R
- added R305: 47k, symbol Device:R
- added U301: S32K148_144LQFP, Package_QFP:LQFP-144_20x20mm_P0.5mm, symbol ecu25kva:S32K148_144LQFP
- added U302: TPS3850G33, Package_SON:VSON-10-1EP_3x3mm_P0.5mm_EP1.2x2mm, symbol ecu25kva:TPS3850G33
Connections:
- net 3V3_MCU: now also C303.1, C304.1, C305.1, C306.1, C307.1, C308.1, C309.1, C310.1, C311.1, C312.1, C313.1, J301.1 (VTref), R301.1, R302.1, U301.11 (VDD), U301.124 (VDD), U301.13 (VDDA), U301.14 (VREFH), U301.32 (VDD), U301.51 (VDD), U301.67 (VDD), U301.91 (VDD), U302.1 (VDD), U302.10 (SENSE)
- net BARO: now also U301.88 (PTD18)
- net BOOST_P: now also U301.113 (PTA1)
- net BOOST_T: now also U301.104 (PTA3)
- net CAM_EDGE: now also U301.63 (PTB3)
- net CAN1_RX: now also U301.9 (PTE4)
- net CAN1_TX: now also U301.8 (PTE5)
- net CAN2_RX: now also U301.118 (PTC6)
- net CAN2_TX: now also U301.117 (PTC7)
- net COOLANT_T: now also U301.85 (PTA6)
- net CRANK_EDGE: now also U301.68 (PTB2)
- net EGR_IN1: now also U301.111 (PTB8)
- net EGR_IN2: now also U301.109 (PTB9)
- net EGR_POS: now also U301.120 (PTA15)
- net GATE_KILL: now also Q301.3 (D), R305.2
- net GND: now also C301.2, C302.2, C303.2, C304.2, C305.2, C306.2, C307.2, C308.2, C309.2, C310.2, C311.2, C312.2, C313.2, J301.3 (GND), J301.5 (GND), J301.9 (GNDDetect), Q301.2 (S), R303.2, R304.2, U301.12 (VSS), U301.123 (VSS), U301.15 (VREFL), U301.16 (VSS), U301.31 (VSS), U301.50 (VSS), U301.66 (VSS), U301.90 (VSS), U302.5 (GND)
- net INJ_HS_A: now also U301.53 (PTC0)
- net INJ_HS_B: now also U301.52 (PTC1)
- net INJ_LS_1: now also U301.43 (PTC2)
- net INJ_LS_2: now also U301.41 (PTB4)
- net INJ_LS_3: now also U301.42 (PTC3)
- net IN_AUDIO_ABORT: now also U301.48 (PTD11)
- net IN_IGNITION: now also U301.28 (PTD16)
- net IN_OVERRIDE_SS: now also U301.47 (PTD12)
- net ISNS_EGR: now also U301.99 (PTD22)
- net ISNS_INJ_A: now also U301.59 (PTC15)
- net ISNS_INJ_B: now also U301.89 (PTD19)
- net ISNS_MU: now also U301.57 (PTC16)
- net JTAG_TCK: now also J301.4 (SWCLK/TCK), U301.140 (PTC4[PD])
- net JTAG_TDI: now also J301.8 (NC/TDI), U301.139 (PTC5[PU])
- net JTAG_TMS: now also J301.2 (SWDIO/TMS), U301.142 (PTA4[PU])
- net MU_PWM: now also U301.49 (PTD10)
- net OIL_P: now also U301.83 (PTA7)
- net RAIL_P: now also U301.119 (PTA16)
- net RLY_BUZZER: now also U301.34 (PTD14)
- net RLY_MAIN: now also U301.35 (PTD13)
- net SENSOR_5V_MON: now also U301.61 (PTC14)
- net SW_COOLANT: now also U301.46 (PTD5)
- net SW_DROOP: now also U301.44 (PTD7)
- net TRIP_SENSE: now also U301.78 (PTB0)
- net VBAT_PROT: now also R305.1
- net V_BAT_1R_SNS: now also U301.115 (PTA0)
- net V_BAT_2R_SNS: now also U301.105 (PTA2)
- net WDT_FAULT: now also J301.10 (~{RESET}), Q301.1 (G), R301.2, R302.2, U301.137 (PTE1), U301.141 (PTA5[PU]), U302.8 (~WDO), U302.9 (~RESET)
- net WDT_KICK: now also U301.138 (PTE0), U302.7 (WDI)
- new net: R304.1, U302.6 (SET1)
- new net: C302.1, U302.2 (CWD)
- new net: R303.1, U302.3 (SET0)
- new net: C301.1, U302.4 (CRST)

Commit message: Correct the injector high side: a diode-OR cannot be chopped or bootstrapped
Choosing a gate driver for the high side found an error in the sheet
drawn two commits ago. The bank node was fed from VBAT_PROT through a
plain diode-OR, with the LOW side chopping for hold, on the argument
that it needed no extra MCU pin. It is wrong three ways, and only the
third is visible from a datasheet -- which is why drawing it did not
catch it and choosing a part for it did.

1. IT CANNOT REGULATE HOLD. With the battery on a diode the only switch
   in the loop is the low side, and when the low side opens the coil's
   current has nowhere to go but the recirculation diode into the 100 V
   boost rail. That is a fast decay against -87 V -- turn-off, not
   chopping. Hold needs a slow freewheel around the coil.

2. IT LEAVES CONNECTOR PINS 03 AND 05 PERMANENTLY LIVE. A diode from
   the battery to a connector pin means a harness short to ground draws
   current whenever the battery is connected, with no switch anywhere
   to stop it.

3. THE GATE DRIVER CANNOT BE BOOTSTRAPPED. A bootstrap capacitor
   charges when the switch node goes LOW. A battery diode holds that
   node at 12.8 V, so it never does, and the high side's floating supply
   can never refresh.

What replaces it is what injector_turnoff.cir already models and spends
a paragraph of its header justifying: two high-side switches per bank
onto a common node -- boost rail for the peak phase, battery for hold --
plus D_fw from GROUND to that node. Hold chopping moves to the high
side, the node swings to -0.7 V on every off-time, and the bootstrap
charges. Both switches have their SOURCE on the bank node, so one
floating supply serves two gates.

The battery switch needs a series BLOCKING diode and would with either
polarity of FET: an N-channel's body diode points source to drain, so
with the bank at 100 V during the peak phase it would dump the boost
rail into the battery. It goes on the drain side, which leaves the FET's
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
Connections:
- net INJ_HS_B_BAT: now reaches U301.92 (PTA17)
- net INJ_HS_A_BAT: now reaches U301.40 (PTB5)
Changed lines of the file:
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@@
     (effects (font (size 1.27 1.27)) (justify right))
+  )
+  (wire (pts (xy 239.52 74.19) (xy 216.66 74.19))
+    (stroke (width 0) (type default))
+  )
+  (hierarchical_label "INJ_HS_A_BAT" (shape output) (at 216.66 74.19 180)
+    (effects (font (size 1.27 1.27)) (justify right))
+  )
+  (wire (pts (xy 125.48 72.92) (xy 148.34 72.92))
+    (stroke (width 0) (type default))
+  )
+  (hierarchical_label "INJ_HS_B_BAT" (shape output) (at 148.34 72.92 0)
+    (effects (font (size 1.27 1.27)) (justify left))
   )
   (wire (pts (xy 64.52 228.19) (xy 41.66 228.19))

Commit message: Draw the EGR bridge: discrete, two AUIRS2184S, coast asserted by copper
Blocked since 20 September on one datasheet: DRV8873-Q1 had exactly the
decoded interface EGR-DRIVER asks for, and a 40 V VM absolute maximum
against a rail that reaches 73.3 V. Integrated automotive bridges cap at
40-45 V as a class. So the bridge is discrete: four 100 V N-FETs, <=20
mOhm, headroom over the 6.4 A stall.

THE DECODE COMES FROM THE DRIVER'S STRUCTURE, NOT A LOGIC GATE.
egr_hbridge.cir found that two logic lines wired to two diagonal switch
pairs short the bridge at 270 A with both asserted, and said "a per-leg
dead time is not enough on its own -- the fault here is a logic state".
AUIRS2184S has ONE input per leg: IN high puts HO on, IN low puts LO on,
with cross-conduction prevention and ~400 ns deadtime. Each leg's high
and low are exclusive by construction, so the 270 A state -- both inputs
high -- becomes a high-side brake.

Same Infineon family as the injector drivers, chosen the opposite way
for the opposite reason: the 2181's lack of interlock is what lets it
fire an injector, whose switches are in series with a coil; the 2184's
interlock is what makes a bridge leg safe.

COAST IS ASSERTED BY COPPER. egr_hbridge.cir argues coast, not brake, is
the safe state: a return spring closes the valve if the motor is let go.
Both drivers' SD-bar share EGR_SD, pulled down 10k, so with the enable
pin Hi-Z at reset both legs are off. A kill FET on the same node gives
coast on GATE_KILL with no MCU involvement. That enable costs one MCU
pin: PTB10, FTM3_CH2, same timer as EGR_IN1/IN2, PE=0/PS=0 at reset.
Pin map 41 -> 42 committed, 87 -> 86 spare.

One 20 mOhm shunt in the shared low-side return into an INA181A1-Q1
(2.56 V at a 6.4 A stall -> PTD22). It reads the drive phase; low-side
recirculation circulates between the two low FETs and misses it, so
firmware samples at the centre of the on-time -- recorded on the part.

The project netlist names the bridge nodes EGR_HIGH_59 and EGR_LO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
Connections:
- net EGR_EN: now reaches U301.108 (PTB10)
Changed lines of the file:
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@@
     (effects (font (size 1.27 1.27)) (justify left))
+  )
+  (wire (pts (xy 239.52 86.89) (xy 216.66 86.89))
+    (stroke (width 0) (type default))
+  )
+  (hierarchical_label "EGR_EN" (shape output) (at 216.66 86.89 180)
+    (effects (font (size 1.27 1.27)) (justify right))
   )
   (wire (pts (xy 64.52 228.19) (xy 41.66 228.19))
