File: hw/mcu.kicad_sch (KiCad schematic)
At the start: 24 parts, among them J301 SWD/JTAG, Q301 2N7002BK, U301 S32K148_144LQFP, U302 TPS3850G33

Commit message: Prototype review fixes: watchdog kill restored, pour checks that can fail
- D302 (BAT54Q-7-F, anode ~RESET, cathode WDT_FAULT) restores the
  watchdog-to-gate-kill path the 15 Oct supervisor fix removed; production
  and prototype. check_netlist WDO_KILL guards it. WDT_FAULT no longer
  records which trip it was; docs corrected.
- gen_board: sync stage (rename shifted refs, place new parts on a routed
  board), clusters stage, rip_thin, per-net IPC targets in widen, outer-only
  routing for nets In2 cannot carry, finish undoes a pass that necks a pour.
- Tests: pour connectivity read from pcbnew (the DRC list stops at ~500),
  test_no_necks, test_track_power_widths (TRACK_AMPS), test_inputs_committed.
- The 5 V buck's output and switch node now run on the outer layers.
- check_pcb: a parity entry with no items no longer crashes it.
- bring-up guide: probe rating, charged boost caps, 5 A limit, kill FETs.
- Decisions §15, status, handoff traps; fab files and PDF rebuilt.
Parts:
- added D302: BAT54Q-7-F, ecu25kva:SOT-23_Zener_K1_A2, symbol Device:D_Schottky
Connections:
- net WDT_FAULT: now also D302.1 (K)
- net ~{RESET}: now also D302.2 (A)
Other:
- note added: "PIN MAP ADDITIONS MADE ON THIS SHEET -- both are gaps in docs/pinmap.md, not changes to it: PTE0 WDT_KICK MCU -> TPS3850 WDI. pinmap.md assigns 37 signals and none of them services the external watchdog, but memo 11's topology requires the MCU to kick it. A window watchdog nobody feeds resets the board on a timer. PTE1 WDT_FAULT TPS3850 WDO -> MCU, a live input. D302 makes WDO pull RESET too, so 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"
- note removed: "PIN MAP ADDITIONS MADE ON THIS SHEET -- both are gaps in docs/pinmap.md, not changes to it: PTE0 WDT_KICK MCU -> TPS3850 WDI. pinmap.md assigns 37 signals and none of them services the external watchdog, but memo 11's topology requires the MCU to kick it. A window watchdog nobody feeds resets the board on a timer. PTE1 WDT_FAULT TPS3850 WDO -> MCU, so firmware can tell a watchdog trip from a rail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"
Changed lines of the file:
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@@
     (effects (font (size 1.27 1.27)) (justify left))
+  )
+  (symbol (lib_id "Device:D_Schottky") (at 178.42 370.4 0) (unit 1)
+    (in_bom yes) (on_board yes) (fields_autoplaced)
+    (property "Reference" "D302" (id 0) (at 178.42000000000002 365.32 0)
+      (effects (font (size 1.27 1.27)))
+    )
+    (property "Value" "BAT54Q-7-F" (id 1) (at 178.42000000000002 375.47999999999996 0)
+      (effects (font (size 1.27 1.27)))
+    )
+    (property "Footprint" "ecu25kva:SOT-23_Zener_K1_A2" (id 2) (at 178.42000000000002 370.4 0)
+      (effects (font (size 1.27 1.27)) hide)
+    )
+    (property "Datasheet" "~" (id 3) (at 178.42000000000002 370.4 0)
+      (effects (font (size 1.27 1.27)) hide)
+    )
+    (property "MPN" "BAT54Q-7-F" (id 4) (at 178.42000000000002 370.4 0)
+      (effects (font (size 1.27 1.27)) hide)
+    )
+    (property "Class" "30V 200mA" (id 5) (at 178.42000000000002 370.4 0)
+      (effects (font (size 1.27 1.27)) hide)
+    )
+    (property "Chosen" "Diodes Inc. BAT54Q, 30 V, 200 mA, VF 320 mV max at 1 mA, AEC-Q101, SOT-23 (DS11005 for the electrical figures)" (id 6) (at 178.42000000000002 370.4 0)
+      (effects (font (size 1.27 1.27)) hide)
+    )
+    (property "Note" "Anode ~RESET, cathode WDT_FAULT: a watchdog fault resets the MCU and kills the gates. VF <= 0.32 V at the 0.33 mA of RESET's 10k pullup, below Q301's 1.1 V minimum Vth" (id 7) (at 178.42000000000002 370.4 0)
+      (effects (font (size 1.27 1.27)) hide)
+    )
+  )
+  (wire (pts (xy 174.61 370.4) (xy 166.99 370.4))
+    (stroke (width 0) (type default))
+  )
+  (label "WDT_FAULT" (at 166.99 370.4 180)
+    (effects (font (size 1.27 1.27)) (justify right bottom))
+  )
+  (wire (pts (xy 182.23 370.4) (xy 189.85 370.4))
+    (stroke (width 0) (type default))
+  )
+  (label "~{RESET}" (at 189.85 370.4 0)
+    (effects (font (size 1.27 1.27)) (justify left bottom))
   )
   (symbol (lib_id "Device:C") (at 400.0 395.0 0) (unit 1)
@@
     (effects (font (size 1.0 1.0)) (justify left))
   )
-  (text "PIN MAP ADDITIONS MADE ON THIS SHEET -- both are gaps in docs/pinmap.md, not changes to it:\n  PTE0  WDT_KICK   MCU -> TPS3850 WDI.  pinmap.md assigns 37 signals and none of them services the external\n                   watchdog, but memo 11's topology requires the MCU to kick it. A window watchdog nobody feeds\n                   resets the board on a timer.\n  PTE1  WDT_FAULT  TPS3850 WDO -> MCU, so firmware can tell a watchdog trip from a rail trip.\nBoth are free GPIO-HD pins, PE=0/PS=0 at reset, from the 91 the pin map leaves spare." (at 40.0 132.0 0)
+  (text "PIN MAP ADDITIONS MADE ON THIS SHEET -- both are gaps in docs/pinmap.md, not changes to it:\n  PTE0  WDT_KICK   MCU -> TPS3850 WDI.  pinmap.md assigns 37 signals and none of them services the external\n                   watchdog, but memo 11's topology requires the MCU to kick it. A window watchdog nobody feeds\n                   resets the board on a timer.\n  PTE1  WDT_FAULT  TPS3850 WDO -> MCU, a live input. D302 makes WDO pull RESET too, so it reads high again\n                   once the MCU is out of reset: it does not record which trip it was.\nBoth are free GPIO-HD pins, PE=0/PS=0 at reset, from the 91 the pin map leaves spare." (at 40.0 132.0 0)
     (effects (font (size 1.6 1.6)) (justify left))
   )
