File: hw/sensors_analog.kicad_sch (KiCad schematic)
At the start: 0 parts

Commit message: Draw the analog sensor front-ends
Eight channels plus the 5V_SENSOR excitation, from battery_sense.cir,
sensor_ratiometric.cir, sensor_differential.cir and ntc_frontend.cir.
Every one ends the same way -- 22 nF and a 3.3 V zener at the MCU pin --
because every one arrives from the harness and the ADC input is what is
being protected. The front ends differ, and the split follows the
HARNESS rather than the sensor.

Boost pressure and coolant temperature share connector pin 34 as their
return; EGR position and oil pressure share pin 36; rail pressure has
pin 08 to itself. A shared return carries both sensors' current, so its
own resistance appears as an offset on both readings.
sensor_differential.cir puts 20 mA down a 1 ohm corroded return and
measures a single-ended reading wrong by the whole offset while the
differential one rejects it, a ratio of 90x. So five channels get a
difference stage and rail pressure, with its dedicated return, gets the
simpler divider.

The difference stages use 26k in and 16k feedback -- gain 16/26, the
same ratio the ratiometric divider reaches a different way. Both put a
0-5 V sensor inside VREFH; only one rejects the return's offset.

THE OP-AMPS ARE DRAWN AS FUNCTION, NOT AS A PART. KiCad ships no generic
op-amp symbol and every specific one carries a real pinout, so placing
LM324 here would assert a choice nobody has made. OPAMP_GENERIC has
placeholder pin numbers and no footprint, and the sheet says so. The
requirement is specified instead, and it is a resistor-network decision
as much as an amplifier one: sensor_differential.cir's own tolerance
note tried the argument down to 60 dB CMRR and found it still holds, so
60 dB is the floor. 0.1% discrete resistors give roughly 48 dB and do
not clear it. A matched network at 0.05% ratio, or a difference
amplifier with the network on-die, does.

Two channels are drawn with their open questions attached rather than
resolved. Boost temperature is drawn differential like its neighbours,
but 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
Parts:
- added C1, C2, C3, C4, C5, C6, C7, C8: 22nF, symbol Device:C
- added D1, D2, D3, D4, D5, D6, D7, D8: 3.3V, symbol Device:D_Zener
- added R1, R3: 120k, symbol Device:R
- added R10, R12, R14, R16, R18, R20, R22, R24, R26, R6, R8: 16k, symbol Device:R
- added R11, R13, R15, R17, R19, R21, R23, R25, R7, R9: 26k, symbol Device:R
- added R2, R4, R5: 10k, symbol Device:R
- added U1, U2, U3, U4, U5: OPAMP_GENERIC, symbol ecu25kva:OPAMP_GENERIC
Connections:
- new net: R25.2, R26.1, U5.2 (IN-)
- new net: R10.1, R9.2, U1.2 (IN-)
- new net: R11.2, R12.1, U2.3 (IN+)
- new net: R23.2, R24.1, U5.3 (IN+)
- new net: R19.2, R20.1, U4.3 (IN+)
- new net: R21.2, R22.1, U4.2 (IN-)
- new net: R13.2, R14.1, U2.2 (IN-)
- new net: R7.2, R8.1, U1.3 (IN+)
- new net: R17.2, R18.1, U3.2 (IN-)
- new net: R15.2, R16.1, U3.3 (IN+)
- new net 5V_MAIN: U1.5 (V+), U2.5 (V+), U3.5 (V+), U4.5 (V+), U5.5 (V+)
- new net BOOST_P: C4.1, D4.1 (K), R10.2, U1.1 (OUT)
- new net BOOST_P_IN: R7.1
- new net BOOST_T: C8.1, D8.1 (K), R26.2, U5.1 (OUT)
- new net BOOST_T_IN: R23.1
- new net COOLANT_T: C5.1, D5.1 (K), R14.2, U2.1 (OUT)
- new net COOLANT_T_IN: R11.1
- new net EGR_POS: C6.1, D6.1 (K), R18.2, U3.1 (OUT)
- new net EGR_POS_IN: R15.1
- new net GND: C1.2, C2.2, C3.2, C4.2, C5.2, C6.2, C7.2, C8.2, D1.2 (A), D2.2 (A), D3.2 (A), D4.2 (A), D5.2 (A), D6.2 (A), D7.2 (A), D8.2 (A), R12.2, R16.2, R2.2, R20.2, R24.2, R4.2, R6.2, R8.2, U1.4 (V-), U2.4 (V-), U3.4 (V-), U4.4 (V-), U5.4 (V-)
- new net OIL_P: C7.1, D7.1 (K), R22.2, U4.1 (OUT)
- new net OIL_P_IN: R19.1
- new net RAIL_P: C3.1, D3.1 (K), R5.2, R6.1
- new net RAIL_P_IN: R5.1
- new net SGND_34: R13.1, R25.1, R9.1
- new net SGND_36: R17.1, R21.1
- new net V_BAT_1R: R1.1
- new net V_BAT_1R_SNS: C1.1, D1.1 (K), R1.2, R2.1
- new net V_BAT_2R: R3.1
- new net V_BAT_2R_SNS: C2.1, D2.1 (K), R3.2, R4.1
Other:
- note added: "5V_SENSOR excitation -- three PTC-protected groups from the rails sheet, out to five connector pins"
- note added: "ECU pin 04 -- battery rail 1 -> PTA0 (ADC0_SE0)"
- note added: "ECU pin 06 -- battery rail 2 -> PTA2 (ADC1_SE0)"
- note added: "ECU pin 33 -- coolant temperature, return SHARED on pin 34 -> PTA6"
- note added: "ECU pin 35 -- rail pressure, DEDICATED return pin 08 -> PTA16 (ADC1_SE13)"
- note added: "ECU pin 37 -- EGR position, return SHARED on pin 36 -> PTA15"
- note added: "ECU pin 41 -- boost pressure, return SHARED on pin 34 -> PTA1"
- note added: "ECU pin 79 -- boost temperature -> PTA3. U2 OPEN: sensor type unmeasured"
- note added: "ECU pin 80 -- oil pressure, return SHARED on pin 36 -> PTA7"
- note added: "OP-AMPS: FUNCTION DRAWN, PART NOT CHOSEN. OPAMP_GENERIC has placeholder pin numbers and no footprint, deliberately -- placing a real symbol here would assert a choice nobody has made. The requirement IS specified: single 5 V supply, rail-to-rail input and output, and a difference network matched well enough for 60 dB CMRR, which is the floor sensor_differential.cir's own tolerance note tried and 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"
- note added: "WHY FIVE CHANNELS ARE DIFFERENTIAL AND ONE IS NOT. The split follows the harness, not the sensor. Boost pressure and coolant temperature SHARE connector pin 34 as their return; EGR position and oil pressure share pin 36. Rail pressure has pin 08 to itself. A shared return carries both sensors' current, so its own resistance appears as an offset on both readings -- sensor_differential.cir puts 20 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"
