File: hw/sensors_analog.kicad_sch (KiCad schematic)
At the start: 57 parts, among them U601 OPAMP_GENERIC, U602 OPAMP_GENERIC, U603 OPAMP_GENERIC, U604 OPAMP_GENERIC, U605 OPAMP_GENERIC, U606 MPXHZ6115A

Commit message: Replace the difference-amplifier placeholders with INA592 at G = 1/2
The last placeholder symbols on the board. The requirement was >=60 dB
CMRR, the floor sensor_differential.cir tried, and the drawn design --
OPAMP_GENERIC with a discrete 26k/16k network -- could not reach it:
0.1% discrete resistors give about 48 dB. The network had to be matched
on-die.

TI INA592 (SBOS914F, retrieved): native G = 1/2, CMRR 88 dB MINIMUM,
gain error 0.03% max, 4.5-36 V single supply, output within 220 mV of
each rail, common mode to 15 V at G = 1/2. Its only input absolute
maximum is 10 mA, and the ~12k internal network holds a 40 V harness
short to about 3.3 mA. G = 1/2 puts a 0.5-4.5 V sensor at 0.25-2.25 V,
straight into the ADC.

THE ARGUMENT FOR DIFFERENTIAL GOT STRONGER WITH A REAL NUMBER.
sensor_differential.cir modelled 80 dB, marked INFERRED, at gain 16/26.
It now carries the chosen part's MINIMUM 88 dB at G = 1/2, and since the
two front-ends no longer share a gain, run_sim.py compares their errors
referred to the SENSOR -- each divided by its own path gain. On a 1 ohm
corroded return, differential beats single-ended by 394x, up from 90x.

A 1k now sits between each amplifier and its ADC tail. The amplifier
runs from 5 V and can rail at 4.78 V on a harness fault; without the
resistor the 3.3 V zener at the pin takes its full short-circuit
current, with it 1.5 mA.

NOT AEC-Q100, recorded on each part. INA2132 was the dual alternative,
but its datasheet's 'G = 1/2' (Figure 12) is a single-ended attenuator;
its matched network gives only a difference G = 1, which pushes a 4.5 V
sensor past its 4 V swing on a 5 V supply. No qualified difference
amplifier with a differential G = 1/2 turned up.

Channel headings moved up so the supply labels stop crossing them.
24/24 blocks, 24/24 netlist checks.

Co-Authored-By: Claude Opus 5 <noreply@anthropic.com>
Parts:
- removed R614, R616, R618, R620, R622, R624, R626, R628: 16k, symbol Device:R
- removed R615, R617, R619, R621, R623, R625: 26k, symbol Device:R
- removed R627: 10k, symbol Device:R
- removed U601, U602, U603, U604, U605: OPAMP_GENERIC, symbol ecu25kva:OPAMP_GENERIC
- added U601, U602, U603, U604, U605: INA592, Package_SO:SOIC-8_3.9x4.9mm_P1.27mm, symbol ecu25kva:INA592
- C604, C606, C608, C610, C612: value 100nF -> 22nF; Note One per amplifier is the conservative count. Five channels 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 -> With the 16k below it, 0.35 ms -- fast against the engine a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; Source hw/check_netlist.py decoupling audit -> sensor_ratiometric.cir C1
- C605, C607, C609, C611, C613: value 22nF -> 100nF; Note With the 16k below it, 0.35 ms -- fast against the engine a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 -> At V+. Found missing on the old op-amps by check_netlist.py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; Source sensor_ratiometric.cir C1 -> (none)
- R607, R611: value 26k -> 1k; Note 26k in, 16k feedback: gain 16/26, the same ratio the ratiom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 -> Limits the pin zener to 1.5 mA if the amplifier rails at 4.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; Source sensor_differential.cir -- input leg -> (none)
- R608: value 16k -> 1k; Note (none) -> Limits the pin zener to 1.5 mA if the amplifier rails at 4.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; Source sensor_differential.cir -- IN+ leg to ground -> (none)
- R609: value 26k -> 1k; Note MATCHED to the input leg's 26k. The pair's ratio match IS t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 -> Limits the pin zener to 1.5 mA if the amplifier rails at 4.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; Source sensor_differential.cir -- return leg -> (none)
- R610: value 16k -> 1k; Note MATCHED to the IN+ leg's 16k -> Limits the pin zener to 1.5 mA if the amplifier rails at 4.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; Source sensor_differential.cir -- feedback -> (none)
- R612: value 16k -> 10k; Note (none) -> 10k/16k, the same ratio every 5 V channel on this sheet use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; Source sensor_differential.cir -- IN+ leg to ground -> (none)
- R613: value 26k -> 16k; Note MATCHED to the input leg's 26k. The pair's ratio match IS t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 -> Bottom of the divider.; Source sensor_differential.cir -- return leg -> (none)
Connections:
- net 5V_MAIN: now also C605.1, C607.1, C609.1, C611.1, C613.1, U601.7 (V+), U602.7 (V+), U603.7 (V+), U604.7 (V+), U605.7 (V+); no longer C604.1, C606.1, C608.1, C610.1, C612.1
- net BARO: now also R612.2, R613.1
- net BOOST_P: now also C604.1, R607.2; no longer C605.1, R610.2
- net BOOST_P_IN: now also U601.3 (+IN); no longer R607.1
- net BOOST_T: now also C612.1, R611.2; no longer C613.1
- net BOOST_T_IN: now also U605.3 (+IN)
- net COOLANT_T: now also C606.1, R608.2; no longer C607.1
- net COOLANT_T_IN: now also U602.3 (+IN); no longer R611.1
- net EGR_POS: now also C608.1, R609.2; no longer C609.1
- net EGR_POS_IN: now also U603.3 (+IN)
- net GND: now also R613.2, U601.1 (REF), U601.4 (V-), U602.1 (REF), U602.4 (V-), U603.1 (REF), U603.4 (V-), U604.1 (REF), U604.4 (V-), U605.1 (REF), U605.4 (V-); no longer R608.2, R612.2
- net OIL_P: now also C610.1, R610.2; no longer C611.1
- net OIL_P_IN: now also U604.3 (+IN)
- net SGND_34: now also U601.2 (-IN), U602.2 (-IN), U605.2 (-IN); no longer R609.1, R613.1
- net SGND_36: now also U603.2 (-IN), U604.2 (-IN)
- net at R608.1: now also U602.5 (SENSE), U602.6 (OUT); no longer R607.2
- net at R610.1: now also U604.5 (SENSE), U604.6 (OUT); no longer R609.2
- net at R612.1: now also U606.4 (VOUT); no longer R611.2
- new net: R611.1, U605.5 (SENSE), U605.6 (OUT)
- new net: R607.1, U601.5 (SENSE), U601.6 (OUT)
- new net: R609.1, U603.5 (SENSE), U603.6 (OUT)
Other:
- note added: "DIFFERENCE AMPLIFIERS: TI INA592 at its native G = 1/2, chosen 22 Sep 2026. The requirement was >=60 dB CMRR -- the floor sensor_differential.cir tried -- and 0.1% discrete resistors give about 48 dB, so the network had to be matched on-die: 88 dB minimum. G = 1/2 puts a 0.5-4.5 V sensor at 0.25-2.25 V; output reaches within 220 mV of each rail. A 1k before each ADC tail limits the pin zener to 1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"
- note removed: "OP-AMPS: FUNCTION DRAWN, PART NOT CHOSEN. OPAMP_GENERIC has placeholder pin numbers and no footprint, deliberately -- placing a real symbol here would assert a choice nobody has made. The requirement IS specified: single 5 V supply, rail-to-rail input and output, and a difference network matched well enough for 60 dB CMRR, which is the floor sensor_differential.cir's own tolerance note tried and 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"
