File: hw/sensors_analog.kicad_sch (KiCad schematic)
At the start: 42 parts, among them U601 INA592, U602 INA592, U603 INA592, U604 INA592, U605 INA592, U606 MPXHZ6115A

Commit message: Package every resistor and capacitor from the voltage across it
hw/assign_passives.py sizes all 188 chip R and C from a per-net table
of continuous and peak voltage (73.3 V pulse 2a, 104 V boost, bootstrap
domains riding on the bank nodes), against Vishay CRCW e3 resistor
ratings (Umax with 1.09x margin, power derated to 0.588x at a 105 C
board) and KEMET's automotive X7R waterfall (parsed by x-coordinate;
the text layout misreads its columns). schlib.place() applies the map
by ref and value; check_netlist fails on any unpackaged R or C.

Found along the way:
- 4.7 uF at 100 V is not in automotive X7R. The EMI filter C1, buck
  input and boost input are now 2 x 2.2 uF 100 V 1210; emi_filter.cir
  models the pair and its cold corner was re-pinned (0.6 dB worse).
- The twelve 470 ohm gate pulldowns need 2010: 0.31 W each at 100%
  duty. Recorded; 1k may now be possible against the real Crss.
- Local labels at 180 degrees were justified in the wrong frame on
  every sheet -- the bug fixed for hierarchical labels earlier -- so
  their text sat across their own wire. Fixed in schlib.label().

Internal nodes whose voltage matters now carry names (FB_BOOST_MID,
CAN1_SPLIT, ...); auto-names like Net-(R407-Pad2) move when parts are
added ahead of them.

24/24 sim blocks, netlist gate passing, 264 of 302 parts footprinted.
Parts:
- C601, C602, C603, C604, C605, C606, C607, C608, C609, C610, C611, C612, C613, C614, C615: footprint (none) -> Capacitor_SMD:C_0603_1608Metric
- R601, R603, R605: footprint (none) -> Resistor_SMD:R_0805_2012Metric
- R602, R604, R606, R607, R608, R609, R610, R611, R612, R613: footprint (none) -> Resistor_SMD:R_0603_1608Metric
Changed lines of the file:
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@@
       (effects (font (size 1.27 1.27)))
     )
-    (property "Footprint" "" (id 2) (at 70.0 40.0 0)
+    (property "Footprint" "Resistor_SMD:R_0805_2012Metric" (id 2) (at 70.0 40.0 0)
       (effects (font (size 1.27 1.27)) hide)
     )
@@
       (effects (font (size 1.27 1.27)))
     )
-    (property "Footprint" "" (id 2) (at 90.0 58.0 0)
+    (property "Footprint" "Resistor_SMD:R_0603_1608Metric" (id 2) (at 90.0 58.0 0)
       (effects (font (size 1.27 1.27)) hide)
     )
@@
       (effects (font (size 1.27 1.27)))
     )
-    (property "Footprint" "" (id 2) (at 106.0 58.0 0)
+    (property "Footprint" "Capacitor_SMD:C_0603_1608Metric" (id 2) (at 106.0 58.0 0)
       (effects (font (size 1.27 1.27)) hide)
     )
@@
       (effects (font (size 1.27 1.27)))
     )
-    (property "Footprint" "" (id 2) (at 70.0 95.0 0)
+    (property "Footprint" "Resistor_SMD:R_0805_2012Metric" (id 2) (at 70.0 95.0 0)
       (effects (font (size 1.27 1.27)) hide)
     )
@@
       (effects (font (size 1.27 1.27)))
     )
-    (property "Footprint" "" (id 2) (at 90.0 113.0 0)
+    (property "Footprint" "Resistor_SMD:R_0603_1608Metric" (id 2) (at 90.0 113.0 0)
       (effects (font (size 1.27 1.27)) hide)
     )
@@
       (effects (font (size 1.27 1.27)))
     )
-    (property "Footprint" "" (id 2) (at 106.0 113.0 0)
+    (property "Footprint" "Capacitor_SMD:C_0603_1608Metric" (id 2) (at 106.0 113.0 0)
       (effects (font (size 1.27 1.27)) hide)
     )
@@
       (effects (font (size 1.27 1.27)))
     )
-    (property "Footprint" "" (id 2) (at 70.0 150.0 0)
+    (property "Footprint" "Resistor_SMD:R_0805_2012Metric" (id 2) (at 70.0 150.0 0)
       (effects (font (size 1.27 1.27)) hide)
     )
@@
       (effects (font (size 1.27 1.27)))
     )
-    (property "Footprint" "" (id 2) (at 90.0 168.0 0)
+    (property "Footprint" "Resistor_SMD:R_0603_1608Metric" (id 2) (at 90.0 168.0 0)
       (effects (font (size 1.27 1.27)) hide)
     )
@@
       (effects (font (size 1.27 1.27)))
     )
-    (property "Footprint" "" (id 2) (at 106.0 168.0 0)
+    (property "Footprint" "Capacitor_SMD:C_0603_1608Metric" (id 2) (at 106.0 168.0 0)
       (effects (font (size 1.27 1.27)) hide)
     )
@@
       (effects (font (size 1.27 1.27)))
     )
-    (property "Footprint" "" (id 2) (at 427.24 42.46 0)
+    (property "Footprint" "Resistor_SMD:R_0603_1608Metric" (id 2) (at 427.24 42.46 0)
       (effects (font (size 1.27 1.27)) hide)
     )
@@
       (effects (font (size 1.27 1.27)))
     )
-    (property "Footprint" "" (id 2) (at 445.24 60.46 0)
+    (property "Footprint" "Capacitor_SMD:C_0603_1608Metric" (id 2) (at 445.24 60.46 0)
       (effects (font (size 1.27 1.27)) hide)
     )
@@
       (effects (font (size 1.27 1.27)))
     )
-    (property "Footprint" "" (id 2) (at 419.24 61.0 0)
+    (property "Footprint" "Capacitor_SMD:C_0603_1608Metric" (id 2) (at 419.24 61.0 0)
       (effects (font (size 1.27 1.27)) hide)
     )
@@
       (effects (font (size 1.27 1.27)))
     )
-    (property "Footprint" "" (id 2) (at 427.24 107.46 0)
+    (property "Footprint" "Resistor_SMD:R_0603_1608Metric" (id 2) (at 427.24 107.46 0)
       (effects (font (size 1.27 1.27)) hide)
     )
@@
       (effects (font (size 1.27 1.27)))
     )
-    (property "Footprint" "" (id 2) (at 445.24 125.46 0)
+    (property "Footprint" "Capacitor_SMD:C_0603_1608Metric" (id 2) (at 445.24 125.46 0)
       (effects (font (size 1.27 1.27)) hide)
     )
@@
       (effects (font (size 1.27 1.27)))
     )
-    (property "Footprint" "" (id 2) (at 419.24 126.0 0)
+    (property "Footprint" "Capacitor_SMD:C_0603_1608Metric" (id 2) (at 419.24 126.0 0)
       (effects (font (size 1.27 1.27)) hide)
     )
@@
       (effects (font (size 1.27 1.27)))
     )
-    (property "Footprint" "" (id 2) (at 427.24 172.46 0)
+    (property "Footprint" "Resistor_SMD:R_0603_1608Metric" (id 2) (at 427.24 172.46 0)
       (effects (font (size 1.27 1.27)) hide)
     )
@@
       (effects (font (size 1.27 1.27)))
     )
-    (property "Footprint" "" (id 2) (at 445.24 190.46 0)
+    (property "Footprint" "Capacitor_SMD:C_0603_1608Metric" (id 2) (at 445.24 190.46 0)
       (effects (font (size 1.27 1.27)) hide)
     )
@@
       (effects (font (size 1.27 1.27)))
     )
-    (property "Footprint" "" (id 2) (at 419.24 191.0 0)
+    (property "Footprint" "Capacitor_SMD:C_0603_1608Metric" (id 2) (at 419.24 191.0 0)
       (effects (font (size 1.27 1.27)) hide)
     )
@@
       (effects (font (size 1.27 1.27)))
     )
-    (property "Footprint" "" (id 2) (at 427.24 237.46 0)
+    (property "Footprint" "Resistor_SMD:R_0603_1608Metric" (id 2) (at 427.24 237.46 0)
       (effects (font (size 1.27 1.27)) hide)
     )
@@
       (effects (font (size 1.27 1.27)))
     )
-    (property "Footprint" "" (id 2) (at 445.24 255.46 0)
+    (property "Footprint" "Capacitor_SMD:C_0603_1608Metric" (id 2) (at 445.24 255.46 0)
       (effects (font (size 1.27 1.27)) hide)
     )
@@
       (effects (font (size 1.27 1.27)))
     )
-    (property "Footprint" "" (id 2) (at 419.24 256.0 0)
+    (property "Footprint" "Capacitor_SMD:C_0603_1608Metric" (id 2) (at 419.24 256.0 0)
       (effects (font (size 1.27 1.27)) hide)
     )
@@
       (effects (font (size 1.27 1.27)))
     )
-    (property "Footprint" "" (id 2) (at 137.24 225.46 0)
+    (property "Footprint" "Resistor_SMD:R_0603_1608Metric" (id 2) (at 137.24 225.46 0)
       (effects (font (size 1.27 1.27)) hide)
     )
@@
       (effects (font (size 1.27 1.27)))
     )
-    (property "Footprint" "" (id 2) (at 155.24 243.46 0)
+    (property "Footprint" "Capacitor_SMD:C_0603_1608Metric" (id 2) (at 155.24 243.46 0)
       (effects (font (size 1.27 1.27)) hide)
     )
@@
       (effects (font (size 1.27 1.27)))
     )
-    (property "Footprint" "" (id 2) (at 129.24 244.0 0)
+    (property "Footprint" "Capacitor_SMD:C_0603_1608Metric" (id 2) (at 129.24 244.0 0)
       (effects (font (size 1.27 1.27)) hide)
     )
@@
       (effects (font (size 1.27 1.27)))
     )
-    (property "Footprint" "" (id 2) (at 170.0 86.0 0)
+    (property "Footprint" "Capacitor_SMD:C_0603_1608Metric" (id 2) (at 170.0 86.0 0)
       (effects (font (size 1.27 1.27)) hide)
     )
@@
       (effects (font (size 1.27 1.27)))
     )
-    (property "Footprint" "" (id 2) (at 223.24 94.92 0)
+    (property "Footprint" "Resistor_SMD:R_0603_1608Metric" (id 2) (at 223.24 94.92 0)
       (effects (font (size 1.27 1.27)) hide)
     )
@@
       (effects (font (size 1.27 1.27)))
     )
-    (property "Footprint" "" (id 2) (at 243.24 112.92 0)
+    (property "Footprint" "Resistor_SMD:R_0603_1608Metric" (id 2) (at 243.24 112.92 0)
       (effects (font (size 1.27 1.27)) hide)
     )
@@
       (effects (font (size 1.27 1.27)))
     )
-    (property "Footprint" "" (id 2) (at 261.24 112.92 0)
-      (effects (font (size 1.27 1.27)) hide)
-    )
+    (property "Footprint" "Capacitor_SMD:C_0603_1608Metric" (id 2) (at 261.24 112.92 0)
+      (effects (font (size 1.27 1.27)) hide)
+    )

Commit message: Replace the analog-input zeners with BAV199-Q rail clamps
LOWV-CLAMP, analog half. The ten 3.3 V zeners on the sensor and cam
inputs leaked at signal level (the datasheet allows 5 uA at 1 V); they
are now BAV199-Q (80 nA max at 150 C, AEC-Q101) to 3V3_MCU and ground,
drawn as one 3-pin part so each pair is one package. The speed input's
split BAV199 halves and the power-input sense clamp use the same part.

A rail clamp needs something the zener did not: the BAV199's upper
diode is high-Vf, so on a 40 V harness short the MCU pad's ESD diode
would take most of the fault current, over the +/-3 mA injection
limit. Each clamped channel now has 1k between clamp and pad: 0.40 mA
injected. sensor_ratiometric and cam_frontend model the pair, the 1k
and the pad diode, and check the injection current.

The new models also showed the old zener loading the cam signal by
84 mV at a 5.25 V rail -- pinned by the old check as the expected
value. Re-pinned to the divider's own 3.231 V.

The discrete inputs stay open: they clamp continuously, which neither
a rail clamp nor an LM4040-class reference (35 uA bias below
breakdown) can do within the pin's ratings.

24/24 sim blocks, netlist gate passing, 197 R/C packaged.
Parts:
- removed D601, D602, D603, D604, D605, D606, D607, D608: 3.3V, symbol Device:D_Zener
- added D601, D602, D603, D604, D605, D606, D607, D608: BAV199-Q, Package_TO_SOT_SMD:SOT-23, symbol ecu25kva:BAV199
- added R614, R615, R616, R617, R618, R619: 1k, Resistor_SMD:R_0603_1608Metric, symbol Device:R
- added R620: 10k, Resistor_SMD:R_0603_1608Metric, symbol Device:R
- added R621: 16k, Resistor_SMD:R_0603_1608Metric, symbol Device:R
- R603: value 120k -> 1k; footprint Resistor_SMD:R_0805_2012Metric -> Resistor_SMD:R_0603_1608Metric; Note 120k/10k puts 40 V at 3.077 V, inside VREFH. The 75k/10k ve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 -> Pad injection on a 40 V short: 0.4 mA, against the S32K148'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; Source battery_sense.cir R3/R4 -> sensor_ratiometric.cir Rpc -- LOWV-CLAMP
- R604: value 10k -> 120k; footprint Resistor_SMD:R_0603_1608Metric -> Resistor_SMD:R_0805_2012Metric; Note (none) -> 120k/10k puts 40 V at 3.077 V, inside VREFH. The 75k/10k ve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
- R605: footprint Resistor_SMD:R_0805_2012Metric -> Resistor_SMD:R_0603_1608Metric; Note 10k/16k scales 0-5 V to 0-3.077 V. Firmware divides out the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 -> (none); Source sensor_ratiometric.cir R1 -> battery_sense.cir R3/R4
- R606: value 16k -> 1k; Note (none) -> Pad injection on a 40 V short: 0.4 mA, against the S32K148'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; Source sensor_ratiometric.cir R2 -> sensor_ratiometric.cir Rpc -- LOWV-CLAMP
- R607: value 1k -> 10k; footprint Resistor_SMD:R_0603_1608Metric -> Resistor_SMD:R_0805_2012Metric; Note Limits the pin zener to 1.5 mA if the amplifier rails at 4.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 -> 10k/16k scales 0-5 V to 0-3.077 V. Firmware divides out the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; Source (none) -> sensor_ratiometric.cir R1
- R608: value 1k -> 16k; Note Limits the pin zener to 1.5 mA if the amplifier rails at 4.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 -> (none); Source (none) -> sensor_ratiometric.cir R2
- R609, R611: Note Limits the pin zener to 1.5 mA if the amplifier rails at 4.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 -> Pad injection on a 40 V short: 0.4 mA, against the S32K148'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; Source (none) -> sensor_ratiometric.cir Rpc -- LOWV-CLAMP
- R612: value 10k -> 1k; Note 10k/16k, the same ratio every 5 V channel on this sheet use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 -> Limits the pin zener to 1.5 mA if the amplifier rails at 4.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
- R613: value 16k -> 1k; Note Bottom of the divider. -> Pad injection on a 40 V short: 0.4 mA, against the S32K148'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; Source (none) -> sensor_ratiometric.cir Rpc -- LOWV-CLAMP
Connections:
- net BARO: now also R620.2, R621.1; no longer R612.2, R613.1
- net BOOST_P: now also R611.2; no longer C604.1, R607.2
- net BOOST_T: now also R619.2; no longer C612.1, R611.2
- net COOLANT_T: now also R613.2; no longer C606.1, R608.2
- net EGR_POS: now also R615.2; no longer C608.1, R609.2
- net GND: now also R605.2, R608.2, D601.1 (A1), D602.1 (A1), D603.1 (A1), D604.1 (A1), D605.1 (A1), D606.1 (A1), D607.1 (A1), D608.1 (A1), R621.2; no longer R604.2, R606.2, R613.2
- net OIL_P: now also R617.2; no longer C610.1, R610.2
- net RAIL_P: now also R609.2; no longer C603.1, R605.2, R606.1
- net RAIL_P_IN: now also R607.1; no longer R605.1
- net V_BAT_1R_SNS: now also R603.2; no longer C601.1, R601.2, R602.1
- net V_BAT_2R: now also R604.1; no longer R603.1
- net V_BAT_2R_SNS: now also R606.2; no longer C602.1, R603.2, R604.1
- net at U603.5 (SENSE), U603.6 (OUT): now also R614.1; no longer R609.1
- net at U604.5 (SENSE), U604.6 (OUT): now also R616.1; no longer R610.1
- net at R612.1: now also U602.5 (SENSE), U602.6 (OUT); no longer U606.4 (VOUT)
- net at U601.5 (SENSE), U601.6 (OUT): now also R610.1; no longer R607.1
- net at U605.5 (SENSE), U605.6 (OUT): now also R618.1; no longer R611.1
- new net: R620.1, U606.4 (VOUT)
- new net 3V3_MCU: D601.2 (K2), D602.2 (K2), D603.2 (K2), D604.2 (K2), D605.2 (K2), D606.2 (K2), D607.2 (K2), D608.2 (K2)
- new net BOOST_P_CL: C604.1, D604.3 (COM), R610.2, R611.1
- new net BOOST_T_CL: C612.1, D608.3 (COM), R618.2, R619.1
- new net COOLANT_T_CL: C606.1, D605.3 (COM), R612.2, R613.1
- new net EGR_POS_CL: C608.1, D606.3 (COM), R614.2, R615.1
- new net OIL_P_CL: C610.1, D607.3 (COM), R616.2, R617.1
- new net RAIL_P_CL: C603.1, D603.3 (COM), R607.2, R608.1, R609.1
- new net V_BAT_1R_SNS_CL: C601.1, D601.3 (COM), R601.2, R602.1, R603.1
- new net V_BAT_2R_SNS_CL: C602.1, D602.3 (COM), R604.2, R605.1, R606.1
