File: hw/connector.kicad_sch (KiCad schematic)
At the start: 0 parts

Commit message: Draw the connector; the power ground turns out to have no pin
Sheet 10 of 10. Not a circuit -- the harness boundary, and its job is to
be checkable against the machine: every pin the wiring diagram shows
wired to the net whichever sheet owns that signal already named, and
every pin it does not show left visibly empty.

41 of 94 pins wired, 53 left empty, every pin accounted for exactly once
in the netlist.

THE FINDING. GP3.8703.C4.pdf shows pin 21 as the battery positive feed
and shows no battery negative anywhere on the ECU connector. That is a
gap in the source rather than a contradiction in it -- the document is a
field troubleshooting diagram and its own scope note says it omits
"power grounds, unused pins and internal-only pins". It is still a gap
that stops a board: every other sheet in this project returns to GND,
the injector low sides carry 18 A into it, and at this boundary that net
has nowhere to go. It cannot be closed by choosing. Fifty pins have no
established function and several are certainly grounds -- a 94-way
connector feeding an 18 A injector stage does not have one return -- but
a wrong ground pin is not a rework, it is a harness that has to be
remade. Same for TRIP_LOOP, which is a NEW signal not on the OEM diagram
at all and needs one of the same fifty.

CONN_ECU_94 carries pin count and pin numbers, which are facts read off
page 4, and no footprint, because no part number is known. Pin names are
the diagram's own signal names where it shows the pin and blank where it
does not. Same treatment the op-amps and the comparator get.

Two distinctions the sheet makes explicit: pins 34 and 36 are SHARED
sensor returns and therefore signals, carried into difference amplifiers
on sensors_analog; pin 08 is rail pressure's dedicated return, with
nothing to reject, so it is simply ground here.

CROSS-SHEET AUDIT. 83 hierarchical net names across the ten sheets, 73
appearing on two or more. All ten that appear on only one sheet are
explained by an open it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
Parts:
- added J1: CONN_ECU_94, symbol ecu25kva:CONN_ECU_94
Connections:
- new net BOOST_P_IN: J1.41 (BOOST_P)
- new net BOOST_T_IN: J1.79 (BOOST_T)
- new net CAM_FREQ_46: J1.46 (CAM_FREQ)
- new net CAM_GND_44: J1.44 (SGND_CAM)
- new net CAN1_H: J1.55 (CAN1_H)
- new net CAN1_L: J1.77 (CAN1_L)
- new net CAN2_H: J1.87 (CAN2_H)
- new net CAN2_L: J1.86 (CAN2_L)
- new net COOLANT_T_IN: J1.33 (COOLANT_T)
- new net CRANK_HI_52: J1.52 (CRANK_HI)
- new net CRANK_LO_74: J1.74 (CRANK_LO)
- new net EGR_HIGH_59: J1.59 (EGR_HIGH)
- new net EGR_LOW_81: J1.81 (EGR_LOW)
- new net EGR_POS_IN: J1.37 (EGR_POS)
- new net EXC_BOOST_11: J1.11 (EXC_BOOST)
- new net EXC_CAM_45: J1.45 (EXC_CAM)
- new net EXC_EGR_15: J1.15 (EXC_EGR)
- new net EXC_OIL_39: J1.39 (EXC_OIL)
- new net EXC_RAIL_32: J1.32 (EXC_RAIL)
- new net GND: J1.8 (SGND_RAIL)
- new net INJ_A_03: J1.3 (INJ_HS_A)
- new net INJ_B_05: J1.5 (INJ_HS_B)
- new net INJ_LS1_73: J1.73 (INJ_LS_CYL1)
- new net INJ_LS2_29: J1.29 (INJ_LS_CYL2)
- new net INJ_LS3_07: J1.7 (INJ_LS_CYL3)
- new net IN_AUDIO_ABORT_H: J1.20 (AUDIO_ABORT)
- new net IN_IGNITION_H: J1.71 (IGNITION)
- new net IN_OVERRIDE_SS_H: J1.24 (OVERRIDE_SS)
- new net MU_RETURN: J1.88 (MU_PWM)
- new net OIL_P_IN: J1.80 (OIL_P)
- new net RAIL_P_IN: J1.35 (RAIL_P)
- new net RLY_BUZZER_OUT: J1.69 (BUZZER_RELAY)
- new net RLY_MAIN_OUT: J1.50 (MAIN_RELAY)
- new net SGND_34: J1.34 (SGND_BOOST_COOLANT)
- new net SGND_36: J1.36 (SGND_EGR_OIL)
- new net SHIELD_30: J1.30 (SGND_CRANK)
- new net SW_COOLANT_C: J1.43 (SW_COOLANT)
- new net SW_DROOP_C: J1.23 (SW_DROOP)
- new net VBAT_IN: J1.21 (BATT_PLUS)
- new net V_BAT_1R: J1.4 (V_BAT_1R)
- new net V_BAT_2R: J1.6 (V_BAT_2R)
Other:
- note added: "41 pins wired, 53 left deliberately empty"
- note added: "J1 -- 94-way ECU harness connector"
- note added: "NO PART NUMBER, SO NO FOOTPRINT. The reference records a 94-pin connector from GP3.8703.C4.pdf page 4 and nothing further -- no Bosch part number, no keying, no mating half. CONN_ECU_94 therefore carries pin COUNT and pin NUMBERS, which are facts read off a document, and no footprint, which would be a guess about a physical interface that has to mate with a harness already on a machine. Pin NAMES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"
- note added: "PINS SHOWN ON THE DIAGRAM AND STILL NOT WIRED 09 SYNCHRONIZATION GROUND. Drawn RED on a diagram whose own legend makes red a positive feed, so the name and the colour disagree. U6 on the unknowns register. 01 G_G_B AT1. 02 G_G_B AT2. Memo 03 suspects these are power grounds rather than switch-return legs. If that is right they are part of the answer to the note on the left. No MCU pin is assigned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"
- note added: "THE POWER GROUND HAS NO PIN, AND THAT IS THIS SHEET'S FINDING. GP3.8703.C4.pdf shows pin 21 as the battery positive feed and shows no battery negative anywhere on the ECU connector. Its own scope note explains why -- it is a field troubleshooting diagram and it omits "power grounds, unused pins and internal-only pins" -- so this is a gap in the SOURCE, not a contradiction in it. It is still a gap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"
- title: 94-way Bosch connector and harness mapping -> 94-way ECU connector and harness mapping

Commit message: Wire the root sheet: the project has a netlist for the first time
Ten sheets each passed their own netlist and the project had none. The
root sheet's ten sheet symbols carried NO hierarchical pins, so a net
name appearing on two sheets was two nets and nothing compared them --
the cross-sheet audit in the last commit was a name comparison, not a
connectivity check.

Each symbol now carries one pin per net its child exports, read OUT of
the child rather than declared in a second list that could drift: 162
pins across the ten, each with a stub and a label. Two labels with the
same name are one net, which is how 162 pins connect without routing
162 wires across a page nobody could read.

Exporting it found the other half of the same problem immediately.
kicad-cli reported annotation errors: every sheet generator allocated
R1, C1, U1 from its own counter, so ten sheets had ten parts called R1.
schlib.REF_BASE gives each sheet its own hundred -- KiCad's own
sheet-number x 100 convention, applied at generation time instead of by
a hand pass in Eeschema. 196 components, no duplicate reference.

hw/check_netlist.py is the gate, and the counterpart to sim/run_sim.py:
that one guards the component values, this one guards the connectivity.
Same rule -- an exemption is not a pass. Every single-pin net is listed
with its reason, and a net that STOPS being single-pin fails the check
until it is removed from the list. An open item that quietly closes is
as much a drift as one that quietly opens.

  196 components, every reference unique
  113 named nets carrying two or more pins
   18 named nets reaching one pin, each a recorded open item
      GND 134 pins, 3V3_MCU 27, VBAT_PROT 12 -- all spanning the project

The root sheet carries those eighteen on the page itself, grouped by
what they wait on, so a reader does not have to run a script to find
which ends are loose.

Full set plots to docs/pdf/ECU-Schematics.pdf, 11 pages.

Two rendering bugs fixed: sheet pin names and their stu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
Parts:
- removed J1: CONN_ECU_94, symbol ecu25kva:CONN_ECU_94
- added J1001: CONN_ECU_94, symbol ecu25kva:CONN_ECU_94
Connections:
- net BOOST_P_IN: now also J1001.41 (BOOST_P)
- net BOOST_T_IN: now also J1001.79 (BOOST_T)
- net CAM_FREQ_46: now also J1001.46 (CAM_FREQ)
- net CAM_GND_44: now also J1001.44 (SGND_CAM)
- net CAN1_H: now also J1001.55 (CAN1_H)
- net CAN1_L: now also J1001.77 (CAN1_L)
- net CAN2_H: now also J1001.87 (CAN2_H)
- net CAN2_L: now also J1001.86 (CAN2_L)
- net COOLANT_T_IN: now also J1001.33 (COOLANT_T)
- net CRANK_HI_52: now also J1001.52 (CRANK_HI)
- net CRANK_LO_74: now also J1001.74 (CRANK_LO)
- net EGR_HIGH_59: now also J1001.59 (EGR_HIGH)
- net EGR_LOW_81: now also J1001.81 (EGR_LOW)
- net EGR_POS_IN: now also J1001.37 (EGR_POS)
- net EXC_BOOST_11: now also J1001.11 (EXC_BOOST)
- net EXC_CAM_45: now also J1001.45 (EXC_CAM)
- net EXC_EGR_15: now also J1001.15 (EXC_EGR)
- net EXC_OIL_39: now also J1001.39 (EXC_OIL)
- net EXC_RAIL_32: now also J1001.32 (EXC_RAIL)
- net GND: now also J1001.8 (SGND_RAIL)
- net INJ_A_03: now also J1001.3 (INJ_HS_A)
- net INJ_B_05: now also J1001.5 (INJ_HS_B)
- net INJ_LS1_73: now also J1001.73 (INJ_LS_CYL1)
- net INJ_LS2_29: now also J1001.29 (INJ_LS_CYL2)
- net INJ_LS3_07: now also J1001.7 (INJ_LS_CYL3)
- net IN_AUDIO_ABORT_H: now also J1001.20 (AUDIO_ABORT)
- net IN_IGNITION_H: now also J1001.71 (IGNITION)
- net IN_OVERRIDE_SS_H: now also J1001.24 (OVERRIDE_SS)
- net MU_RETURN: now also J1001.88 (MU_PWM)
- net OIL_P_IN: now also J1001.80 (OIL_P)
- net RAIL_P_IN: now also J1001.35 (RAIL_P)
- net RLY_BUZZER_OUT: now also J1001.69 (BUZZER_RELAY)
- net RLY_MAIN_OUT: now also J1001.50 (MAIN_RELAY)
- net SGND_34: now also J1001.34 (SGND_BOOST_COOLANT)
- net SGND_36: now also J1001.36 (SGND_EGR_OIL)
- net SHIELD_30: now also J1001.30 (SGND_CRANK)
- net SW_COOLANT_C: now also J1001.43 (SW_COOLANT)
- net SW_DROOP_C: now also J1001.23 (SW_DROOP)
- net VBAT_IN: now also J1001.21 (BATT_PLUS)
- net V_BAT_1R: now also J1001.4 (V_BAT_1R)
- net V_BAT_2R: now also J1001.6 (V_BAT_2R)
Changed lines of the file:
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@@
   (symbol (lib_id "ecu25kva:CONN_ECU_94") (at 297.0 200.0 0) (unit 1)
     (in_bom yes) (on_board yes) (fields_autoplaced)
-    (property "Reference" "J1" (id 0) (at 297.0 194.92 0)
+    (property "Reference" "J1001" (id 0) (at 297.0 194.92 0)
       (effects (font (size 1.27 1.27)))
     )
@@
   (symbol (lib_id "power:GND") (at 204.9 125.36 0) (unit 1)
     (in_bom yes) (on_board yes) (fields_autoplaced)
-    (property "Reference" "#PWR1" (id 0) (at 204.89999999999998 120.28000000000002 0)
+    (property "Reference" "#PWR1001" (id 0) (at 204.89999999999998 120.28000000000002 0)
       (effects (font (size 1.27 1.27)) hide)
     )

Commit message: Correct the connector sheet: the part number was in the repo
hw/connector.kicad_sch said no Bosch part number was known. The repo has
had it since 18 September. refs/field-evidence-2026-09-18.md sec.2b
closed U1 off a photograph of the housing angled to the light:

  BOSCH + armature-in-circle logo   moulded on the side body
  1 928 405 194                     under the BOSCH text
  1 928 405 192                     strip along the lower body
  code C                            beside it -- MECHANICAL coding
  >PA66-GF50<                       on the locking lever

Read off the physical part, which beats a catalogue match because it
cannot be a mis-identification. Bosch 94-way ECU connector, EDC17 family.

Code C is load-bearing rather than trivia: Bosch supplies these housings
in mechanically coded variants so differently-coded plugs cannot mate,
so any replacement or adapter must match it or it will not engage -- the
kind of detail that is invisible until a part arrives and will not fit.

Still missing, and the sheet now says which is which: the OEM PIN LIST,
a different document from the part number, and the board-side land
pattern. Neither number returns a catalogue hit, so the footprint has to
come through a Bosch distributor quoting them. None is assigned, because
a mating land pattern is not a thing to infer from a photograph.

Same shape as the six findings this project has already turned up -- a
document and a file disagreeing with nothing comparing them -- and this
one was mine. The sheet was drawn from refs/ecu-pinout-extracted.md,
which predates the field visit and still says a complete pinout needs
the connector part number, and I did not read the newer file beside it.

Co-Authored-By: Claude Opus 5 <noreply@anthropic.com>
Parts:
- J1001: FootprintStatus (none) -> not assigned: the board-side land pattern needs the mating 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; MPN (none) -> Bosch 1 928 405 192 / 194, CODE C; Note 94-way. Part number unknown, so no footprint is assigned --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 -> Bosch 94-way ECU connector, EDC17 family, PA66-GF50 housing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; Source refs/ecu-pinout-extracted.md, from GP3.8703.C4.pdf page 4 -> refs/ecu-pinout-extracted.md (pin count and 44 functions); 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
Other:
- note added: "THE PART IS IDENTIFIED; THE LAND PATTERN IS NOT. refs/field-evidence-2026-09-18.md sec.2b closed U1 off a photograph of the housing angled to the light: BOSCH and the armature-in-circle logo moulded on the side body, 1 928 405 194 under the BOSCH text, 1 928 405 192 on the lower body strip, CODE C beside it, >PA66-GF50< on the locking lever. Read off the physical part, which beats a catalogue mat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"
- note removed: "NO PART NUMBER, SO NO FOOTPRINT. The reference records a 94-pin connector from GP3.8703.C4.pdf page 4 and nothing further -- no Bosch part number, no keying, no mating half. CONN_ECU_94 therefore carries pin COUNT and pin NUMBERS, which are facts read off a document, and no footprint, which would be a guess about a physical interface that has to mate with a harness already on a machine. Pin NAMES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"
Changed lines of the file:
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@@
     (comment 2 "Pin count and 44 pin functions from GP3.8703.C4.pdf via refs/ecu-pinout-extracted.md")
     (comment 3 "50 pins have no established function -- including, so far, the power ground")
-    (comment 4 "No part number and no footprint: neither is known")
+    (comment 4 "Bosch 1 928 405 192 / 194 code C -- part identified off the housing; land pattern is not")
   )
   (symbol (lib_id "ecu25kva:CONN_ECU_94") (at 297.0 200.0 0) (unit 1)
@@
       (effects (font (size 1.27 1.27)) hide)
     )
-    (property "Source" "refs/ecu-pinout-extracted.md, from GP3.8703.C4.pdf page 4" (id 4) (at 297.0 200.0 0)
-      (effects (font (size 1.27 1.27)) hide)
-    )
-    (property "Note" "94-way. Part number unknown, so no footprint is assigned -- see the sheet note." (id 5) (at 297.0 200.0 0)
-      (effects (font (size 1.27 1.27)) hide)
-    )
-    (property "Shown" "44 of 94 pins appear on the wiring diagram" (id 6) (at 297.0 200.0 0)
+    (property "Source" "refs/ecu-pinout-extracted.md (pin count and 44 functions); refs/field-evidence-2026-09-18.md sec.2b (part numbers, off the housing)" (id 4) (at 297.0 200.0 0)
+      (effects (font (size 1.27 1.27)) hide)
+    )
+    (property "MPN" "Bosch 1 928 405 192 / 194, CODE C" (id 5) (at 297.0 200.0 0)
+      (effects (font (size 1.27 1.27)) hide)
+    )
+    (property "Note" "Bosch 94-way ECU connector, EDC17 family, PA66-GF50 housing. Code C is a MECHANICAL coding variant -- a differently-coded housing will not mate." (id 6) (at 297.0 200.0 0)
+      (effects (font (size 1.27 1.27)) hide)
+    )
+    (property "FootprintStatus" "not assigned: the board-side land pattern needs the mating half's drawing, via a Bosch distributor. No catalogue hit on either number." (id 7) (at 297.0 200.0 0)
+      (effects (font (size 1.27 1.27)) hide)
+    )
+    (property "Shown" "44 of 94 pins appear on the wiring diagram" (id 8) (at 297.0 200.0 0)
       (effects (font (size 1.27 1.27)) hide)
     )
@@
     (effects (font (size 1.6 1.6)) (justify left))
   )
-  (text "NO PART NUMBER, SO NO FOOTPRINT. The reference records a 94-pin connector from GP3.8703.C4.pdf page 4 and nothing further -- no Bosch part number, no keying, no mating half. CONN_ECU_94 therefore carries pin COUNT and pin NUMBERS, which are facts read off a document, and\nno footprint, which would be a guess about a physical interface that has to mate with a harness already on a machine. Pin NAMES on the symbol are the diagram's own signal names where it shows the pin, and KiCad's blank elsewhere. This is the same treatment the op-amps on\nsensors_analog and the comparator on speed_inputs get, for the same reason: the symbol asserts what is known and declines to assert what is not." (at 14.0 390.0 0)
+  (text "THE PART IS IDENTIFIED; THE LAND PATTERN IS NOT. refs/field-evidence-2026-09-18.md sec.2b closed U1 off a photograph of the housing angled to the light: BOSCH and the armature-in-circle logo moulded on the side body, 1 928 405 194 under the BOSCH text, 1 928 405 192 on the lower\nbody strip, CODE C beside it, >PA66-GF50< on the locking lever. Read off the physical part, which beats a catalogue match because it cannot be a mis-identification. CODE C IS LOAD-BEARING: Bosch supplies these housings mechanically coded\nso differently-coded plugs cannot mate, so any replacement or adapter must match it or it will not engage -- the kind of detail that is invisible until a part arrives and will not fit. Still missing: the OEM PIN LIST, a different document\nfrom the part number, and the board-side footprint. A search for both numbers returned no catalogue hit, so the land pattern has to come through a Bosch distributor quoting them. Nothing is assigned here, because a mating land pattern is\nnot a thing to infer from a photograph. Pin NAMES on the symbol are the wiring diagram's own signal names where it shows the pin and KiCad's blank elsewhere -- the same treatment the op-amps and the comparator get: the symbol\nasserts what is known and declines to assert what is not." (at 14.0 390.0 0)
     (effects (font (size 1.6 1.6)) (justify left))
   )
