File: hw/injector.kicad_sch (KiCad schematic)
At the start: 0 parts

Commit message: Draw the injector stage, and give the boost reservoir the bleed it was missing
Sheet 9 of 10.

TWO WIRING QUESTIONS THE BLOCKS LEFT OPEN, settled here because a
netlist is where wiring gets decided.

Where the hold current comes from. boost_converter.cir measured that
supplying hold from the boost rail costs 28x the peak phase's charge
and collapses the rail, so hold comes from the battery -- but not
through what. It is a DIODE-OR: anode on VBAT_PROT, cathode on the bank
node. Reverse biased while the bank sits near 100 V; supplies 13.5 V
once the high-side FET stops conducting. One control pin per bank, no
sequencing, no extra MCU pin. It also does the job injector_turnoff.cir
had to invent D_fw for, at 13.5 V instead of 0 V -- so the turn-off
clamp is 86.5 V rather than the bare 100 V that block modelled, and
turn-off takes about 41.6 us instead of 34 us.

Where the current-sense shunts go. pinmap 1.6 called the per-bank split
INFERRED and said outright: settle it when the sheet is drawn. Settled
low-side and ground-referenced, one per bank. Cylinders 1 and 3 fire 240
crank degrees apart and never overlap, so one shunt in their shared
source return is unambiguous -- the same fact that lets the high side be
bank-shared -- and it reads the same current a high-side shunt would
without needing an amplifier whose common-mode range reaches 100 V.

NEW FINDING. Spec sec.4's fail-safe list names pins 03/05 alongside the
four low-side gates. supervisor.cir sized a ground-referenced clamp for
them and pinmap sec.2 confirmed all six pins' reset state against NXP's
own table. All three agree, and all three are silent on the source of a
high-side N-FET swinging to the boost rail: a pulldown to ground would
hold Vgs at minus the source voltage and fight the driver on every edge,
and a kill FET referenced to ground cannot short a gate floating 100 V
up. The 470 ohm goes across gate and SOURCE, and the kill path moves
into the driver's shutdown input.

THE BLEED PATH injector_tur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
Parts:
- added C1: 47uF 150V, symbol Device:C_Polarized
- added D1, D2, D3, D4, D5: 150V 20A ultrafast, symbol Device:D
- added Q1, Q2: 150V N-ch, bootstrapped high side, symbol Device:Q_NMOS_GSD
- added Q3, Q5, Q7: 150V N-ch, 18A peak, symbol Device:Q_NMOS_GSD
- added Q4, Q6, Q8: 60V small-signal, symbol Device:Q_NMOS_GSD
- added R1: 22k 1W, symbol Device:R
- added R2, R3, R4, R5, R6: 470R, symbol Device:R
- added R7, R8: 5mOhm 2W 1%, symbol Device:R
Connections:
- new net BOOST_100V: C1.1, D3.1 (K), D4.1 (K), D5.1 (K), Q1.3 (D), Q2.3 (D), R1.1
- new net GATE_KILL: Q4.1 (G), Q6.1 (G), Q8.1 (G)
- new net GND: C1.2, Q4.2 (S), Q6.2 (S), Q8.2 (S), R1.2, R4.2, R5.2, R6.2, R7.2, R8.2
- new net HSA_GATE: Q1.1 (G), R2.1
- new net HSB_GATE: Q2.1 (G), R3.1
- new net INJ_A_03: D1.1 (K), Q1.2 (S), R2.2
- new net INJ_B_05: D2.1 (K), Q2.2 (S), R3.2
- new net INJ_LS1_73: D3.2 (A), Q3.3 (D)
- new net INJ_LS2_29: D5.2 (A), Q7.3 (D)
- new net INJ_LS3_07: D4.2 (A), Q5.3 (D)
- new net ISNS_INJ_A_SENSE: Q3.2 (S), Q5.2 (S), R7.1
- new net ISNS_INJ_B_SENSE: Q7.2 (S), R8.1
- new net LS1_GATE: Q3.1 (G), Q4.3 (D), R4.1
- new net LS2_GATE: Q7.1 (G), Q8.3 (D), R6.1
- new net LS3_GATE: Q5.1 (G), Q6.3 (D), R5.1
- new net VBAT_PROT: D1.2 (A), D2.2 (A)
Other:
- note added: "A GROUND-REFERENCED KILL CLAMP CANNOT SERVICE A HIGH-SIDE GATE, and spec sec.4's fail-safe list names pins 03/05 alongside the four low-side gates as though it could. The three low sides here get exactly the network supervisor.cir sized and docs/pinmap.md sec.2 confirmed pin by pin: a 470 ohm pulldown to ground, plus a small-signal FET that shorts the gate to ground when GATE_KILL asserts, with n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"
- note added: "BOOST RAIL -- 100 V reservoir for the injector peak phase"
- note added: "GATE_KILL reaches the two high sides through the driver's own SHUTDOWN input, not through a clamp -- a ground-referenced kill FET cannot short a gate that floats 100 V up. Nothing is drawn for it here because the driver is not chosen; see the note at the foot of the sheet."
- note added: "PARTS NOT CHOSEN ON THIS SHEET. Five gate drivers and two current-sense amplifiers, on the same named-net treatment power_input gives its two controller gates. LOW-SIDE DRIVERS (LS1/LS2/LS3_DRV_IN -> *_GATE). Output impedance <= 25 ohm, from supervisor.cir claim 2: the 470 ohm pulldown is not a perturbation on the driver, it is the bottom half of a divider with it, and at 100 ohm the gate reaches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"
- note added: "THE BOOST CONVERTER ITSELF IS NOT DRAWN. boost_converter.cir models it as an average charging current and says so: 'no inductor, no switch, no control loop.' That is enough to size the reservoir and it is not enough to draw a converter, so what is on this sheet is the part the block DID size -- the 47 uF reservoir, its 150 V class, and the bleed -- with VBAT_PROT and BOOST_100V naming the two end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"
- note added: "bank A (cyl 1+3)"
- note added: "bank B (cyl 2)"
- note added: "the converter is NOT drawn -- it sits between VBAT_PROT and BOOST_100V; see the note at the foot of the sheet"

Commit message: Draw the connector; the power ground turns out to have no pin
Sheet 10 of 10. Not a circuit -- the harness boundary, and its job is to
be checkable against the machine: every pin the wiring diagram shows
wired to the net whichever sheet owns that signal already named, and
every pin it does not show left visibly empty.

41 of 94 pins wired, 53 left empty, every pin accounted for exactly once
in the netlist.

THE FINDING. GP3.8703.C4.pdf shows pin 21 as the battery positive feed
and shows no battery negative anywhere on the ECU connector. That is a
gap in the source rather than a contradiction in it -- the document is a
field troubleshooting diagram and its own scope note says it omits
"power grounds, unused pins and internal-only pins". It is still a gap
that stops a board: every other sheet in this project returns to GND,
the injector low sides carry 18 A into it, and at this boundary that net
has nowhere to go. It cannot be closed by choosing. Fifty pins have no
established function and several are certainly grounds -- a 94-way
connector feeding an 18 A injector stage does not have one return -- but
a wrong ground pin is not a rework, it is a harness that has to be
remade. Same for TRIP_LOOP, which is a NEW signal not on the OEM diagram
at all and needs one of the same fifty.

CONN_ECU_94 carries pin count and pin numbers, which are facts read off
page 4, and no footprint, because no part number is known. Pin names are
the diagram's own signal names where it shows the pin and blank where it
does not. Same treatment the op-amps and the comparator get.

Two distinctions the sheet makes explicit: pins 34 and 36 are SHARED
sensor returns and therefore signals, carried into difference amplifiers
on sensors_analog; pin 08 is rail pressure's dedicated return, with
nothing to reject, so it is simply ground here.

CROSS-SHEET AUDIT. 83 hierarchical net names across the ten sheets, 73
appearing on two or more. All ten that appear on only one sheet are
explained by an open it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
Changed lines of the file:
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@@
   )
   (hierarchical_label "GATE_KILL" (shape input) (at 34.84 213.0 180)
-    (effects (font (size 1.27 1.27)) (justify left))
+    (effects (font (size 1.27 1.27)) (justify right))
   )
   (hierarchical_label "INJ_LS_1" (shape input) (at 39.92 178.0 0)
@@
   )
   (hierarchical_label "GATE_KILL" (shape input) (at 204.84 213.0 180)
-    (effects (font (size 1.27 1.27)) (justify left))
+    (effects (font (size 1.27 1.27)) (justify right))
   )
   (hierarchical_label "INJ_LS_3" (shape input) (at 209.92 178.0 0)
@@
   )
   (hierarchical_label "GATE_KILL" (shape input) (at 374.84 213.0 180)
-    (effects (font (size 1.27 1.27)) (justify left))
+    (effects (font (size 1.27 1.27)) (justify right))
   )
   (hierarchical_label "INJ_LS_2" (shape input) (at 379.92 178.0 0)

Commit message: Wire the root sheet: the project has a netlist for the first time
Ten sheets each passed their own netlist and the project had none. The
root sheet's ten sheet symbols carried NO hierarchical pins, so a net
name appearing on two sheets was two nets and nothing compared them --
the cross-sheet audit in the last commit was a name comparison, not a
connectivity check.

Each symbol now carries one pin per net its child exports, read OUT of
the child rather than declared in a second list that could drift: 162
pins across the ten, each with a stub and a label. Two labels with the
same name are one net, which is how 162 pins connect without routing
162 wires across a page nobody could read.

Exporting it found the other half of the same problem immediately.
kicad-cli reported annotation errors: every sheet generator allocated
R1, C1, U1 from its own counter, so ten sheets had ten parts called R1.
schlib.REF_BASE gives each sheet its own hundred -- KiCad's own
sheet-number x 100 convention, applied at generation time instead of by
a hand pass in Eeschema. 196 components, no duplicate reference.

hw/check_netlist.py is the gate, and the counterpart to sim/run_sim.py:
that one guards the component values, this one guards the connectivity.
Same rule -- an exemption is not a pass. Every single-pin net is listed
with its reason, and a net that STOPS being single-pin fails the check
until it is removed from the list. An open item that quietly closes is
as much a drift as one that quietly opens.

  196 components, every reference unique
  113 named nets carrying two or more pins
   18 named nets reaching one pin, each a recorded open item
      GND 134 pins, 3V3_MCU 27, VBAT_PROT 12 -- all spanning the project

The root sheet carries those eighteen on the page itself, grouped by
what they wait on, so a reader does not have to run a script to find
which ends are loose.

Full set plots to docs/pdf/ECU-Schematics.pdf, 11 pages.

Two rendering bugs fixed: sheet pin names and their stu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
Parts:
- removed C1: 47uF 150V, symbol Device:C_Polarized
- removed D1, D2, D3, D4, D5: 150V 20A ultrafast, symbol Device:D
- removed Q1, Q2: 150V N-ch, bootstrapped high side, symbol Device:Q_NMOS_GSD
- removed Q3, Q5, Q7: 150V N-ch, 18A peak, symbol Device:Q_NMOS_GSD
- removed Q4, Q6, Q8: 60V small-signal, symbol Device:Q_NMOS_GSD
- removed R1: 22k 1W, symbol Device:R
- removed R2, R3, R4, R5, R6: 470R, symbol Device:R
- removed R7, R8: 5mOhm 2W 1%, symbol Device:R
- added C401: 47uF 150V, symbol Device:C_Polarized
- added D401, D402, D403, D404, D405: 150V 20A ultrafast, symbol Device:D
- added Q401, Q402: 150V N-ch, bootstrapped high side, symbol Device:Q_NMOS_GSD
- added Q403, Q405, Q407: 150V N-ch, 18A peak, symbol Device:Q_NMOS_GSD
- added Q404, Q406, Q408: 60V small-signal, symbol Device:Q_NMOS_GSD
- added R401: 22k 1W, symbol Device:R
- added R402, R403, R404, R405, R406: 470R, symbol Device:R
- added R407, R408: 5mOhm 2W 1%, symbol Device:R
Connections:
- net BOOST_100V: now also C401.1, D403.1 (K), D404.1 (K), D405.1 (K), Q401.3 (D), Q402.3 (D), R401.1
- net GATE_KILL: now also Q404.1 (G), Q406.1 (G), Q408.1 (G)
- net GND: now also C401.2, Q404.2 (S), Q406.2 (S), Q408.2 (S), R401.2, R404.2, R405.2, R406.2, R407.2, R408.2
- net HSA_GATE: now also Q401.1 (G), R402.1
- net HSB_GATE: now also Q402.1 (G), R403.1
- net INJ_A_03: now also D401.1 (K), Q401.2 (S), R402.2
- net INJ_B_05: now also D402.1 (K), Q402.2 (S), R403.2
- net INJ_LS1_73: now also D403.2 (A), Q403.3 (D)
- net INJ_LS2_29: now also D405.2 (A), Q407.3 (D)
- net INJ_LS3_07: now also D404.2 (A), Q405.3 (D)
- net ISNS_INJ_A_SENSE: now also Q403.2 (S), Q405.2 (S), R407.1
- net ISNS_INJ_B_SENSE: now also Q407.2 (S), R408.1
- net LS1_GATE: now also Q403.1 (G), Q404.3 (D), R404.1
- net LS2_GATE: now also Q407.1 (G), Q408.3 (D), R406.1
- net LS3_GATE: now also Q405.1 (G), Q406.3 (D), R405.1
- net VBAT_PROT: now also D401.2 (A), D402.2 (A)
Changed lines of the file:
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@@
   (symbol (lib_id "Device:C_Polarized") (at 80.0 68.0 0) (unit 1)
     (in_bom yes) (on_board yes) (fields_autoplaced)
-    (property "Reference" "C1" (id 0) (at 80.0 62.92 0)
+    (property "Reference" "C401" (id 0) (at 80.0 62.92 0)
       (effects (font (size 1.27 1.27)))
     )
@@
   (symbol (lib_id "power:GND") (at 80.0 79.43 0) (unit 1)
     (in_bom yes) (on_board yes) (fields_autoplaced)
-    (property "Reference" "#PWR1" (id 0) (at 80.0 74.35000000000001 0)
+    (property "Reference" "#PWR401" (id 0) (at 80.0 74.35000000000001 0)
       (effects (font (size 1.27 1.27)) hide)
     )
@@
   (symbol (lib_id "Device:R") (at 120.0 68.0 0) (unit 1)
     (in_bom yes) (on_board yes) (fields_autoplaced)
-    (property "Reference" "R1" (id 0) (at 120.0 62.92 0)
+    (property "Reference" "R401" (id 0) (at 120.0 62.92 0)
       (effects (font (size 1.27 1.27)))
     )
@@
   (symbol (lib_id "power:GND") (at 120.0 79.43 0) (unit 1)
     (in_bom yes) (on_board yes) (fields_autoplaced)
-    (property "Reference" "#PWR2" (id 0) (at 120.0 74.35000000000001 0)
+    (property "Reference" "#PWR402" (id 0) (at 120.0 74.35000000000001 0)
       (effects (font (size 1.27 1.27)) hide)
     )
@@
   (symbol (lib_id "Device:Q_NMOS_GSD") (at 210.0 85.0 0) (unit 1)
     (in_bom yes) (on_board yes) (fields_autoplaced)
-    (property "Reference" "Q1" (id 0) (at 210.0 79.92 0)
+    (property "Reference" "Q401" (id 0) (at 210.0 79.92 0)
       (effects (font (size 1.27 1.27)))
     )
@@
   (symbol (lib_id "Device:R") (at 190.0 95.0 0) (unit 1)
     (in_bom yes) (on_board yes) (fields_autoplaced)
-    (property "Reference" "R2" (id 0) (at 190.0 89.92 0)
+    (property "Reference" "R402" (id 0) (at 190.0 89.92 0)
       (effects (font (size 1.27 1.27)))
     )
@@
   (symbol (lib_id "Device:D") (at 240.54 91.0 90) (unit 1)
     (in_bom yes) (on_board yes) (fields_autoplaced)
-    (property "Reference" "D1" (id 0) (at 240.54 85.92 0)
+    (property "Reference" "D401" (id 0) (at 240.54 85.92 0)
       (effects (font (size 1.27 1.27)))
     )
@@
   (symbol (lib_id "Device:Q_NMOS_GSD") (at 420.0 85.0 0) (unit 1)
     (in_bom yes) (on_board yes) (fields_autoplaced)
-    (property "Reference" "Q2" (id 0) (at 420.0 79.92 0)
+    (property "Reference" "Q402" (id 0) (at 420.0 79.92 0)
       (effects (font (size 1.27 1.27)))
     )
@@
   (symbol (lib_id "Device:R") (at 400.0 95.0 0) (unit 1)
     (in_bom yes) (on_board yes) (fields_autoplaced)
-    (property "Reference" "R3" (id 0) (at 400.0 89.92 0)
+    (property "Reference" "R403" (id 0) (at 400.0 89.92 0)
       (effects (font (size 1.27 1.27)))
     )
@@
   (symbol (lib_id "Device:D") (at 450.54 91.0 90) (unit 1)
     (in_bom yes) (on_board yes) (fields_autoplaced)
-    (property "Reference" "D2" (id 0) (at 450.54 85.92 0)
+    (property "Reference" "D402" (id 0) (at 450.54 85.92 0)
       (effects (font (size 1.27 1.27)))
     )
@@
   (symbol (lib_id "Device:Q_NMOS_GSD") (at 130.0 195.0 0) (unit 1)
     (in_bom yes) (on_board yes) (fields_autoplaced)
-    (property "Reference" "Q3" (id 0) (at 130.0 189.92 0)
+    (property "Reference" "Q403" (id 0) (at 130.0 189.92 0)
       (effects (font (size 1.27 1.27)))
     )
@@
   (symbol (lib_id "Device:D") (at 146.54 156.0 270) (unit 1)
     (in_bom yes) (on_board yes) (fields_autoplaced)
-    (property "Reference" "D3" (id 0) (at 146.54 150.92 0)
+    (property "Reference" "D403" (id 0) (at 146.54 150.92 0)
       (effects (font (size 1.27 1.27)))
     )
@@
   (symbol (lib_id "Device:R") (at 84.92 213.0 0) (unit 1)
     (in_bom yes) (on_board yes) (fields_autoplaced)
-    (property "Reference" "R4" (id 0) (at 84.92 207.92 0)
+    (property "Reference" "R404" (id 0) (at 84.92 207.92 0)
       (effects (font (size 1.27 1.27)))
     )
@@
   (symbol (lib_id "power:GND") (at 84.92 224.43 0) (unit 1)
     (in_bom yes) (on_board yes) (fields_autoplaced)
-    (property "Reference" "#PWR3" (id 0) (at 84.92 219.35 0)
+    (property "Reference" "#PWR403" (id 0) (at 84.92 219.35 0)
       (effects (font (size 1.27 1.27)) hide)
     )
@@
   (symbol (lib_id "Device:Q_NMOS_GSD") (at 54.92 213.0 0) (unit 1)
     (in_bom yes) (on_board yes) (fields_autoplaced)
-    (property "Reference" "Q4" (id 0) (at 54.92 207.92 0)
+    (property "Reference" "Q404" (id 0) (at 54.92 207.92 0)
       (effects (font (size 1.27 1.27)))
     )
@@
   (symbol (lib_id "power:GND") (at 57.46 225.7 0) (unit 1)
     (in_bom yes) (on_board yes) (fields_autoplaced)
-    (property "Reference" "#PWR4" (id 0) (at 57.46 220.62 0)
+    (property "Reference" "#PWR404" (id 0) (at 57.46 220.62 0)
       (effects (font (size 1.27 1.27)) hide)
     )
@@
   (symbol (lib_id "Device:Q_NMOS_GSD") (at 300.0 195.0 0) (unit 1)
     (in_bom yes) (on_board yes) (fields_autoplaced)
-    (property "Reference" "Q5" (id 0) (at 300.0 189.92 0)
+    (property "Reference" "Q405" (id 0) (at 300.0 189.92 0)
       (effects (font (size 1.27 1.27)))
     )
@@
   (symbol (lib_id "Device:D") (at 316.54 156.0 270) (unit 1)
     (in_bom yes) (on_board yes) (fields_autoplaced)
-    (property "Reference" "D4" (id 0) (at 316.54 150.92 0)
+    (property "Reference" "D404" (id 0) (at 316.54 150.92 0)
       (effects (font (size 1.27 1.27)))
     )
@@
   (symbol (lib_id "Device:R") (at 254.92 213.0 0) (unit 1)
     (in_bom yes) (on_board yes) (fields_autoplaced)
-    (property "Reference" "R5" (id 0) (at 254.92000000000002 207.92 0)
+    (property "Reference" "R405" (id 0) (at 254.92000000000002 207.92 0)
       (effects (font (size 1.27 1.27)))
     )
@@
   (symbol (lib_id "power:GND") (at 254.92 224.43 0) (unit 1)
     (in_bom yes) (on_board yes) (fields_autoplaced)
-    (property "Reference" "#PWR5" (id 0) (at 254.92000000000002 219.35 0)
+    (property "Reference" "#PWR405" (id 0) (at 254.92000000000002 219.35 0)
       (effects (font (size 1.27 1.27)) hide)
     )
@@
   (symbol (lib_id "Device:Q_NMOS_GSD") (at 224.92 213.0 0) (unit 1)
     (in_bom yes) (on_board yes) (fields_autoplaced)
-    (property "Reference" "Q6" (id 0) (at 224.92000000000002 207.92 0)
+    (property "Reference" "Q406" (id 0) (at 224.92000000000002 207.92 0)
       (effects (font (size 1.27 1.27)))
     )
@@
   (symbol (lib_id "power:GND") (at 227.46 225.7 0) (unit 1)
     (in_bom yes) (on_board yes) (fields_autoplaced)
-    (property "Reference" "#PWR6" (id 0) (at 227.46 220.62 0)
+    (property "Reference" "#PWR406" (id 0) (at 227.46 220.62 0)
       (effects (font (size 1.27 1.27)) hide)
     )
@@
   (symbol (lib_id "Device:Q_NMOS_GSD") (at 470.0 195.0 0) (unit 1)
     (in_bom yes) (on_board yes) (fields_autoplaced)
-    (property "Reference" "Q7" (id 0) (at 470.0 189.92 0)
+    (property "Reference" "Q407" (id 0) (at 470.0 189.92 0)
       (effects (font (size 1.27 1.27)))
     )
@@
   (symbol (lib_id "Device:D") (at 486.54 156.0 270) (unit 1)
     (in_bom yes) (on_board yes) (fields_autoplaced)
-    (property "Reference" "D5" (id 0) (at 486.54 150.92 0)
+    (property "Reference" "D405" (id 0) (at 486.54 150.92 0)
       (effects (font (size 1.27 1.27)))
     )
@@
   (symbol (lib_id "Device:R") (at 424.92 213.0 0) (unit 1)
     (in_bom yes) (on_board yes) (fields_autoplaced)
-    (property "Reference" "R6" (id 0) (at 424.92 207.92 0)
+    (property "Reference" "R406" (id 0) (at 424.92 207.92 0)
       (effects (font (size 1.27 1.27)))
     )
@@
   (symbol (lib_id "power:GND") (at 424.92 224.43 0) (unit 1)
     (in_bom yes) (on_board yes) (fields_autoplaced)
-    (property "Reference" "#PWR7" (id 0) (at 424.92 219.35 0)
+    (property "Reference" "#PWR407" (id 0) (at 424.92 219.35 0)
       (effects (font (size 1.27 1.27)) hide)
     )
@@
   (symbol (lib_id "Device:Q_NMOS_GSD") (at 394.92 213.0 0) (unit 1)
     (in_bom yes) (on_board yes) (fields_autoplaced)
-    (property "Reference" "Q8" (id 0) (at 394.92 207.92 0)
+    (property "Reference" "Q408" (id 0) (at 394.92 207.92 0)
       (effects (font (size 1.27 1.27)))
     )
@@
   (symbol (lib_id "power:GND") (at 397.46 225.7 0) (unit 1)
     (in_bom yes) (on_board yes) (fields_autoplaced)
-    (property "Reference" "#PWR8" (id 0) (at 397.46000000000004 220.62 0)
+    (property "Reference" "#PWR408" (id 0) (at 397.46000000000004 220.62 0)
       (effects (font (size 1.27 1.27)) hide)
     )
@@
   (symbol (lib_id "Device:R") (at 200.0 260.0 0) (unit 1)
     (in_bom yes) (on_board yes) (fields_autoplaced)
-    (property "Reference" "R7" (id 0) (at 200.0 254.92 0)
+    (property "Reference" "R407" (id 0) (at 200.0 254.92 0)
       (effects (font (size 1.27 1.27)))
     )
@@
   (symbol (lib_id "power:GND") (at 200.0 271.43 0) (unit 1)
     (in_bom yes) (on_board yes) (fields_autoplaced)
-    (property "Reference" "#PWR9" (id 0) (at 200.0 266.35 0)
+    (property "Reference" "#PWR409" (id 0) (at 200.0 266.35 0)
       (effects (font (size 1.27 1.27)) hide)
     )
@@
   (symbol (lib_id "Device:R") (at 500.0 260.0 0) (unit 1)
     (in_bom yes) (on_board yes) (fields_autoplaced)
-    (property "Reference" "R8" (id 0) (at 500.0 254.92 0)
+    (property "Reference" "R408" (id 0) (at 500.0 254.92 0)
       (effects (font (size 1.27 1.27)))
     )
@@
   (symbol (lib_id "power:GND") (at 500.0 271.43 0) (unit 1)
     (in_bom yes) (on_board yes) (fields_autoplaced)
-    (property "Reference" "#PWR10" (id 0) (at 500.0 266.35 0)
-      (effects (font (size 1.27 1.27)) hide)
-    )
+    (property "Reference" "#PWR410" (id 0) (at 500.0 266.35 0)
+      (effects (font (size 1.27 1.27)) hide)
+    )
