File: hw/injector.kicad_sch (KiCad schematic)
At the start: 22 parts, among them Q401 150V N-ch, bootstrapped high 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, Q402 150V N-ch, bootstrapped high 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, Q403 150V N-ch, 18A peak, Q404 60V small-signal, Q405 150V N-ch, 18A peak, Q406 60V small-signal, Q407 150V N-ch, 18A peak, Q408 60V small-signal

Commit message: Choose the injector boost controller: TPS40210-Q1, on an off-time
Track B's first part. TI SLVS861F (Aug 2008, rev. Jun 2020), retrieved
and text-extracted, not recalled.

CHOSEN ON ONE NUMBER, and the reasoning runs backwards from the usual.
tOFF(min) = 200 ns max (Table 6.6). A boost from the 6 V cranking dip to
100 V needs D = 1 - 6/100.9 = 94.05%, and a controller's minimum
off-time is a floor in TIME, not in duty. At 150 kHz that 200 ns is 3%
of the period, so Dmax = 97.0% and the cranking corner clears by 2.95
points. At 2.2 MHz -- where most wide-input boost controllers in this
class sit, and where the magnetics would be far smaller -- the same
200 ns is 44% of the period and Dmax falls to 56%, below even the 86.6%
the rail needs at a NOMINAL 13.5 V battery. "Higher frequency, smaller
inductor" is the wrong optimisation here and the part that looks less
modern is the one that works.

THE RATING THAT DOES NOT FIT, for the third time on this board. VDD
absolute maximum is 52 V (Table 6.1); VBAT_PROT reaches 73.3 V for about
50 us on ISO 7637-2 pulse 2a. Over by 1.41x. Same shape as DRV8873-Q1's
40 V VM, which took that part off the EGR bridge -- and solvable here
for a reason that did not apply there: a motor bridge's VM carries the
motor current, this pin carries 2.5 mA plus gate charge. So it gets 47
ohm and a 43 V zener.

43 V rather than 39 V is the whole point of the value. A 39 V clamp
would sit in conduction for the load dump's entire 400 ms at roughly
0.8 W; a 43 V clamp only works during the 50 us pulse, where 1.39 mJ is
nothing. The 47 ohm is squeezed from both ends: small enough that
6.25 mA does not drop the part below UVLO at the cranking dip (VDD
5.71 V against a 4.5 V ceiling), large enough that the zener sees
645 mA and not more.

The power stage is untouched by any of that -- inductor and FET see the
rail directly and are 150 V class for it.

CHECKED AS ARITHMETIC, NOT AS PROSE. boost_converter.cir models the
converter as an average charging cu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
Parts:
- removed D402: 150V 20A ultrafast, symbol Device:D
- added C402: 4.7uF 100V, symbol Device:C
- added C403: 1uF 100V, symbol Device:C
- added C404: 330pF, symbol Device:C
- added C405: 100nF, symbol Device:C
- added C406: 1uF, symbol Device:C
- added C407: 6.8nF, symbol Device:C
- added D402: 43V 1W, symbol Device:D_Zener
- added D406, D407: 150V 20A ultrafast, symbol Device:D
- added L401: 330uH 3A, symbol Device:L
- added Q409: 60V small-signal, symbol Device:Q_NMOS_GSD
- added R409: 10k, symbol Device:R
- added R410, R411, R412, R413, R414: 470R, symbol Device:R
- added R415, R416: 5mOhm 2W 1%, symbol Device:R
- added U401: TPS40210, Package_SO:HVSSOP-10-1EP_3x3mm_P0.5mm_EP1.57x1.88mm, symbol ecu25kva:TPS40210
- D401: value 150V 20A ultrafast -> 150V 2A ultrafast; Note Anode on the battery. Reverse biased while the bank sits ne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 -> The boost diode. Reverse voltage is the output, 100 V, so t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; Source settled on this sheet -- see the module docstring -> (none); Vr (none) -> 150 V
- D403, D404: Note Low side back into the boost reservoir. NOT a Zener active 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 -> Anode on the battery. Reverse biased while the bank sits ne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; Peak 28.7 W instantaneous during turn-off, ~8x the 3.6 W average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 -> (none); Source injector_turnoff.cir Drc -- the diode memo 10 recommends an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 -> settled on this sheet -- see the module docstring
- Q401: value 150V N-ch, bootstrapped high side -> 150V N-ch, logic-level; Note Bank-shared: cylinders 1 and 3 fire 240 crank degrees apart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 -> Grounded source, which is what TPS40210-Q1 requires. LOGIC-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; Qg (none) -> <=25 nC -- it sets the 3.75 mA of gate-drive current the VD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; Source injector_boost.cir -- the 100 V branch; injector_turnoff.ci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 -> sized here -- see the sheet note; Vds 150 V class against a 100 V rail that the recirculation bum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 -> 150 V
- Q402: Note One cylinder in this bank. Kept as a separate switch rather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 -> Bank-shared: cylinders 1 and 3 fire 240 crank degrees apart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
- Q403: value 150V N-ch, 18A peak -> 150V N-ch, bootstrapped high side; Note Cylinder 1. Independent per channel -- the high side is ban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 -> One cylinder in this bank. Kept as a separate switch rather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; Source injector_turnoff.cir Sls (Ron 20 mOhm) -> injector_boost.cir -- the 100 V branch; injector_turnoff.ci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; Vds 150 V class: at turn-off this drain is driven above the 100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 -> 150 V class against a 100 V rail that the recirculation bum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
- Q404: value 60V small-signal -> 150V N-ch, 18A peak; Note In parallel with the 470 ohm pulldown, not instead of it. R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 -> Cylinder 1. Independent per channel -- the high side is ban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; Source supervisor.cir -- the kill FET -> injector_turnoff.cir Sls (Ron 20 mOhm); Vds (none) -> 150 V class: at turn-off this drain is driven above the 100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
- Q405: value 150V N-ch, 18A peak -> 60V small-signal; Note Cylinder 3. Independent per channel -- the high side is ban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 -> In parallel with the 470 ohm pulldown, not instead of it. R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; Source injector_turnoff.cir Sls (Ron 20 mOhm) -> supervisor.cir -- the kill FET; Vds 150 V class: at turn-off this drain is driven above the 100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 -> (none)
- Q406: value 60V small-signal -> 150V N-ch, 18A peak; Note In parallel with the 470 ohm pulldown, not instead of it. R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 -> Cylinder 3. Independent per channel -- the high side is ban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; Source supervisor.cir -- the kill FET -> injector_turnoff.cir Sls (Ron 20 mOhm); Vds (none) -> 150 V class: at turn-off this drain is driven above the 100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
- Q407: value 150V N-ch, 18A peak -> 60V small-signal; Note Cylinder 2. Independent per channel -- the high side is ban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 -> In parallel with the 470 ohm pulldown, not instead of it. R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; Source injector_turnoff.cir Sls (Ron 20 mOhm) -> supervisor.cir -- the kill FET; Vds 150 V class: at turn-off this drain is driven above the 100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 -> (none)
- Q408: value 60V small-signal -> 150V N-ch, 18A peak; Note In parallel with the 470 ohm pulldown, not instead of it. R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 -> Cylinder 2. Independent per channel -- the high side is ban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; Source supervisor.cir -- the kill FET -> injector_turnoff.cir Sls (Ron 20 mOhm); Vds (none) -> 150 V class: at turn-off this drain is driven above the 100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
- R402: value 470R -> 82mOhm 1%; Note Across gate and source, because the source of a high-side N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 -> Current limit lands in 1.46-2.20 A across the threshold's o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; Power (none) -> 1.06^2 * 82 mOhm = 92 mW; Source supervisor.cir claim 6, referenced to SOURCE rather than to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 -> TPS40210-Q1 Table 6.5, VISNS(oc) 120-180 mV
- R403: value 470R -> 10k; Note Across gate and source, because the source of a high-side N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 -> Pulled down rather than left floating, so the enable state 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; Source supervisor.cir claim 6, referenced to SOURCE rather than to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 -> TPS40210-Q1 Table 6.5 -- DIS/EN has a 1 MOhm internal pulld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
- R404: value 470R -> 7.06k 1%; Cost 21.3 mA per gate at 10 V; 1.28 W across all six -> (none); Note Largest standard value holding the gate under Vgs(th)=1.0 V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 -> With 998k above: 0.700 * (998000+7060)/7060 = 99.7 V. The r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; Source supervisor.cir claim 6; bom_requirements GATE-PULLDOWN -> TPS40210-Q1 VFB = 700 mV (686-714 mV over temp)
- R405: value 470R -> 47R 1W; Cost 21.3 mA per gate at 10 V; 1.28 W across all six -> (none); Note Largest standard value holding the gate under Vgs(th)=1.0 V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 -> The other half of the clamp. Small enough that 6.25 mA drop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; Source supervisor.cir claim 6; bom_requirements GATE-PULLDOWN -> (none); Tag (none) -> BOOST-VDD-CLAMP
- R406: value 470R -> 365k 1%; Cost 21.3 mA per gate at 10 V; 1.28 W across all six -> (none); Note Largest standard value holding the gate under Vgs(th)=1.0 V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 -> 365k with 330 pF gives 150 kHz. Frequency line regulation i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; Source supervisor.cir claim 6; bom_requirements GATE-PULLDOWN -> TPS40210-Q1 -- RC resistor returns to VDD, not to a rail of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
- R407: value 5mOhm 2W 1% -> 499k 1%; Note Bank A, cylinders 1 and 3 sharing one return. They fire 240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 -> Two in series, not one. 100 V across a single 1206 is insid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; Power 1.62 W at peak, but ~1.25% duty per cylinder at 1500 rpm -> (none); Signal 90 mV at the 18 A peak, 50 mV at the 10 A hold -- too small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 -> (none); Source settled on this sheet -- docs/pinmap.md sec.1.6 asked for t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 -> (none)
- R408: value 5mOhm 2W 1% -> 499k 1%; Note Bank B, cylinder 2 alone. Drawn as its own shunt rather tha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 -> Second half of the pair.; Power 1.62 W at peak, but ~1.25% duty per cylinder at 1500 rpm -> (none); Signal 90 mV at the 18 A peak, 50 mV at the 10 A hold -- too small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 -> (none); Source settled on this sheet -- docs/pinmap.md sec.1.6 asked for t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 -> (none)
Connections:
- net BOOST_100V: now also D401.1 (K), Q403.3 (D), R407.1, D406.1 (K), D407.1 (K); no longer D403.1 (K), D404.1 (K), Q401.3 (D)
- net GATE_KILL: now also Q405.1 (G), Q407.1 (G), Q409.1 (G); no longer Q404.1 (G), Q406.1 (G), Q408.1 (G)
- net GND: now also Q405.2 (S), Q407.2 (S), R402.2, R403.2, C402.2, C403.2, C404.2, C405.2, C406.2, D402.2 (A), Q409.2 (S), R412.2, R413.2, R414.2, R415.2, R416.2, U401.6 (GND); no longer Q404.2 (S), Q406.2 (S), Q408.2 (S), R405.2, R406.2, R407.2, R408.2
- net HSA_GATE: now also Q402.1 (G), R410.1; no longer Q401.1 (G), R402.1
- net HSB_GATE: now also Q403.1 (G), R411.1; no longer Q402.1 (G), R403.1
- net INJ_A_03: now also D403.1 (K), Q402.2 (S), R410.2; no longer D401.1 (K), Q401.2 (S), R402.2
- net INJ_B_05: now also D404.1 (K), Q403.2 (S), R411.2; no longer Q402.2 (S), R403.2
- net INJ_LS1_73: now also D405.2 (A), Q404.3 (D); no longer D403.2 (A), Q403.3 (D)
- net INJ_LS2_29: now also Q408.3 (D), D407.2 (A); no longer D405.2 (A), Q407.3 (D)
- net INJ_LS3_07: now also Q406.3 (D), D406.2 (A); no longer D404.2 (A), Q405.3 (D)
- net ISNS_INJ_A_SENSE: now also Q404.2 (S), Q406.2 (S), R415.1; no longer Q403.2 (S), Q405.2 (S), R407.1
- net ISNS_INJ_B_SENSE: now also Q408.2 (S), R416.1; no longer Q407.2 (S), R408.1
- net LS1_GATE: now also Q404.1 (G), Q405.3 (D), R412.1; no longer Q403.1 (G), Q404.3 (D), R404.1
- net LS2_GATE: now also Q408.1 (G), Q409.3 (D), R414.1; no longer Q407.1 (G), Q408.3 (D), R406.1
- net LS3_GATE: now also Q406.1 (G), Q407.3 (D), R413.1; no longer Q405.1 (G), Q406.3 (D), R405.1
- net VBAT_PROT: now also D403.2 (A), D404.2 (A), R405.1, C402.1, L401.1; no longer D401.2 (A)
- new net: R407.2, R408.1
- new net: C407.1, R409.2
- new net BP_BOOST: C406.1, U401.9 (BP)
- new net COMP_BOOST: R409.1, U401.4 (COMP)
- new net EN_BOOST: R403.1, U401.3 (DIS/EN)
- new net FB_BOOST: C407.2, R404.1, R408.2, U401.5 (FB)
- new net GDRV_BOOST: Q401.1 (G), U401.8 (GDRV)
- new net ISNS_BOOST: Q401.2 (S), R402.1, U401.7 (ISNS)
- new net RC_BOOST: C404.1, R406.2, U401.1 (RC)
- new net SS_BOOST: C405.1, U401.2 (SS)
- new net SW_BOOST: D401.2 (A), L401.2, Q401.3 (D)
- new net VDD_BOOST: C403.1, D402.1 (K), R405.2, R406.1, U401.10 (VDD)
Other:
- note added: "BOOST CONVERTER -- TPS40210-Q1, 6-40 V in, 100 V out at 50 mA average. The reservoir above delivers the pulse; this delivers the trickle."
- note added: "THE BOOST CONVERTER IS NOW DRAWN, AND THE PART WAS CHOSEN ON ONE NUMBER: tOFF(min) = 200 ns max, TI SLVS861F Table 6.6. A boost needs 94.1% duty at the 6 V cranking corner, and at 150 kHz that off-time floor allows 97.0%. Most wide-input boost controllers in this class switch at 2.2 MHz, where the same 200 ns caps duty at 56% -- below even the 86.6% the rail needs at a nominal 13.5 V battery. Swi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"
- note added: "THE COMPENSATION VALUES ARE A STARTING POINT AND THE SHEET SAYS SO. Rcomp 10k and Ccomp 6.8 nF put the error amplifier's zero at 2.3 kHz, below the right-half-plane zero a boost converter puts at (1-D)^2 * Rload / (2*pi*L) = 17.3 kHz at 13.5 V in -- which is the constraint that actually bounds crossover, and it MOVES with duty cycle, so the cranking corner is the hard one. Everything else on this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"
- note removed: "THE BOOST CONVERTER ITSELF IS NOT DRAWN. boost_converter.cir models it as an average charging current and says so: 'no inductor, no switch, no control loop.' That is enough to size the reservoir and it is not enough to draw a converter, so what is on this sheet is the part the block DID size -- the 47 uF reservoir, its 150 V class, and the bleed -- with VBAT_PROT and BOOST_100V naming the two end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"
- title: Injector drive: boost rail, high sides, low sides -> Injector drive: boost converter, boost rail, high sides, low sides

Commit message: Correct the injector high side: a diode-OR cannot be chopped or bootstrapped
Choosing a gate driver for the high side found an error in the sheet
drawn two commits ago. The bank node was fed from VBAT_PROT through a
plain diode-OR, with the LOW side chopping for hold, on the argument
that it needed no extra MCU pin. It is wrong three ways, and only the
third is visible from a datasheet -- which is why drawing it did not
catch it and choosing a part for it did.

1. IT CANNOT REGULATE HOLD. With the battery on a diode the only switch
   in the loop is the low side, and when the low side opens the coil's
   current has nowhere to go but the recirculation diode into the 100 V
   boost rail. That is a fast decay against -87 V -- turn-off, not
   chopping. Hold needs a slow freewheel around the coil.

2. IT LEAVES CONNECTOR PINS 03 AND 05 PERMANENTLY LIVE. A diode from
   the battery to a connector pin means a harness short to ground draws
   current whenever the battery is connected, with no switch anywhere
   to stop it.

3. THE GATE DRIVER CANNOT BE BOOTSTRAPPED. A bootstrap capacitor
   charges when the switch node goes LOW. A battery diode holds that
   node at 12.8 V, so it never does, and the high side's floating supply
   can never refresh.

What replaces it is what injector_turnoff.cir already models and spends
a paragraph of its header justifying: two high-side switches per bank
onto a common node -- boost rail for the peak phase, battery for hold --
plus D_fw from GROUND to that node. Hold chopping moves to the high
side, the node swings to -0.7 V on every off-time, and the bootstrap
charges. Both switches have their SOURCE on the bank node, so one
floating supply serves two gates.

The battery switch needs a series BLOCKING diode and would with either
polarity of FET: an N-channel's body diode points source to drain, so
with the bank at 100 V during the peak phase it would dump the boost
rail into the battery. It goes on the drain side, which leaves the FET's
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
Parts:
- added D408, D409: 150V 20A ultrafast, symbol Device:D
- added Q410: 150V N-ch, 18A peak, symbol Device:Q_NMOS_GSD
- added Q411: 60V small-signal, symbol Device:Q_NMOS_GSD
- added R417, R418: 470R, symbol Device:R
- added R419, R420: 5mOhm 2W 1%, symbol Device:R
- D403: Note Anode on the battery. Reverse biased while the bank sits ne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 -> BLOCKING, not freewheeling. Without it the battery FET's ow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; Source settled on this sheet -- see the module docstring -> (none); Tag (none) -> INJ-RECIRC
- D404: Note Anode on the battery. Reverse biased while the bank sits ne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 -> Anode to GROUND, cathode to the bank node. This is the slow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; Source settled on this sheet -- see the module docstring -> injector_turnoff.cir D_fw; Tag (none) -> INJ-RECIRC
- D405: Note Low side back into the boost reservoir. NOT a Zener active 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 -> BLOCKING, not freewheeling. Without it the battery FET's ow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; Peak 28.7 W instantaneous during turn-off, ~8x the 3.6 W average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 -> (none); Source injector_turnoff.cir Drc -- the diode memo 10 recommends an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 -> (none); Tag (none) -> INJ-RECIRC
- D406: Note Low side back into the boost reservoir. NOT a Zener active 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 -> Anode to GROUND, cathode to the bank node. This is the slow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; Peak 28.7 W instantaneous during turn-off, ~8x the 3.6 W average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 -> (none); Source injector_turnoff.cir Drc -- the diode memo 10 recommends an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 -> injector_turnoff.cir D_fw; Tag (none) -> INJ-RECIRC
- Q402: value 150V N-ch, bootstrapped high side -> 150V N-ch, 18A peak; Vds 150 V class against a 100 V rail that the recirculation bum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 -> 150 V class against a 100 V rail the recirculation bump can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
- Q403: value 150V N-ch, bootstrapped high side -> 60V N-ch, 18A; Note One cylinder in this bank. Kept as a separate switch rather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 -> Chops for hold. 60 V class, not 150 V: the series blocking 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; Source injector_boost.cir -- the 100 V branch; injector_turnoff.ci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 -> boost_converter.cir arrangement A -- hold current comes fro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; Vds 150 V class against a 100 V rail that the recirculation bum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 -> 60 V
- Q404: Note Cylinder 1. Independent per channel -- the high side is ban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 -> One cylinder in this bank. Kept as a separate switch rather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; Source injector_turnoff.cir Sls (Ron 20 mOhm) -> injector_boost.cir -- the 100 V branch; injector_turnoff.ci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; Vds 150 V class: at turn-off this drain is driven above the 100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 -> 150 V class against a 100 V rail the recirculation bump can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
- Q405: value 60V small-signal -> 60V N-ch, 18A; Note In parallel with the 470 ohm pulldown, not instead of it. R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 -> Chops for hold. 60 V class, not 150 V: the series blocking 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; Source supervisor.cir -- the kill FET -> boost_converter.cir arrangement A -- hold current comes fro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; Vds (none) -> 60 V
- Q406: Note Cylinder 3. Independent per channel -- the high side is ban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 -> Cylinder 1. Independent per channel -- the high side is ban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
- Q408: Note Cylinder 2. Independent per channel -- the high side is ban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 -> Cylinder 3. Independent per channel -- the high side is ban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
- R410, R411: Note Across gate and source, because the source of a high-side N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 -> A pulldown to GROUND here would hold Vgs at minus the bank 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
- R412: value 470R -> 100k; Cost 21.3 mA per gate at 10 V; 1.28 W across all six -> (none); Note Largest standard value holding the gate under Vgs(th)=1.0 V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 -> Bleed. With both high sides off and the low sides off, noth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; Source supervisor.cir claim 6; bom_requirements GATE-PULLDOWN -> (none)
- R413, R414: Cost 21.3 mA per gate at 10 V; 1.28 W across all six -> (none); Note Largest standard value holding the gate under Vgs(th)=1.0 V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 -> A pulldown to GROUND here would hold Vgs at minus the bank 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; Source supervisor.cir claim 6; bom_requirements GATE-PULLDOWN -> supervisor.cir claim 6, referenced to SOURCE rather than to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
- R415: value 5mOhm 2W 1% -> 100k; Note Bank A, cylinders 1 and 3 sharing one return. They fire 240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 -> Bleed. With both high sides off and the low sides off, noth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; Power 1.62 W at peak, but ~1.25% duty per cylinder at 1500 rpm -> (none); Signal 90 mV at the 18 A peak, 50 mV at the 10 A hold -- too small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 -> (none); Source settled on this sheet -- docs/pinmap.md sec.1.6 asked for t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 -> (none)
- R416: value 5mOhm 2W 1% -> 470R; Cost (none) -> 21.3 mA per gate at 10 V; 1.28 W across all six; Note Bank B, cylinder 2 alone. Drawn as its own shunt rather tha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 -> Largest standard value holding the gate under Vgs(th)=1.0 V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; Power 1.62 W at peak, but ~1.25% duty per cylinder at 1500 rpm -> (none); Signal 90 mV at the 18 A peak, 50 mV at the 10 A hold -- too small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 -> (none); Source settled on this sheet -- docs/pinmap.md sec.1.6 asked for t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 -> supervisor.cir claim 6; bom_requirements GATE-PULLDOWN
Connections:
- net BOOST_100V: now also Q404.3 (D), D408.1 (K), D409.1 (K); no longer D405.1 (K), D406.1 (K), Q403.3 (D)
- net GATE_KILL: now also Q411.1 (G); no longer Q405.1 (G)
- net GND: now also D404.2 (A), D406.2 (A), Q411.2 (S), R417.2, R418.2, R419.2, R420.2; no longer Q405.2 (S), R413.2, R414.2
- net INJ_A_03: now also D404.1 (K), Q403.2 (S), R411.2, R412.1; no longer D403.1 (K)
- net INJ_B_05: now also D406.1 (K), Q404.2 (S), Q405.2 (S), R413.2, R414.2, R415.1; no longer D404.1 (K), Q403.2 (S), R411.2
- net INJ_LS1_73: now also D407.2 (A), Q406.3 (D); no longer D405.2 (A), Q404.3 (D)
- net INJ_LS2_29: now also D409.2 (A), Q410.3 (D); no longer D407.2 (A), Q408.3 (D)
- net INJ_LS3_07: now also Q408.3 (D), D408.2 (A); no longer D406.2 (A), Q406.3 (D)
- net ISNS_INJ_A_SENSE: now also Q408.2 (S), R419.1; no longer Q404.2 (S), R415.1
- net ISNS_INJ_B_SENSE: now also Q410.2 (S), R420.1; no longer Q408.2 (S), R416.1
- net LS1_GATE: now also Q406.1 (G), Q407.3 (D), R416.1; no longer Q404.1 (G), Q405.3 (D), R412.1
- net LS2_GATE: now also Q410.1 (G), Q411.3 (D), R418.1; no longer Q408.1 (G), Q409.3 (D), R414.1
- net LS3_GATE: now also Q408.1 (G), Q409.3 (D), R417.1; no longer Q406.1 (G), Q407.3 (D), R413.1
- net VBAT_PROT: now also D405.2 (A); no longer D404.2 (A)
- net HSA_GATE renamed HSA_BOOST_GATE
- net HSB_GATE renamed HSA_BAT_GATE
- new net: D405.1 (K), Q405.3 (D)
- new net: D403.1 (K), Q403.3 (D)
- new net HSB_BAT_GATE: Q405.1 (G), R414.1
- new net HSB_BOOST_GATE: Q404.1 (G), R413.1
Other:
- note added: "GATE_KILL reaches the four high sides through the driver's own SHUTDOWN input, not through a clamp -- a ground-referenced kill FET cannot short a gate that floats 100 V up. Nothing is drawn for it here because the driver is not chosen; see the note at the foot of the sheet."
- note added: "PARTS NOT CHOSEN ON THIS SHEET. Seven gate drivers and two current-sense amplifiers, on the same named-net treatment power_input gives its two controller gates. LOW-SIDE DRIVERS (LS1/LS2/LS3_DRV_IN -> *_GATE). Output impedance <= 25 ohm, from supervisor.cir claim 2: the 470 ohm pulldown is not a perturbation on the driver, it is the bottom half of a divider with it, and at 100 ohm the gate reache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"
- note added: "the converter that feeds this rail is drawn at the foot of the sheet -- TPS40210-Q1, VBAT_PROT to BOOST_100V"
- note removed: "GATE_KILL reaches the two high sides through the driver's own SHUTDOWN input, not through a clamp -- a ground-referenced kill FET cannot short a gate that floats 100 V up. Nothing is drawn for it here because the driver is not chosen; see the note at the foot of the sheet."
- note removed: "PARTS NOT CHOSEN ON THIS SHEET. Five gate drivers and two current-sense amplifiers, on the same named-net treatment power_input gives its two controller gates. LOW-SIDE DRIVERS (LS1/LS2/LS3_DRV_IN -> *_GATE). Output impedance <= 25 ohm, from supervisor.cir claim 2: the 470 ohm pulldown is not a perturbation on the driver, it is the bottom half of a divider with it, and at 100 ohm the gate reaches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"
- note removed: "the converter is NOT drawn -- it sits between VBAT_PROT and BOOST_100V; see the note at the foot of the sheet"
