File: hw/injector.kicad_sch (KiCad schematic)
At the start: 84 parts, among them Q401 150V N-ch, logic-level, Q402 60V small-signal, Q403 60V small-signal, Q404 60V small-signal, Q405 60V small-signal, Q406 NPN 160V, DPAK, Q407 NPN small-signal, Q408 150V N-ch, 18A peak, Q409 60V N-ch, 18A, Q410 150V N-ch, 18A peak, Q411 60V N-ch, 18A, Q412 150V N-ch, 18A peak, Q413 60V small-signal, Q414 150V N-ch, 18A peak, Q415 60V small-signal, Q416 150V N-ch, 18A peak, Q417 60V small-signal, U401 TPS40210, U402 AUIRS2181S, U403 AUIRS2181S, U404 AUIRS2181S, U405 AUIRS2181S, U406 INA181A1, U407 INA181A1

Commit message: Clamp GATE_KILL at 12 V and buffer the relay gates to 5 V
Choosing the small-signal FETs found two gate-drive errors.

GATE_KILL is pulled to VBAT_PROT so the kill path survives a 3V3
brownout, but only FET gates load it, so it followed the rail to
73.3 V on pulse 2a -- 3.7x a +/-20 V Vgs rating. A BZX84-C12-Q now
holds it at 12.7 V (13.7 V hot); transient_clamp checks the margin,
the zener current and the pullup dissipation.

The relay FETs were driven straight from 3.3 V GPIOs, with a note
claiming full enhancement at 3.0 V. No 100 V automotive small-signal
FET checked (PMV280ENEA, DMN10H220LQ, BSS123N) is specified below
Vgs = 4.5 V. An SN74AHCT1G125-Q1 on 5V_MAIN now drives each gate,
with a 100k input pulldown for reset; relay_driver checks overdrive
and drop.

Parts: 2N7002BK for the nine kill FETs and the reset inverter,
PMV280ENEA for the relay FETs. Also fixes the diagonal VBAT_PROT wire
to both relay flyback diodes.

24/24 sim blocks, netlist gate passing, 43 of 297 parts with footprints.
Parts:
- Q402, Q403, Q404, Q405, Q413, Q415, Q417: value 60V small-signal -> 2N7002BK; footprint (none) -> Package_TO_SOT_SMD:SOT-23; MPN (none) -> 2N7002BK

Commit message: Choose the power FETs, and draw DPAK parts with G-D-S symbols
Four part numbers for all sixteen power FETs, each against a retrieved
datasheet:
  SQD50P08-25L    reverse-battery P-FET, 31 mOhm max at -4.5 V
  IPD90N10S4-06   x8: negative clamp, metering, EGR bridge, injector
                  battery switches; 6.7 mOhm at 10 V, +/-20 V Vgs
                  (the logic-level -S4L-06 is +/-16 V, and every one of
                  these gates is driven from 12V_GATE)
  SQM85N15-19     x5: injector boost-side and low-side, 19 mOhm, TO-263
  DMN15H310SK3    boost switch, Rds(on) specified at a 4 V gate

Every FET was drawn as Q_NMOS_GSD, the SOT-23 order. DPAK and D2PAK are
G-D-S with the drain on the tab, so a TO-252 footprint on that symbol
puts the source on the tab. The power FETs now use Q_NMOS_GDS /
Q_PMOS_GDS: same pin positions, verified against the library, drains
on pin 2 in the netlist.

Checks that had run on placeholders now use the chosen parts: bootstrap
droop at 120 nC max (126 mV, was 60 nC), cranking duty including the
boost switch and sense drop (94.8% of 97.0%), and the pulldowns' 500 pF
Crss sizing against the worst chosen part (300 pF).

24/24 sim blocks, netlist gate passing, 58 of 297 parts with footprints.
Parts:
- removed Q401: 150V N-ch, logic-level, symbol Device:Q_NMOS_GSD
- removed Q408, Q410, Q412, Q414, Q416: 150V N-ch, 18A peak, symbol Device:Q_NMOS_GSD
- removed Q409, Q411: 60V N-ch, 18A, symbol Device:Q_NMOS_GSD
- added Q401: DMN15H310SK3, Package_TO_SOT_SMD:TO-252-2, symbol Device:Q_NMOS_GDS
- added Q408, Q410, Q412, Q414, Q416: SQM85N15-19, Package_TO_SOT_SMD:TO-263-2, symbol Device:Q_NMOS_GDS
- added Q409, Q411: IPD90N10S4-06, Package_TO_SOT_SMD:TO-252-2, symbol Device:Q_NMOS_GDS
Connections:
- net BOOST_100V: now also Q408.2 (D), Q410.2 (D)
- net GDRV_BOOST: now also Q401.1 (G)
- net HSA_BAT_GATE: now also Q409.1 (G)
- net HSA_BOOST_GATE: now also Q408.1 (G)
- net HSB_BAT_GATE: now also Q411.1 (G)
- net HSB_BOOST_GATE: now also Q410.1 (G)
- net INJ_A_03: now also Q408.3 (S), Q409.3 (S)
- net INJ_B_05: now also Q410.3 (S), Q411.3 (S)
- net INJ_LS1_73: now also Q412.2 (D)
- net INJ_LS2_29: now also Q416.2 (D)
- net INJ_LS3_07: now also Q414.2 (D)
- net ISNS_BOOST: now also Q401.3 (S)
- net ISNS_INJ_A_SENSE: now also Q412.3 (S), Q414.3 (S)
- net ISNS_INJ_B_SENSE: now also Q416.3 (S)
- net LS1_GATE: now also Q412.1 (G)
- net LS2_GATE: now also Q416.1 (G)
- net LS3_GATE: now also Q414.1 (G)
- net SW_BOOST: now also Q401.2 (D)
- net at D408.1 (K): now also Q409.2 (D)
- net at D410.1 (K): now also Q411.2 (D)

Commit message: Choose the diodes; the boost VDD clamp was 10 V over its pin rating
Part numbers for 27 diodes, each against a retrieved datasheet, applied
through one table (schlib.CHOSEN) keyed by symbol and class value, so
the class stays on the part as a field:
  VS-16EDH02HM3 x7   injector recirculation / blocking / freewheel
  VS-2EMH02HM3       boost diode
  VS-1EMH02HM3 x8    bootstrap and relay flyback
  VS-3ECH02HM3       metering freewheel
  SS20PH102HM3       negative-clamp backstop Schottky
  SMCJ43CA-HM3, SMAJ48CA-HE3, BZX84-C12-Q x2, BZX84-C13-Q, BZG03C36-HM3

The TPS40210 VDD clamp had been checked as an ideal 43.0 V source
behind 47 ohm. The real part in that class (40-46 V, +0.12 %/K, 45 ohm)
puts 61.9 V on a 52 V pin at 125 C, and its 40 V minimum conducts on
the load dump it was chosen to avoid. Now 220 ohm -- which the chosen
switch's gate charge allows -- and a 36 V zener: 46.6 V worst case with
tolerance, tempco and impedance, 33 mA on the dump. 39 V was tried
first; the transient_clamp rail table rejected it at 1.05x. The old
design stays as a pinned check.

TO-277A and SOT-23 zeners put the cathode on pad 3. gen_footprints.py
derives renumbered copies into lib/ecu25kva.pretty (new fp-lib-table).
The GATE_KILL zener, footprinted in the previous commit with the stock
SOT-23, had been reversed.

Left open as LOWV-CLAMP: the 15 zeners at 3.0 and 3.3 V. At tens of uA
a sub-5 V zener's knee is soft -- the datasheet allows 10 uA at 1 V --
and the model's sharp-knee zener hides it.

24/24 sim blocks, netlist gate passing, 74 of 297 parts with footprints.
Parts:
- C403: Note VDD bypass, INSIDE the 47 ohm. 100 V class anyway -- it is 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 -> VDD bypass, INSIDE the 220 ohm. 100 V class anyway -- it is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
- D401: value 150V 2A ultrafast -> VS-2EMH02HM3; footprint (none) -> Diode_SMD:D_SMA; Chosen (none) -> Vishay FRED Pt, 200 V, 2 A, trr 25 ns, AEC-Q101, SMA; Class (none) -> 150V 2A ultrafast; MPN (none) -> VS-2EMH02HM3
- D402: value 43V 1W -> BZG03C36-HM3; footprint (none) -> Diode_SMD:D_SMA; Chosen (none) -> Vishay BZG03C-M, 34-38 V at 10 mA, ZZ 40 ohm max, +0.06-0.1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; Class (none) -> 36V 3W; MPN (none) -> BZG03C36-HM3; Note Cathode to VDD. 43 V, not 39 V, so it stays OUT of conducti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 -> Cathode to VDD. Pulse 2a: 121 mA for 50 us, VDD 46.6 V wors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
- D403, D404, D405, D406: value 200V 1A fast -> VS-1EMH02HM3; footprint (none) -> Diode_SMD:D_SMA; Chosen (none) -> Vishay FRED Pt, 200 V, 1 A, 50 A surge, AEC-Q101, SMA; Class (none) -> 200V 1A fast; MPN (none) -> VS-1EMH02HM3
- D407: value 13V -> BZX84-C13-Q; footprint (none) -> ecu25kva:SOT-23_Zener_K1_A2; Chosen (none) -> Nexperia BZX84-Q, 12.4-14.1 V at 5 mA, AEC-Q101; Class (none) -> 13V; MPN (none) -> BZX84-C13-Q
- D408, D409, D410, D411, D412, D413, D414: value 150V 20A ultrafast -> VS-16EDH02HM3; Chosen (none) -> Vishay FRED Pt, 200 V, 16 A avg, 250 A surge, trr 32 ns, AE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; Class (none) -> 150V 20A ultrafast; MPN (none) -> VS-16EDH02HM3
- R405: value 47R 1W -> 220R 1W; Note The other half of the clamp. Small enough that 6.25 mA drop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 -> The other half of the clamp. Small enough that 3.8 mA (DMN1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

Commit message: Choose the 12V_GATE transistors; move half the pass dissipation out
The pass transistor was specified as a >=160 V DPAK NPN, but no such
datasheet could be retrieved (onsemi and Diodes refused the download).
The one that was, PZTA42-Q (300 V, SOT223, 104 K/W), may dissipate
0.43 W at a 105 C board -- and alone it would carry 0.44 W normally,
1.16 W into a short. Two 3.3k 2512 collector resistors now take half:
0.27 W in the transistor (Tj 133 C), 0.45 W per resistor shorted. The
cost is headroom: the rail must stay above 46.5 V, half its worst
droop. The 105 C board ambient is an assumption; the spec states none.

Current limit: PMBT3904-Q. SOT-23 bipolar order is B-E-C, so it uses a
new Q_NPN_BEC entry -- same positions as BCE, numbers swapped, verified
against the library.

24/24 sim blocks, netlist gate passing.
Parts:
- removed Q407: NPN small-signal, symbol Device:Q_NPN_BCE
- added Q407: PMBT3904-Q, Package_TO_SOT_SMD:SOT-23, symbol Device:Q_NPN_BEC
- added R428, R429: 5mOhm 2W 1%, symbol Device:R
- Q406: value NPN 160V, DPAK -> PZTA42-Q; footprint (none) -> Package_TO_SOT_SMD:SOT-223-3_TabPin2; Class AEC-Q101, Vceo >= 160 V, DPAK -> (none); MPN (none) -> PZTA42-Q; Note Pass transistor. 88 V across it at 5 mA is 0.44 W; into a s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 -> Pass transistor. Nexperia PZTA42-Q: 300 V, 100 mA, AEC-Q101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; Pins (none) -> SOT223 is B-C-E with the collector on the tab, which is thi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
- R416: value 56R -> 3.3k 2512; Note The limit's sense resistor. 0.28 V drop at the 5 mA design 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 -> Collector resistor, first of two. 16.5 V and 83 mW at 5 mA;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
- R417: value 470R -> 3.3k 2512; Note A pulldown to GROUND here would hold Vgs at minus the bank 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 -> Second of two.; Source supervisor.cir claim 6, referenced to SOURCE rather than to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 -> (none)
- R418: value 470R -> 56R; Note A pulldown to GROUND here would hold Vgs at minus the bank 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 -> The limit's sense resistor. 0.28 V drop at the 5 mA design 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; Source supervisor.cir claim 6, referenced to SOURCE rather than to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 -> (none)
- R419, R422: value 100k -> 470R; Note Bleed. With both high sides off and the low sides off, noth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 -> A pulldown to GROUND here would hold Vgs at minus the bank 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; Source (none) -> supervisor.cir claim 6, referenced to SOURCE rather than to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
- R421: value 470R -> 100k; Note A pulldown to GROUND here would hold Vgs at minus the bank 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 -> Bleed. With both high sides off and the low sides off, noth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; Source supervisor.cir claim 6, referenced to SOURCE rather than to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 -> (none)
- R423: Cost 21.3 mA per gate at 10 V; 1.28 W across all six -> (none); Note Largest standard value holding the gate under Vgs(th)=1.0 V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 -> A pulldown to GROUND here would hold Vgs at minus the bank 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; Source supervisor.cir claim 6; bom_requirements GATE-PULLDOWN -> supervisor.cir claim 6, referenced to SOURCE rather than to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
- R424: value 470R -> 100k; Cost 21.3 mA per gate at 10 V; 1.28 W across all six -> (none); Note Largest standard value holding the gate under Vgs(th)=1.0 V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 -> Bleed. With both high sides off and the low sides off, noth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; Source supervisor.cir claim 6; bom_requirements GATE-PULLDOWN -> (none)
- R426: value 5mOhm 2W 1% -> 470R; Cost (none) -> 21.3 mA per gate at 10 V; 1.28 W across all six; Note Bank A, cylinders 1 and 3 sharing one return. They fire 240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 -> Largest standard value holding the gate under Vgs(th)=1.0 V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; Power 1.62 W at peak, but ~1.25% duty per cylinder at 1500 rpm -> (none); Signal 90 mV at the 18 A peak, 50 mV at the 10 A hold -- too small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 -> (none); Source settled on this sheet -- docs/pinmap.md sec.1.6 asked for t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 -> supervisor.cir claim 6; bom_requirements GATE-PULLDOWN
- R427: value 5mOhm 2W 1% -> 470R; Cost (none) -> 21.3 mA per gate at 10 V; 1.28 W across all six; Note Bank B, cylinder 2 alone. Drawn as its own shunt rather tha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 -> Largest standard value holding the gate under Vgs(th)=1.0 V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; Power 1.62 W at peak, but ~1.25% duty per cylinder at 1500 rpm -> (none); Signal 90 mV at the 18 A peak, 50 mV at the 10 A hold -- too small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 -> (none); Source settled on this sheet -- docs/pinmap.md sec.1.6 asked for t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 -> supervisor.cir claim 6; bom_requirements GATE-PULLDOWN
Connections:
- net 12V_GATE: now also R418.2, Q407.2 (E); no longer R416.2
- net BASE_12V: now also Q407.3 (C)
- net BOOST_100V: now also R416.1; no longer Q406.2 (C)
- net GND: now also R421.2, R428.2, R429.2; no longer R419.2, R422.2, R423.2
- net HSA_BAT_GATE: now also R420.1; no longer R418.1
- net HSA_BOOST_GATE: now also R419.1; no longer R417.1
- net HSB_BAT_GATE: now also R423.1; no longer R421.1
- net HSB_BOOST_GATE: now also R422.1; no longer R420.1
- net INJ_A_03: now also R419.2, R420.2, R421.1; no longer R417.2, R418.2, R419.1
- net INJ_B_05: now also R422.2, R423.2, R424.1; no longer R420.2, R421.2, R422.1
- net ISNS_INJ_A_SENSE: now also R428.1; no longer R426.1
- net ISNS_INJ_B_SENSE: now also R429.1; no longer R427.1
- net LS1_GATE: now also R425.1; no longer R423.1
- net LS2_GATE: now also R427.1; no longer R425.1
- net LS3_GATE: now also R426.1; no longer R424.1
- net Q1E_12V: now also R418.1, Q407.1 (B); no longer R416.1
- new net: R416.2, R417.1
- new net Q1C_12V: Q406.2 (C), R417.2
Changed lines of the file:
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@@
       (effects (font (size 1.27 1.27)))
     )
-    (property "Value" "NPN 160V, DPAK" (id 1) (at 760.0 387.08 0)
-      (effects (font (size 1.27 1.27)))
-    )
-    (property "Footprint" "" (id 2) (at 760.0 382.0 0)
+    (property "Value" "PZTA42-Q" (id 1) (at 760.0 387.08 0)
+      (effects (font (size 1.27 1.27)))
+    )
+    (property "Footprint" "Package_TO_SOT_SMD:SOT-223-3_TabPin2" (id 2) (at 760.0 382.0 0)
       (effects (font (size 1.27 1.27)) hide)
     )
@@
       (effects (font (size 1.27 1.27)) hide)
     )
-    (property "Note" "Pass transistor. 88 V across it at 5 mA is 0.44 W; into a short, the limit below holds it to 11.6 mA and 1.16 W. Vceo >= 160 V -- the collector sits on a rail that reaches ~102 V, and a shorted output puts all of it across the part." (id 4) (at 760.0 382.0 0)
-      (effects (font (size 1.27 1.27)) hide)
-    )
-    (property "Class" "AEC-Q101, Vceo >= 160 V, DPAK" (id 5) (at 760.0 382.0 0)
+    (property "MPN" "PZTA42-Q" (id 4) (at 760.0 382.0 0)
+      (effects (font (size 1.27 1.27)) hide)
+    )
+    (property "Note" "Pass transistor. Nexperia PZTA42-Q: 300 V, 100 mA, AEC-Q101, SOT223, 104 K/W, Tj 150 C. Alone it would carry 88 V x 5 mA = 0.44 W, and 1.16 W into a short -- over the 0.43 W it may dissipate at a 105 C board. The collector resistors take half: 0.27 W normal, 0.24 W shorted." (id 5) (at 760.0 382.0 0)
+      (effects (font (size 1.27 1.27)) hide)
+    )
+    (property "Pins" "SOT223 is B-C-E with the collector on the tab, which is this symbol's numbering" (id 6) (at 760.0 382.0 0)
       (effects (font (size 1.27 1.27)) hide)
     )
@@
     (stroke (width 0) (type default))
   )
-  (label "BOOST_100V" (at 762.54 370.92 90)
+  (label "Q1C_12V" (at 762.54 370.92 90)
     (effects (font (size 1.27 1.27)) (justify left bottom))
   )
@@
     (effects (font (size 1.27 1.27)) (justify left bottom))
   )
-  (symbol (lib_id "Device:Q_NPN_BCE") (at 810.0 382.0 0) (unit 1)
+  (symbol (lib_id "Device:Q_NPN_BEC") (at 810.0 382.0 0) (unit 1)
     (in_bom yes) (on_board yes) (fields_autoplaced)
     (property "Reference" "Q407" (id 0) (at 810.0 376.92 0)
       (effects (font (size 1.27 1.27)))
     )
-    (property "Value" "NPN small-signal" (id 1) (at 810.0 387.08 0)
-      (effects (font (size 1.27 1.27)))
-    )
-    (property "Footprint" "" (id 2) (at 810.0 382.0 0)
+    (property "Value" "PMBT3904-Q" (id 1) (at 810.0 387.08 0)
+      (effects (font (size 1.27 1.27)))
+    )
+    (property "Footprint" "Package_TO_SOT_SMD:SOT-23" (id 2) (at 810.0 382.0 0)
       (effects (font (size 1.27 1.27)) hide)
     )
@@
       (effects (font (size 1.27 1.27)) hide)
     )
-    (property "Note" "Current limit. Conducts when the drop across the 56 ohm reaches one Vbe -- 0.65 V / 56 = 11.6 mA -- and steals the pass transistor's base drive. Without it a shorted 12V_GATE gets hFE x the full bias current from a 100 V rail." (id 4) (at 810.0 382.0 0)
+    (property "MPN" "PMBT3904-Q" (id 4) (at 810.0 382.0 0)
+      (effects (font (size 1.27 1.27)) hide)
+    )
+    (property "Pins" "SOT-23 bipolar order is B-E-C, hence the BEC symbol. 40 V: it never sees more than the ~13 V between the pass base and the output" (id 5) (at 810.0 382.0 0)
+      (effects (font (size 1.27 1.27)) hide)
+    )
+    (property "Note" "Current limit. Conducts when the drop across the 56 ohm reaches one Vbe -- 0.65 V / 56 = 11.6 mA -- and steals the pass transistor's base drive. Without it a shorted 12V_GATE gets hFE x the full bias current from a 100 V rail." (id 6) (at 810.0 382.0 0)
       (effects (font (size 1.27 1.27)) hide)
     )
@@
     (effects (font (size 1.27 1.27)) (justify left bottom))
   )
+  (label "BOOST_100V" (at 610.0 331.0 180)
+    (effects (font (size 1.27 1.27)) (justify left bottom))
+  )
+  (symbol (lib_id "Device:R") (at 650.0 331.0 90) (unit 1)
+    (in_bom yes) (on_board yes) (fields_autoplaced)
+    (property "Reference" "R416" (id 0) (at 650.0 325.92 0)
+      (effects (font (size 1.27 1.27)))
+    )
+    (property "Value" "3.3k 2512" (id 1) (at 650.0 336.08 0)
+      (effects (font (size 1.27 1.27)))
+    )
+    (property "Footprint" "" (id 2) (at 650.0 331.0 0)
+      (effects (font (size 1.27 1.27)) hide)
+    )
+    (property "Datasheet" "~" (id 3) (at 650.0 331.0 0)
+      (effects (font (size 1.27 1.27)) hide)
+    )
+    (property "Note" "Collector resistor, first of two. 16.5 V and 83 mW at 5 mA; 38 V and 0.44 W into a shorted output." (id 4) (at 650.0 331.0 0)
+      (effects (font (size 1.27 1.27)) hide)
+    )
+  )
+  (wire (pts (xy 610.0 331.0) (xy 646.19 331.0))
+    (stroke (width 0) (type default))
+  )
+  (symbol (lib_id "Device:R") (at 690.0 331.0 90) (unit 1)
+    (in_bom yes) (on_board yes) (fields_autoplaced)
+    (property "Reference" "R417" (id 0) (at 690.0 325.92 0)
+      (effects (font (size 1.27 1.27)))
+    )
+    (property "Value" "3.3k 2512" (id 1) (at 690.0 336.08 0)
+      (effects (font (size 1.27 1.27)))
+    )
+    (property "Footprint" "" (id 2) (at 690.0 331.0 0)
+      (effects (font (size 1.27 1.27)) hide)
+    )
+    (property "Datasheet" "~" (id 3) (at 690.0 331.0 0)
+      (effects (font (size 1.27 1.27)) hide)
+    )
+    (property "Note" "Second of two." (id 4) (at 690.0 331.0 0)
+      (effects (font (size 1.27 1.27)) hide)
+    )
+  )
+  (wire (pts (xy 653.81 331.0) (xy 686.19 331.0))
+    (stroke (width 0) (type default))
+  )
+  (wire (pts (xy 693.81 331.0) (xy 720.0 331.0))
+    (stroke (width 0) (type default))
+  )
+  (label "Q1C_12V" (at 720.0 331.0 0)
+    (effects (font (size 1.27 1.27)) (justify left bottom))
+  )
   (label "Q1E_12V" (at 640.0 412.0 180)
     (effects (font (size 1.27 1.27)) (justify left bottom))
@@
   (symbol (lib_id "Device:R") (at 680.0 412.0 90) (unit 1)
     (in_bom yes) (on_board yes) (fields_autoplaced)
-    (property "Reference" "R416" (id 0) (at 680.0 406.92 0)
+    (property "Reference" "R418" (id 0) (at 680.0 406.92 0)
       (effects (font (size 1.27 1.27)))
     )
@@
   (symbol (lib_id "Device:R") (at 225.0 95.0 0) (unit 1)
     (in_bom yes) (on_board yes) (fields_autoplaced)
-    (property "Reference" "R417" (id 0) (at 225.0 89.92 0)
+    (property "Reference" "R419" (id 0) (at 225.0 89.92 0)
       (effects (font (size 1.27 1.27)))
     )
@@
   (symbol (lib_id "Device:R") (at 315.0 95.0 0) (unit 1)
     (in_bom yes) (on_board yes) (fields_autoplaced)
-    (property "Reference" "R418" (id 0) (at 315.0 89.92 0)
+    (property "Reference" "R420" (id 0) (at 315.0 89.92 0)
       (effects (font (size 1.27 1.27)))
     )
@@
   (symbol (lib_id "Device:R") (at 420.0 123.0 0) (unit 1)
     (in_bom yes) (on_board yes) (fields_autoplaced)
-    (property "Reference" "R419" (id 0) (at 420.0 117.92 0)
+    (property "Reference" "R421" (id 0) (at 420.0 117.92 0)
       (effects (font (size 1.27 1.27)))
     )
@@
   (symbol (lib_id "Device:R") (at 555.0 95.0 0) (unit 1)
     (in_bom yes) (on_board yes) (fields_autoplaced)
-    (property "Reference" "R420" (id 0) (at 555.0 89.92 0)
+    (property "Reference" "R422" (id 0) (at 555.0 89.92 0)
       (effects (font (size 1.27 1.27)))
     )
@@
   (symbol (lib_id "Device:R") (at 645.0 95.0 0) (unit 1)
     (in_bom yes) (on_board yes) (fields_autoplaced)
-    (property "Reference" "R421" (id 0) (at 645.0 89.92 0)
+    (property "Reference" "R423" (id 0) (at 645.0 89.92 0)
       (effects (font (size 1.27 1.27)))
     )
@@
   (symbol (lib_id "Device:R") (at 750.0 123.0 0) (unit 1)
     (in_bom yes) (on_board yes) (fields_autoplaced)
-    (property "Reference" "R422" (id 0) (at 750.0 117.92 0)
+    (property "Reference" "R424" (id 0) (at 750.0 117.92 0)
       (effects (font (size 1.27 1.27)))
     )
@@
   (symbol (lib_id "Device:R") (at 84.92 213.0 0) (unit 1)
     (in_bom yes) (on_board yes) (fields_autoplaced)
-    (property "Reference" "R423" (id 0) (at 84.92 207.92 0)
+    (property "Reference" "R425" (id 0) (at 84.92 207.92 0)
       (effects (font (size 1.27 1.27)))
     )
@@
   (symbol (lib_id "Device:R") (at 254.92 213.0 0) (unit 1)
     (in_bom yes) (on_board yes) (fields_autoplaced)
-    (property "Reference" "R424" (id 0) (at 254.92000000000002 207.92 0)
+    (property "Reference" "R426" (id 0) (at 254.92000000000002 207.92 0)
       (effects (font (size 1.27 1.27)))
     )
@@
   (symbol (lib_id "Device:R") (at 424.92 213.0 0) (unit 1)
     (in_bom yes) (on_board yes) (fields_autoplaced)
-    (property "Reference" "R425" (id 0) (at 424.92 207.92 0)
+    (property "Reference" "R427" (id 0) (at 424.92 207.92 0)
       (effects (font (size 1.27 1.27)))
     )
@@
   (symbol (lib_id "Device:R") (at 200.0 260.0 0) (unit 1)
     (in_bom yes) (on_board yes) (fields_autoplaced)
-    (property "Reference" "R426" (id 0) (at 200.0 254.92 0)
+    (property "Reference" "R428" (id 0) (at 200.0 254.92 0)
       (effects (font (size 1.27 1.27)))
     )
@@
   (symbol (lib_id "Device:R") (at 500.0 260.0 0) (unit 1)
     (in_bom yes) (on_board yes) (fields_autoplaced)
-    (property "Reference" "R427" (id 0) (at 500.0 254.92 0)
-      (effects (font (size 1.27 1.27)))
-    )
+    (property "Reference" "R429" (id 0) (at 500.0 254.92 0)
+      (effects (font (size 1.27 1.27)))
+    )
