File: hw/injector.kicad_sch (KiCad schematic)
At the start: 86 parts, among them Q401 DMN15H310SK3, Q402 2N7002BK, Q403 2N7002BK, Q404 2N7002BK, Q405 2N7002BK, Q406 PZTA42-Q, Q407 PMBT3904-Q, Q408 SQM85N15-19, Q409 IPD90N10S4-06, Q410 SQM85N15-19, Q411 IPD90N10S4-06, Q412 SQM85N15-19, Q413 2N7002BK, Q414 SQM85N15-19, Q415 2N7002BK, Q416 SQM85N15-19, Q417 2N7002BK, U401 TPS40210, U402 AUIRS2181S, U403 AUIRS2181S, U404 AUIRS2181S, U405 AUIRS2181S, U406 INA181A1, U407 INA181A1

Commit message: Package every resistor and capacitor from the voltage across it
hw/assign_passives.py sizes all 188 chip R and C from a per-net table
of continuous and peak voltage (73.3 V pulse 2a, 104 V boost, bootstrap
domains riding on the bank nodes), against Vishay CRCW e3 resistor
ratings (Umax with 1.09x margin, power derated to 0.588x at a 105 C
board) and KEMET's automotive X7R waterfall (parsed by x-coordinate;
the text layout misreads its columns). schlib.place() applies the map
by ref and value; check_netlist fails on any unpackaged R or C.

Found along the way:
- 4.7 uF at 100 V is not in automotive X7R. The EMI filter C1, buck
  input and boost input are now 2 x 2.2 uF 100 V 1210; emi_filter.cir
  models the pair and its cold corner was re-pinned (0.6 dB worse).
- The twelve 470 ohm gate pulldowns need 2010: 0.31 W each at 100%
  duty. Recorded; 1k may now be possible against the real Crss.
- Local labels at 180 degrees were justified in the wrong frame on
  every sheet -- the bug fixed for hierarchical labels earlier -- so
  their text sat across their own wire. Fixed in schlib.label().

Internal nodes whose voltage matters now carry names (FB_BOOST_MID,
CAN1_SPLIT, ...); auto-names like Net-(R407-Pad2) move when parts are
added ahead of them.

24/24 sim blocks, netlist gate passing, 264 of 302 parts footprinted.
Parts:
- added C419: 100nF, Capacitor_SMD:C_0603_1608Metric, symbol Device:C
- C402: value 4.7uF 100V -> 2.2uF 100V; footprint (none) -> Capacitor_SMD:C_1210_3225Metric; Note Input bulk. 100 V class because it sits on VBAT_PROT, which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 -> Input bulk, one of two -- see the next part.
- C403: value 1uF 100V -> 2.2uF 100V; footprint (none) -> Capacitor_SMD:C_1210_3225Metric; Note VDD bypass, INSIDE the 220 ohm. 100 V class anyway -- it is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 -> Input bulk. 100 V class because it sits on VBAT_PROT, which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
- C404: value 330pF -> 1uF 100V; footprint (none) -> Capacitor_SMD:C_1206_3216Metric; Note The datasheet's own reference point is 182k/330pF = 300 kHz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 -> VDD bypass, INSIDE the 220 ohm. 100 V class anyway -- it is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; Source TPS40210-Q1 -- with 365k to VDD this sets 150 kHz -> (none)
- C405: value 100nF -> 330pF; footprint (none) -> Capacitor_SMD:C_0603_1608Metric; Note Soft start. Also the overcurrent retry timer -- the part di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 -> The datasheet's own reference point is 182k/330pF = 300 kHz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; Source (none) -> TPS40210-Q1 -- with 365k to VDD this sets 150 kHz
- C406: value 1uF -> 100nF; footprint (none) -> Capacitor_SMD:C_0603_1608Metric; Note The internal 8 V regulator's reservoir, and the gate driver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 -> Soft start. Also the overcurrent retry timer -- the part di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; Source TPS40210-Q1 pin table -- 1 uF from BP to GND -> (none)
- C407: value 6.8nF -> 1uF; footprint (none) -> Capacitor_SMD:C_0805_2012Metric; Note Zero at 2.3 kHz, below the 17.3 kHz right-half-plane zero a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 -> The internal 8 V regulator's reservoir, and the gate driver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; Source (none) -> TPS40210-Q1 pin table -- 1 uF from BP to GND
- C408: value 1uF 25V -> 6.8nF; footprint (none) -> Capacitor_SMD:C_0603_1608Metric; Note Bootstrap capacitor. A 60 nC gate over the 38 us peak phase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 -> Zero at 2.3 kHz, below the 17.3 kHz right-half-plane zero a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
- C409, C411, C413, C415: footprint (none) -> Capacitor_SMD:C_0805_2012Metric; Note VCC bypass, at the pin. -> Bootstrap capacitor. A 60 nC gate over the 38 us peak phase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
- C410, C412, C414: footprint (none) -> Capacitor_SMD:C_0805_2012Metric; Note Bootstrap capacitor. A 60 nC gate over the 38 us peak phase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 -> VCC bypass, at the pin.
- C416: value 10uF 25V -> 1uF 25V; footprint (none) -> Capacitor_SMD:C_0805_2012Metric; Note Holds the rail through each driver's gate-charge pulse. -> VCC bypass, at the pin.
- C417: value 100nF -> 10uF 25V; footprint (none) -> Capacitor_SMD:C_1206_3216Metric; Note At the VS pin. -> Holds the rail through each driver's gate-charge pulse.
- C418: footprint (none) -> Capacitor_SMD:C_0603_1608Metric
- R401, R405, R416, R417, R428, R429: footprint (none) -> Resistor_SMD:R_2512_6332Metric
- R402: footprint (none) -> Resistor_SMD:R_1206_3216Metric
- R403, R404, R406, R408, R409, R410, R411, R412, R413, R414, R415, R418: footprint (none) -> Resistor_SMD:R_0603_1608Metric
- R407, R421, R424: footprint (none) -> Resistor_SMD:R_0805_2012Metric
- R419, R420, R422, R423, R425, R426, R427: footprint (none) -> Resistor_SMD:R_2010_5025Metric
Connections:
- net 12V_GATE: now also C410.1, C412.1, C414.1, C417.1; no longer C409.1, C411.1, C413.1, C415.1
- net 3V3_MCU: now also C419.1; no longer C417.1
- net BP_BOOST: now also C407.1; no longer C406.1
- net FB_BOOST: now also C408.2; no longer C407.2
- net GND: now also C407.2, C410.2, C412.2, C414.2, C419.2; no longer C409.2, C411.2, C413.2, C415.2
- net INJ_A_03: now also C409.2, C411.2; no longer C408.2, C410.2
- net INJ_B_05: now also C413.2, C415.2; no longer C412.2, C414.2
- net RC_BOOST: now also C405.1; no longer C404.1
- net SS_BOOST: now also C406.1; no longer C405.1
- net UA1_VB: now also C409.1; no longer C408.1
- net UA2_VB: now also C411.1; no longer C410.1
- net UB1_VB: now also C413.1; no longer C412.1
- net UB2_VB: now also C415.1; no longer C414.1
- net VBAT_PROT: now also C403.1
- net VDD_BOOST: now also C404.1; no longer C403.1
- net FB_BOOST_MID: now reaches R407.2, R408.1
- net BIAS_12V_MID: now reaches R414.2, R415.1
- net COMP_RC_BOOST: now reaches R409.2
- net COMP_RC_BOOST: now also C408.1; no longer C407.1
- net Q1C_MID: now reaches R416.2, R417.1

Commit message: Move the injector and EGR supply onto pins 04 and 06 (POWER-PATH)
Every high-current load drew through pin 21, whose reverse FET was
sized for 5 A and whose EMI filter never stated a DC current. Pin 04
now feeds VBAT_INJ (the injector hold switches and the boost power
stage), and pin 06 feeds VBAT_EGR (the EGR bridge). Each is fused 10 A
in the loom and has its own SMCJ43CA TVS, SQM120P10-10m1L reverse
P-FET (passive gate, as Q1), SS20PH102HM3 backstop and 2 x 2.2 uF.
Pin 21 keeps the buck, the relays, the metering freewheel and the
boost controller's VDD.

The pin-21 FET could not simply be copied: at the EGR's 6.4 A stall it
would pass its junction limit on a 105 C board. The new part, from
Vishay doc 76943 Rev. A, runs at Tj 139 C (155 C cranking) on the EGR
rail and 117 C on the injector rail. The new block power_path.cir
holds those figures as 18 checks. check_netlist now fails unless each
rail leaves its own FET for its own loads and VBAT_PROT reaches
neither power stage.

The sheets are generated against KiCad 7.0.11's symbol library, which
regenerates an unchanged sheet identically. KiCad 10's library would
have rewritten every embedded symbol.

Gates: 25/25 blocks; connectivity OK with the same 2 open items; 333
components, 314 with footprints; 208 passives packaged. The questions
put to the owner -- the split, the reverse protection, what stays on
pin 21, and the KiCad/ngspice choices -- are in decisions-log.md
sections 5 and 6. The spec, the BOM requirements, the handbook, status
and the handoff are updated to match, and the bible is rebuilt (333
pages).
Parts:
- C403: Note Input bulk. 100 V class because it sits on VBAT_PROT, which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 -> Input bulk. 100 V class because it sits on VBAT_INJ, which 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
Connections:
- net VBAT_PROT: no longer C402.1, C403.1, D408.2 (A), D410.2 (A), L401.1
- new net VBAT_INJ: C402.1, C403.1, D408.2 (A), D410.2 (A), L401.1
Changed lines of the file:
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@@
     (effects (font (size 2.0 2.0)) (justify left))
   )
-  (hierarchical_label "VBAT_PROT" (shape input) (at 40.0 455.0 0)
+  (hierarchical_label "VBAT_INJ" (shape input) (at 40.0 455.0 0)
     (effects (font (size 1.27 1.27)) (justify left))
   )
@@
       (effects (font (size 1.27 1.27)) hide)
     )
-    (property "Note" "Input bulk. 100 V class because it sits on VBAT_PROT, which reaches 73.3 V on pulse 2a -- the same rule every other battery-connected part on this board is held to." (id 4) (at 75.0 473.0 0)
+    (property "Note" "Input bulk. 100 V class because it sits on VBAT_INJ, which reaches 73.3 V on pulse 2a -- the same rule every other battery-connected part on this board is held to." (id 4) (at 75.0 473.0 0)
       (effects (font (size 1.27 1.27)) hide)
     )
@@
     (stroke (width 0) (type default))
   )
-  (hierarchical_label "VBAT_PROT" (shape input) (at 342.54 46.11 90)
+  (hierarchical_label "VBAT_INJ" (shape input) (at 342.54 46.11 90)
     (effects (font (size 1.27 1.27)) (justify left))
   )
@@
     (stroke (width 0) (type default))
   )
-  (hierarchical_label "VBAT_PROT" (shape input) (at 672.54 46.11 90)
+  (hierarchical_label "VBAT_INJ" (shape input) (at 672.54 46.11 90)
     (effects (font (size 1.27 1.27)) (justify left))
   )

Commit message: Build BOOST-SLOPE: the boost controller runs from its own output, 150 uH
TPS40210-Q1's slope compensation scales with VDD, and on the battery
VDD is about 5 V while cranking: Equation 9 failed there. VDD now comes
from a follower off the 100 V output, 34.3-45.0 V. It is 12V_GATE's
circuit with a BZG03C39 reference: PZTA42-Q pass, 2x3.3k collector
resistors, and a PMBT3904-Q limiting at 11.6 mA, because a follower off
a 100 V rail burns if its output shorts. The battery path starts the
part only: 180 ohm (was 220), the 36 V clamp moved onto VDD_BAT, then
an SS20PH102 Schottky so the follower cannot push ~0.1 A back into the
battery rail. Start-up VDD at 6 V is 4.77 V against the 4.5 V threshold.

L401 is Wurth 7447709151, 150 uH, not the approved 100 uH. Two
questions to the owner settled it (decisions log 8). The suggested
10x10x4 mm part saturates at 1.4 A and cannot work. The 12x12 mm
150 uH, in the same footprint, beats 100 uH on stability and
saturation. Sense is 62 mOhm.

Equation 9 holds at the worst corner by 1.12x: VDD 34.3 V, L -20%,
6 V in, and the oscillator at -20%. Its RC returns to VDD, and TI
specifies -20%/+7% across VDD; that corner would have failed the
100 uH design outright. Equation 49 holds by 1.05x. The current limit
is 1.94-2.90 A: past L401's 10% saturation by 7%, under its 30% point
by 14%. Stated: start-up margin is 17 mV at twice the FET's typical
gate charge, and the first milliseconds of a cranking start still run
on the battery's shallow ramp.

Datasheets retrieved and read: TPS40210-Q1 SLVS861F, Wurth 7447709101
and 7447709151, 7447714151 (the 10x10x4 part), Vishay SS20PH102 and
BZG03C-M 86574. The decisions log, BOM requirements, status and handoff
are updated; the handbook and the bible (360 pages) are regenerated.

Gates: 25/25 blocks, connectivity OK, 362 components, 345 with
footprints, 230 passives.
Parts:
- added D415: BZG03C39-HM3, Diode_SMD:D_SMA, symbol Device:D_Zener
- added D416: SS20PH102HM3, ecu25kva:TO-277A_K1_A2, symbol Device:D_Schottky
- added Q418: PZTA42-Q, Package_TO_SOT_SMD:SOT-223-3_TabPin2, symbol Device:Q_NPN_BCE
- added Q419: PMBT3904-Q, Package_TO_SOT_SMD:SOT-23, symbol Device:Q_NPN_BEC
- added R430, R431: 7.5k, Resistor_SMD:R_1210_3225Metric, symbol Device:R
- added R432, R433: 3.3k 2512, Resistor_SMD:R_2512_6332Metric, symbol Device:R
- added R434: 56R, Resistor_SMD:R_0603_1608Metric, symbol Device:R
- C404: Note VDD bypass, INSIDE the 220 ohm. 100 V class anyway -- it is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 -> VDD bypass. 100 V class anyway -- a Schottky and a resistor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
- D402: Note Cathode to VDD. Pulse 2a: 121 mA for 50 us, VDD 46.6 V wors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 -> On the battery side of the Schottky, so it clamps the start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
- L401: value 330uH 3A -> 7447709151; footprint (none) -> Inductor_SMD:L_Wuerth_WE-PD-Typ-LS; Chosen (none) -> Wurth WE-PD 1210, 150 uH, IR 2.1 A, Isat 2.7 A (10%) / 3.3 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; Class (none) -> 150uH; DCR <=0.2 ohm -- 0.2 W at the 1 A cranking corner -> 200 mOhm max -- 0.2 W at the 1 A cranking corner; MPN (none) -> 7447709151; Note At 150 kHz and 13.5 V in, ripple is 0.24 A on a 0.44 A aver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 -> 150 uH, not the 330 uH first drawn (no SMD part) or the 100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; Source sized here -- boost_converter.cir models the converter as a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 -> run_sim boost_converter, BOOST-SLOPE -- decisions log 2b an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
- R402: value 82mOhm 1% -> 62mOhm 1%; Note Current limit lands in 1.46-2.20 A across the threshold's o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 -> Inside TI's 80% stability ceiling by 1.12x at the worst cor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; Power 1.06^2 * 82 mOhm = 92 mW -> 1.18^2 * 62 mOhm = 86 mW; Source TPS40210-Q1 Table 6.5, VISNS(oc) 120-180 mV -> TPS40210-Q1 Table 6.5, VISNS(oc) 120-180 mV; Eq. 9 and Eq. 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
- R405: value 220R 1W -> 180R 1W; Note The other half of the clamp. Small enough that 3.8 mA (DMN1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 -> START-UP feed only since BOOST-SLOPE: the follower off the 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
Connections:
- net BOOST_100V: now also R430.1, R432.1
- net GND: now also D415.2 (A)
- net VDD_BOOST: now also D416.1 (K), Q419.2 (E), R434.2; no longer D402.1 (K), R405.2
- new net VDD_BAT: D402.1 (K), D416.2 (A), R405.2
- new net VDD_Q1C: Q418.2 (C), R433.2
- new net VDD_Q1C_MID: R432.2, R433.1
- new net VDD_Q1E: Q418.3 (E), Q419.1 (B), R434.1
- new net VDD_REF: D415.1 (K), Q418.1 (B), Q419.3 (C), R431.2
- new net VDD_REF_MID: R430.2, R431.1
Other:
- note added: "VDD FOLLOWER (BOOST-SLOPE) -- the TPS40210-Q1 runs from its own output once started: VDD 34.3-45.0 V. The battery path only starts it."
