File: hw/injector.kicad_sch (KiCad schematic)
At the start: 96 parts, among them Q401 DMN15H310SK3, Q402 2N7002BK, Q403 2N7002BK, Q404 2N7002BK, Q405 2N7002BK, Q406 PZTA42-Q, Q407 PMBT3904-Q, Q408 SQM85N15-19, Q409 IPD90N10S4-06, Q410 SQM85N15-19, Q411 IPD90N10S4-06, Q412 SQM85N15-19, Q413 2N7002BK, Q414 SQM85N15-19, Q415 2N7002BK, Q416 SQM85N15-19, Q417 2N7002BK, Q418 PZTA42-Q, Q419 PMBT3904-Q, U401 TPS40210, U402 AUIRS2181S, U403 AUIRS2181S, U404 AUIRS2181S, U405 AUIRS2181S, U406 INA181A1, U407 INA181A1

Commit message: Choose the three non-ceramic capacitors; the boost tank becomes a 2-can stack
C313: KEMET T599 150 uF polymer tantalum plus a 22 mOhm series resistor
(R306). No datasheet gives an ESR minimum, so the resistor is PDN-BULK's
floor; the pair is 21.8-72.2 mOhm and mcu_pdn passes both ends at 96 uF.

C211: Chemi-Con HXC 47 uF 63 V hybrid polymer. sensor_rail now runs its
worst corners at 26.3 uF (tolerance plus end of life) and passes.

C401 + C420: two HXC 82 uF 80 V in series, the owner's choice over one
160 V wet can, because no part rated above 100 V publishes a cold ESR.
Worst stack ESR 224 mOhm aged at -55 C; 18 A in 45 us at -40 C. The sims
run 41 uF, every check uses the 85.1 V worst low point, and the 22k bleed
is split 2 x 11k to balance the cans. Decisions log section 9.
Parts:
- added C420: HHXC800ARA820MJC5G, Capacitor_SMD:CP_Elec_10x12.5, symbol Device:C_Polarized
- added R435: 11k 1W, Resistor_SMD:R_2512_6332Metric, symbol Device:R
- C401: value 47uF 150V -> HHXC800ARA820MJC5G; footprint (none) -> Capacitor_SMD:CP_Elec_10x12.5; Chosen (none) -> Chemi-Con HXC hybrid polymer, 82 uF, 80 V, 10 x 12.5 mm, 28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; Class (none) -> 82uF 80V; MPN (none) -> HHXC800ARA820MJC5G; Note The converter cannot deliver 18 A -- it delivers a trickle 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 -> TOP of a two-can stack with C420 -- 41 uF, 160 V. The conve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; Source boost_converter.cir Ca -> boost_converter.cir Ca; decisions log 9; Vr 150 V class: 100 V setpoint plus the recirculation bump, sa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 -> (none); Why two (none) -> No capacitor rated above 100 V publishes a cold ESR. These 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
- R401: value 22k 1W -> 11k 1W; Also (none) -> Balances the stack: with R435 it holds each can at 52.4 V w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; Cost 455 mW burned continuously whenever the rail is up -> 250 mW each, 455 mW the pair; Note The charger regulates from BELOW only -- 50 mA while the ra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 -> Half of the 22k bleed, across C401. The charger regulates f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; Sizing one 100 uC event is 2.14 V on 47 uF; above setpoint the cha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 -> (none); Source boost_converter.cir arrangement C; bom_requirements BOOST-BLEED -> boost_converter.cir arrangement C; bom_requirements BOOST-BLEED; decisions log 9
Connections:
- net GND: now also C420.2, R435.2; no longer C401.2, R401.2
- new net BOOST_MID: C401.2, C420.1, R401.2, R435.1

Commit message: Draw the four missing land patterns: SMPD, WE-PD 1050, DGX0019A, DDA0008J
Each comes from the maker's recommended layout, written in KiCad 7
format by gen_footprints.py:
- Vishay SMPD (doc 95604) for D408-D414: tab = cathode = pad 1, both
  leads = anode = pad 2, matching Device:D
- Wurth WE-PD 1050 for L201: 3.5 x 2.0 pads, 7.0 inner gap
- TI DGX0019A for U203: 0.5 mm pitch, position 16 empty
- TI DDA0008J for U204-U206: 2.95 x 4.9 thermal copper with a
  2.6 x 3.2 solder-mask-defined opening, which no stock variant has

The installed KiCad 10 stock library is newer than KiCad 7 can open, so
the two renumbered stock copies are skipped rather than rewritten.
363 of 365 components now have a footprint; J1001 (Bosch drawing) and
D806 (trip-loop clamp) remain.
Parts:
- D408, D409, D410, D411, D412, D413, D414: footprint (none) -> ecu25kva:Vishay_SMPD_TO-263AC_K1_A2; Chosen Vishay FRED Pt, 200 V, 16 A avg, 250 A surge, trr 32 ns, AEC-Q101. SMPD (TO-263AC), cathode on the tab -- no KiCad 7 footprint, drawn in phase 3 -> Vishay FRED Pt, 200 V, 16 A avg, 250 A surge, trr 32 ns, AEC-Q101. SMPD (TO-263AC), cathode on the tab -- land pattern drawn from Vishay doc 95604 (gen_footprints.py)
Changed lines of the file:
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@@
       (effects (font (size 1.27 1.27)))
     )
-    (property "Footprint" "" (id 2) (at 342.54 63.92 0)
+    (property "Footprint" "ecu25kva:Vishay_SMPD_TO-263AC_K1_A2" (id 2) (at 342.54 63.92 0)
       (effects (font (size 1.27 1.27)) hide)
     )
@@
       (effects (font (size 1.27 1.27)) hide)
     )
-    (property "Chosen" "Vishay FRED Pt, 200 V, 16 A avg, 250 A surge, trr 32 ns, AEC-Q101. SMPD (TO-263AC), cathode on the tab -- no KiCad 7 footprint, drawn in phase 3" (id 6) (at 342.54 63.92 0)
+    (property "Chosen" "Vishay FRED Pt, 200 V, 16 A avg, 250 A surge, trr 32 ns, AEC-Q101. SMPD (TO-263AC), cathode on the tab -- land pattern drawn from Vishay doc 95604 (gen_footprints.py)" (id 6) (at 342.54 63.92 0)
       (effects (font (size 1.27 1.27)) hide)
     )
@@
       (effects (font (size 1.27 1.27)))
     )
-    (property "Footprint" "" (id 2) (at 390.0 119.0 0)
+    (property "Footprint" "ecu25kva:Vishay_SMPD_TO-263AC_K1_A2" (id 2) (at 390.0 119.0 0)
       (effects (font (size 1.27 1.27)) hide)
     )
@@
       (effects (font (size 1.27 1.27)) hide)
     )
-    (property "Chosen" "Vishay FRED Pt, 200 V, 16 A avg, 250 A surge, trr 32 ns, AEC-Q101. SMPD (TO-263AC), cathode on the tab -- no KiCad 7 footprint, drawn in phase 3" (id 6) (at 390.0 119.0 0)
+    (property "Chosen" "Vishay FRED Pt, 200 V, 16 A avg, 250 A surge, trr 32 ns, AEC-Q101. SMPD (TO-263AC), cathode on the tab -- land pattern drawn from Vishay doc 95604 (gen_footprints.py)" (id 6) (at 390.0 119.0 0)
       (effects (font (size 1.27 1.27)) hide)
     )
@@
       (effects (font (size 1.27 1.27)))
     )
-    (property "Footprint" "" (id 2) (at 672.54 63.92 0)
+    (property "Footprint" "ecu25kva:Vishay_SMPD_TO-263AC_K1_A2" (id 2) (at 672.54 63.92 0)
       (effects (font (size 1.27 1.27)) hide)
     )
@@
       (effects (font (size 1.27 1.27)) hide)
     )
-    (property "Chosen" "Vishay FRED Pt, 200 V, 16 A avg, 250 A surge, trr 32 ns, AEC-Q101. SMPD (TO-263AC), cathode on the tab -- no KiCad 7 footprint, drawn in phase 3" (id 6) (at 672.54 63.92 0)
+    (property "Chosen" "Vishay FRED Pt, 200 V, 16 A avg, 250 A surge, trr 32 ns, AEC-Q101. SMPD (TO-263AC), cathode on the tab -- land pattern drawn from Vishay doc 95604 (gen_footprints.py)" (id 6) (at 672.54 63.92 0)
       (effects (font (size 1.27 1.27)) hide)
     )
@@
       (effects (font (size 1.27 1.27)))
     )
-    (property "Footprint" "" (id 2) (at 720.0 119.0 0)
+    (property "Footprint" "ecu25kva:Vishay_SMPD_TO-263AC_K1_A2" (id 2) (at 720.0 119.0 0)
       (effects (font (size 1.27 1.27)) hide)
     )
@@
       (effects (font (size 1.27 1.27)) hide)
     )
-    (property "Chosen" "Vishay FRED Pt, 200 V, 16 A avg, 250 A surge, trr 32 ns, AEC-Q101. SMPD (TO-263AC), cathode on the tab -- no KiCad 7 footprint, drawn in phase 3" (id 6) (at 720.0 119.0 0)
+    (property "Chosen" "Vishay FRED Pt, 200 V, 16 A avg, 250 A surge, trr 32 ns, AEC-Q101. SMPD (TO-263AC), cathode on the tab -- land pattern drawn from Vishay doc 95604 (gen_footprints.py)" (id 6) (at 720.0 119.0 0)
       (effects (font (size 1.27 1.27)) hide)
     )
@@
       (effects (font (size 1.27 1.27)))
     )
-    (property "Footprint" "" (id 2) (at 146.54 156.0 0)
+    (property "Footprint" "ecu25kva:Vishay_SMPD_TO-263AC_K1_A2" (id 2) (at 146.54 156.0 0)
       (effects (font (size 1.27 1.27)) hide)
     )
@@
       (effects (font (size 1.27 1.27)) hide)
     )
-    (property "Chosen" "Vishay FRED Pt, 200 V, 16 A avg, 250 A surge, trr 32 ns, AEC-Q101. SMPD (TO-263AC), cathode on the tab -- no KiCad 7 footprint, drawn in phase 3" (id 6) (at 146.54 156.0 0)
+    (property "Chosen" "Vishay FRED Pt, 200 V, 16 A avg, 250 A surge, trr 32 ns, AEC-Q101. SMPD (TO-263AC), cathode on the tab -- land pattern drawn from Vishay doc 95604 (gen_footprints.py)" (id 6) (at 146.54 156.0 0)
       (effects (font (size 1.27 1.27)) hide)
     )
@@
       (effects (font (size 1.27 1.27)))
     )
-    (property "Footprint" "" (id 2) (at 316.54 156.0 0)
+    (property "Footprint" "ecu25kva:Vishay_SMPD_TO-263AC_K1_A2" (id 2) (at 316.54 156.0 0)
       (effects (font (size 1.27 1.27)) hide)
     )
@@
       (effects (font (size 1.27 1.27)) hide)
     )
-    (property "Chosen" "Vishay FRED Pt, 200 V, 16 A avg, 250 A surge, trr 32 ns, AEC-Q101. SMPD (TO-263AC), cathode on the tab -- no KiCad 7 footprint, drawn in phase 3" (id 6) (at 316.54 156.0 0)
+    (property "Chosen" "Vishay FRED Pt, 200 V, 16 A avg, 250 A surge, trr 32 ns, AEC-Q101. SMPD (TO-263AC), cathode on the tab -- land pattern drawn from Vishay doc 95604 (gen_footprints.py)" (id 6) (at 316.54 156.0 0)
       (effects (font (size 1.27 1.27)) hide)
     )
@@
       (effects (font (size 1.27 1.27)))
     )
-    (property "Footprint" "" (id 2) (at 486.54 156.0 0)
+    (property "Footprint" "ecu25kva:Vishay_SMPD_TO-263AC_K1_A2" (id 2) (at 486.54 156.0 0)
       (effects (font (size 1.27 1.27)) hide)
     )
@@
       (effects (font (size 1.27 1.27)) hide)
     )
-    (property "Chosen" "Vishay FRED Pt, 200 V, 16 A avg, 250 A surge, trr 32 ns, AEC-Q101. SMPD (TO-263AC), cathode on the tab -- no KiCad 7 footprint, drawn in phase 3" (id 6) (at 486.54 156.0 0)
-      (effects (font (size 1.27 1.27)) hide)
-    )
+    (property "Chosen" "Vishay FRED Pt, 200 V, 16 A avg, 250 A surge, trr 32 ns, AEC-Q101. SMPD (TO-263AC), cathode on the tab -- land pattern drawn from Vishay doc 95604 (gen_footprints.py)" (id 6) (at 486.54 156.0 0)
+      (effects (font (size 1.27 1.27)) hide)
+    )
