File: hw/speed_inputs.kicad_sch (KiCad schematic)
At the start: 0 parts

Commit message: Draw the speed inputs; the crank clamps are chosen by leakage, not drop
Sheet 8 of 10. Two engine-position inputs whose front ends have nothing
in common because their sensors have nothing in common.

CRANK. vr_conditioner.cir models the comparator as SW(Vt=0 Vh=0.2) -- an
ideal element with no input current, no supply and no clamp. Turning that
into parts is what the sheet does:

  Vwindow = Vswing * Rth / (Rth + Rfb)
          = 3.3 * 4489 / (4489 + 33000) = 0.395 V, i.e. +/-198 mV

against the +/-200 mV the block modelled, from E24 values. That matters
because the block's own tolerance section found the failure point sits
almost exactly AT Vh: a cranking signal that never leaves the window
cannot flip the comparator whatever its amplitude.

The floating coil is biased to mid-rail rather than level-shifted, which
removes the constraint that usually makes a zero-cross detector hard --
no part is needed whose common-mode range includes ground.

CAM. Drawn as cam_frontend.cir validates it. One 16k resistor turns spec
sec.4's literal 'pull-up to 5V_SENSOR' into the same 10k/16k divider the
ratiometric channels use, which is what keeps a 5 V swing off PTB3.
pinmap sec.4 asked for that check by name before this sheet was drawn;
it is now closed there.

NEW FINDING, from the parts rather than the pins. Every clamp earlier in
this project was chosen by forward drop -- the negative-clamp Schottky's
0.547 V at 15 A decomposes into junction and bulk terms, and that
decomposition ruled out paralleling junction devices. These four conduct
only on a fault into a 4.7k resistor already doing the limiting, so what
matters is what they do when OFF. Schottky leakage at 125 C (~200 uA)
across the input's 4.489k Thevenin is 0.90 V of offset -- 4.5x the whole
hysteresis window. The comparator latches and a running engine has no
speed signal. BAV199-class low-leakage silicon gives under 4.5 mV.
vr_conditioner.cir cannot see this: its comparator has no input network,
so no clamp, no leak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
Parts:
- added C1, C2: 1nF, symbol Device:C
- added C3: 100nF, symbol Device:C
- added C4: 1uF, symbol Device:C
- added C5: 22nF, symbol Device:C
- added D1: SMAJ48CA, symbol Device:D_TVS
- added D2, D4: BAV199 (upper half), symbol Device:D
- added D3, D5: BAV199 (lower half), symbol Device:D
- added D6: 3.3V, symbol Device:D_Zener
- added R1, R2: 4.7k, symbol Device:R
- added R3, R4: 100k, symbol Device:R
- added R5: 33k, symbol Device:R
- added R6, R7: 2.2k, symbol Device:R
- added R8: 10k, symbol Device:R
- added R9: 16k, symbol Device:R
- added U1: COMPARATOR_GENERIC, symbol ecu25kva:COMPARATOR_GENERIC
Connections:
- new net 3V3_MCU: C3.1, D2.1 (K), D4.1 (K), R6.1, U1.5 (V+)
- new net CAM_EDGE: C5.1, D6.1 (K), R8.2, R9.1
- new net CRANK_EDGE: R5.2, U1.1 (OUT)
- new net CRANK_HI_52: D1.2 (A2), R1.1
- new net CRANK_LO_74: D1.1 (A1), R2.1
- new net EXC_CAM_45: R8.1
- new net GND: C1.2, C2.2, C3.2, C4.2, C5.2, D3.2 (A), D5.2 (A), D6.2 (A), R7.2, R9.2, U1.4 (V-)
- new net VR_BIAS: C1.1, C2.1, C4.1, D2.2 (A), D3.1 (K), D4.2 (A), D5.1 (K), R1.2, R2.2, R3.1, R3.2, R4.1, R4.2, R5.1, R6.2, R7.1, U1.2 (IN-), U1.3 (IN+)
Other:
- note added: "CAM -- digital Hall, ECU pins 45 / 46 / 44 -> PTB3 (FTM1_CH1). CORRECTS the front-end spec sec.4 specifies literally"
- note added: "CLAMP LEAKAGE IS THE BINDING SPEC, WHICH INVERTS THE RULE THIS PROJECT USED ON THE POWER PATH. Every earlier clamp on this board was chosen for forward drop -- the negative-clamp Schottky's 0.547 V at 15 A decomposes into junction and bulk terms and that decomposition is what ruled out paralleling junction devices. Here the forward drop does not matter at all: these diodes conduct only on a fault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"
- note added: "CRANK -- variable reluctance, ECU pins 52 / 74, shield 30 -> zero-cross comparator -> PTB2 (FTM1_CH0)"
- note added: "ECU pin 30 -- crank sensor shield, terminated at THIS end only. Grounding both ends makes the shield a second conductor between two grounds that differ by the injector return current, and that current then flows down the shield around the pair it is there to protect."
- note added: "PARTS NOT CHOSEN ON THIS SHEET: the comparator (COMPARATOR_GENERIC -- placeholder pins, no footprint) and the cam Hall sensor itself, which is U8 on the unknowns register and needs the machine. The comparator's requirement is unusually easy, and deliberately so: biasing the floating coil to VR_BIAS means the inputs never leave mid-rail, so no part is needed whose common-mode range includes ground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"
- note added: "VR_BIAS -- mid-rail reference for the floating VR coil"
- note added: "WHY THE CAM FRONT-END ON THIS SHEET IS NOT THE ONE THE SPEC ASKS FOR. Spec sec.4 and docs/pinmap.md sec.1.3 both give pin 46's front end as "Pull-up to 5V_SENSOR -> timer capture": the Hall output pulled to 5 V and taken straight into PTB3. NXP S32K1xx Data Sheet Rev. 15, Table 17, puts Vih max at VDD + 0.3 V, about 3.6 V at VDD = 3.3 V, so a full 5 V swing is not a guaranteed valid logic level. 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"
