File: prototype/can.kicad_sch (KiCad schematic)
At the start: 18 parts, among them U901 TCAN1042HGV, U902 TCAN1042HGV

Commit message: Prototype: board placed, critical loops packed as clusters, placement DRC clean
Parts:
- TP21, TP22, TP23, TP24: now left out of the parts list
Changed lines of the file:
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@@
   )
   (symbol (lib_id "Connector:TestPoint") (at 271.78 30.48 0) (unit 1)
-    (in_bom yes) (on_board yes) (fields_autoplaced)
+    (in_bom no) (on_board yes) (fields_autoplaced)
     (property "Reference" "TP21" (id 0) (at 271.78000000000003 25.4 0)
       (effects (font (size 1.27 1.27)))
@@
   )
   (symbol (lib_id "Connector:TestPoint") (at 271.78 45.72 0) (unit 1)
-    (in_bom yes) (on_board yes) (fields_autoplaced)
+    (in_bom no) (on_board yes) (fields_autoplaced)
     (property "Reference" "TP22" (id 0) (at 271.78000000000003 40.64 0)
       (effects (font (size 1.27 1.27)))
@@
   )
   (symbol (lib_id "Connector:TestPoint") (at 271.78 60.96 0) (unit 1)
-    (in_bom yes) (on_board yes) (fields_autoplaced)
+    (in_bom no) (on_board yes) (fields_autoplaced)
     (property "Reference" "TP23" (id 0) (at 271.78000000000003 55.88 0)
       (effects (font (size 1.27 1.27)))
@@
   )
   (symbol (lib_id "Connector:TestPoint") (at 271.78 76.2 0) (unit 1)
-    (in_bom yes) (on_board yes) (fields_autoplaced)
+    (in_bom no) (on_board yes) (fields_autoplaced)
     (property "Reference" "TP24" (id 0) (at 271.78000000000003 71.12 0)
       (effects (font (size 1.27 1.27)))
