File: prototype/injector.kicad_sch (KiCad schematic)
At the start: 107 parts, among them Q401 DMN15H310SK3, Q402 2N7002BK, Q403 2N7002BK, Q404 2N7002BK, Q405 2N7002BK, Q406 PZTA42-Q, Q407 PMBT3904-Q, Q408 SQM85N15-19, Q409 IPD90N10S4-06, Q410 SQM85N15-19, Q411 IPD90N10S4-06, Q412 SQM85N15-19, Q413 2N7002BK, Q414 SQM85N15-19, Q415 2N7002BK, Q416 SQM85N15-19, Q417 2N7002BK, Q418 PZTA42-Q, Q419 PMBT3904-Q, U401 TPS40210, U402 AUIRS2181S, U403 AUIRS2181S, U404 AUIRS2181S, U405 AUIRS2181S, U406 INA181A1, U407 INA181A1

Commit message: Prototype: board placed, critical loops packed as clusters, placement DRC clean
Parts:
- TP15, TP16: now left out of the parts list
Changed lines of the file:
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@@
   )
   (symbol (lib_id "Connector:TestPoint") (at 850.9 76.2 0) (unit 1)
-    (in_bom yes) (on_board yes) (fields_autoplaced)
+    (in_bom no) (on_board yes) (fields_autoplaced)
     (property "Reference" "TP15" (id 0) (at 850.9 71.12 0)
       (effects (font (size 1.27 1.27)))
@@
   )
   (symbol (lib_id "Connector:TestPoint") (at 850.9 91.44 0) (unit 1)
-    (in_bom yes) (on_board yes) (fields_autoplaced)
+    (in_bom no) (on_board yes) (fields_autoplaced)
     (property "Reference" "TP16" (id 0) (at 850.9 86.36 0)
       (effects (font (size 1.27 1.27)))
