File: prototype/metering_egr.kicad_sch (KiCad schematic)
At the start: 33 parts, among them Q501 IPD90N10S4-06, Q502 2N7002BK, Q503 IPD90N10S4-06, Q504 IPD90N10S4-06, Q505 IPD90N10S4-06, Q506 IPD90N10S4-06, Q507 2N7002BK, U501 INA181A1, U502 AUIRS2181S, U503 INA181A1, U504 AUIRS2184S, U505 AUIRS2184S

Commit message: Prototype: board placed, critical loops packed as clusters, placement DRC clean
Parts:
- TP17, TP18: now left out of the parts list
Changed lines of the file:
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@@
   )
   (symbol (lib_id "Connector:TestPoint") (at 591.82 30.48 0) (unit 1)
-    (in_bom yes) (on_board yes) (fields_autoplaced)
+    (in_bom no) (on_board yes) (fields_autoplaced)
     (property "Reference" "TP17" (id 0) (at 591.82 25.4 0)
       (effects (font (size 1.27 1.27)))
@@
   )
   (symbol (lib_id "Connector:TestPoint") (at 591.82 45.72 0) (unit 1)
-    (in_bom yes) (on_board yes) (fields_autoplaced)
+    (in_bom no) (on_board yes) (fields_autoplaced)
     (property "Reference" "TP18" (id 0) (at 591.82 40.64 0)
       (effects (font (size 1.27 1.27)))
