File: prototype/speed_inputs.kicad_sch (KiCad schematic)
At the start: 22 parts, among them U701 TLV3201

Commit message: Prototype: board placed, critical loops packed as clusters, placement DRC clean
Parts:
- TP19, TP20: now left out of the parts list
Changed lines of the file:
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@@
   )
   (symbol (lib_id "Connector:TestPoint") (at 370.84 30.48 0) (unit 1)
-    (in_bom yes) (on_board yes) (fields_autoplaced)
+    (in_bom no) (on_board yes) (fields_autoplaced)
     (property "Reference" "TP19" (id 0) (at 370.84000000000003 25.4 0)
       (effects (font (size 1.27 1.27)))
@@
   )
   (symbol (lib_id "Connector:TestPoint") (at 370.84 45.72 0) (unit 1)
-    (in_bom yes) (on_board yes) (fields_autoplaced)
+    (in_bom no) (on_board yes) (fields_autoplaced)
     (property "Reference" "TP20" (id 0) (at 370.84000000000003 40.64 0)
       (effects (font (size 1.27 1.27)))
