File: prototype/prototype.kicad_pcb (KiCad board)
At the start: 4 copper layers, 220 x 160 mm, 433 parts, among them J1001 J1001, J1002 J1002, J1003 J1003, J1004 J1004, J1005 J1005, J1006 J1006, J1007 J1007, J1008 J1008, J1009 J1009, J301 SWD/JTAG, J302 USB-C, Q101 SQD50P08-25L, Q102 IPD90N10S4-06, Q103 SQM120P10-10m1L, Q104 SQM120P10-10m1L, Q201 IPD90N10S4-06, Q301 2N7002BK, Q401 DMN15H310SK3, Q402 2N7002BK, Q403 2N7002BK, Q404 2N7002BK, Q405 2N7002BK, Q406 PZTA42-Q, Q407 PMBT3904-Q, Q408 SQM85N15-19, Q409 IPD90N10S4-06, Q410 SQM85N15-19, Q411 IPD90N10S4-06, Q412 SQM85N15-19, Q413 2N7002BK, Q414 SQM85N15-19, Q415 2N7002BK, Q416 SQM85N15-19, Q417 2N7002BK, Q418 PZTA42-Q, Q419 PMBT3904-Q, Q501 IPD90N10S4-06, Q502 2N7002BK, Q503 IPD90N10S4-06, Q504 IPD90N10S4-06, Q505 IPD90N10S4-06, Q506 IPD90N10S4-06, Q507 2N7002BK, Q801 PMBT3904-Q, Q802 PMBT3904-Q, Q803 PMBT3904-Q, Q804 PMBT3904-Q, Q805 PMBT3904-Q, Q806 PMV280ENEA, Q807 PMV280ENEA, U101 TLV3201, U102 UCC27517A, U201 LM5164, U202 TLV76733, U203 TPS48110, U204 TPS7B4253, U205 TPS7B4253, U206 TPS7B4253, U301 STM32G474VETx, U302 TPS3850G33, U303 USBLC6-2SC6, U401 TPS40210, U402 AUIRS2181S, U403 AUIRS2181S, U404 AUIRS2181S, U405 AUIRS2181S, U406 INA181A1, U407 INA181A1, U501 INA181A1, U502 AUIRS2181S, U503 INA181A1, U504 AUIRS2184S, U505 AUIRS2184S, U601 INA592, U602 INA592, U603 INA592, U604 INA592, U605 INA592, U606 MPXHZ6115A, U701 TLV3201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

Commit message: Prototype: power pours as fixed copper, ground fanout to L2, three-layer router input (routing not complete)
Pours reach Freerouting as fixed wires, their vias fixed; L2 and ground
leave the router's view, every SMD ground pad has its own via to the
plane. Pour bars union per net and layer, via pads at layer hops sized
for the current, vias only where they join two layers and clear every
other net. Placement groups small parts with the part they serve.
Pin necks of 0.15 mm allowed inside courtyards (owner, 16 Oct).
Run 9: 27 connections open, 12 clearance errors; work continues.
Parts:
- moved D806 169.0 mm to (300.5, 163.5), turned to 90 degrees
- moved Q402 161.6 mm to (192.2, 121.7)
- moved R807 160.6 mm to (295.5, 165.0), turned to 180 degrees
- moved R809 160.6 mm to (291.3, 167.3)
- moved C220 156.9 mm to (299.3, 24.0)
- moved Q803 156.3 mm to (296.2, 161.7), turned to 180 degrees
- moved R410 155.9 mm to (191.7, 124.8), turned to 180 degrees
- moved R804 155.8 mm to (286.6, 165.0), turned to 180 degrees
- moved Q403 155.7 mm to (192.2, 127.8)
- moved Q802 151.9 mm to (287.3, 161.7), turned to 180 degrees
- moved R411 150.7 mm to (191.7, 130.8), turned to 180 degrees
- moved Q404 149.9 mm to (192.2, 133.8)
- moved Q801 147.6 mm to (278.4, 161.7), turned to 180 degrees
- moved U802 146.2 mm to (300.8, 169.3)
- moved R412 145.7 mm to (191.7, 136.8), turned to 180 degrees
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Routing:
- net GND: track 0.00 -> 2328.5 mm, vias 0 -> 379
- net /3V3_MCU: track 0.00 -> 771.7 mm, vias 0 -> 27
- net /5V_MAIN: track 0.00 -> 673.4 mm, vias 0 -> 18
- net /12V_GATE: track 0.00 -> 452.4 mm, vias 0 -> 8
- net /VBAT_PROT: track 0.00 -> 385.4 mm, vias 0 -> 75
- net /GATE_KILL: track 0.00 -> 364.9 mm, vias 0 -> 12
- net /V_BAT_1R: track 0.00 -> 237.9 mm, vias 0 -> 7
- net /RLY_BUZZER_OUT: track 0.00 -> 224.5 mm, vias 0 -> 1
- net /V_BAT_2R: track 0.00 -> 216.1 mm, vias 0 -> 13
- net /RLY_MAIN_OUT: track 0.00 -> 213.4 mm, vias 0 -> 1
- net /INJ_LS_3: track 0.00 -> 211.5 mm, vias 0 -> 13
- net /INJ_LS_2: track 0.00 -> 209.3 mm, vias 0 -> 4
- net /injector/UA2_HIN: track 0.00 -> 192.4 mm, vias 0 -> 3
- net /injector/UB1_HIN: track 0.00 -> 189.1 mm, vias 0 -> 3
- net /injector/UB2_HIN: track 0.00 -> 184.3 mm, vias 0 -> 2
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- added copper zone on B.Cu, net /EGR_HIGH_59
- added copper zone on F.Cu, net /EGR_HIGH_59
- added copper zone on B.Cu, net /EGR_LOW_81
- added copper zone on F.Cu, net /EGR_LOW_81
- added copper zone on B.Cu, net /INJ_A_03
- added copper zone on F.Cu, net /INJ_A_03
- added copper zone on In2.Cu, net /INJ_A_03
- added copper zone on B.Cu, net /INJ_B_05
- added copper zone on F.Cu, net /INJ_B_05
- added copper zone on In2.Cu, net /INJ_B_05
- added copper zone on F.Cu, net /INJ_LS1_73
- added copper zone on B.Cu, net /INJ_LS2_29
- added copper zone on F.Cu, net /INJ_LS2_29
- added copper zone on F.Cu, net /INJ_LS3_07
- added copper zone on F.Cu, net /MU_RETURN
- added copper zone on In2.Cu, net /MU_RETURN
- added copper zone on B.Cu, net /VBAT_EGR
- added copper zone on F.Cu, net /VBAT_EGR
- added copper zone on B.Cu, net /VBAT_IN
- added copper zone on F.Cu, net /VBAT_IN
- added copper zone on In2.Cu, net /VBAT_IN
- added copper zone on B.Cu, net /VBAT_INJ
- added copper zone on F.Cu, net /VBAT_INJ
- added copper zone on B.Cu, net /VBAT_PROT
- added copper zone on F.Cu, net /VBAT_PROT
- added copper zone on In2.Cu, net /VBAT_PROT
- added copper zone on F.Cu, net /V_BAT_1R
- added copper zone on B.Cu, net /V_BAT_2R
- added copper zone on F.Cu, net /V_BAT_2R
- added copper zone on B.Cu, net /injector/BOOST_100V
- added copper zone on F.Cu, net /injector/BOOST_100V
- added copper zone on F.Cu, net /injector/ISNS_BOOST
- added copper zone on B.Cu, net /injector/ISNS_INJ_A_SENSE
- added copper zone on F.Cu, net /injector/ISNS_INJ_A_SENSE
- added copper zone on In2.Cu, net /injector/ISNS_INJ_A_SENSE
- added copper zone on F.Cu, net /injector/ISNS_INJ_B_SENSE
- added copper zone on In2.Cu, net /injector/ISNS_INJ_B_SENSE
- added copper zone on F.Cu, net /injector/SW_BOOST
- added copper zone on F.Cu, net /metering_egr/EGR_ISNS
- added copper zone on In2.Cu, net /metering_egr/EGR_ISNS
- added copper zone on F.Cu, net /metering_egr/ISNS_MU_SENSE
- added copper zone on B.Cu, net /power_input/VBAT_CLAMPED
- added copper zone on F.Cu, net /power_input/VBAT_CLAMPED
- added copper zone on B.Cu, net /power_input/VBAT_EGR_IN
- added copper zone on F.Cu, net /power_input/VBAT_EGR_IN
- added copper zone on In2.Cu, net /power_input/VBAT_EGR_IN
- added copper zone on F.Cu, net /power_input/VBAT_EMI1
- added copper zone on B.Cu, net /power_input/VBAT_INJ_IN
- added copper zone on F.Cu, net /power_input/VBAT_INJ_IN
- added copper zone on In2.Cu, net /power_input/VBAT_INJ_IN
- added copper zone on B.Cu, net /rails/VSNS
- added copper zone on F.Cu, net /rails/VSNS
- added copper zone on B.Cu, net GND
- added copper zone on F.Cu, net GND
- added copper zone on In1.Cu, net GND
- added copper zone on B.Cu, net Net-(D408-K)
- added copper zone on F.Cu, net Net-(D408-K)
- added copper zone on In2.Cu, net Net-(D408-K)
- added copper zone on B.Cu, net Net-(D410-K)
- added copper zone on B.Cu, net Net-(F101-Pad2)
- added copper zone on F.Cu, net Net-(F101-Pad2)
- added copper zone on In2.Cu, net Net-(F101-Pad2)
Other:
- board size 220 x 160 mm -> 300 x 200 mm
