File: prototype/prototype.kicad_pcb (KiCad board)
At the start: 4 copper layers, 300 x 200 mm, 433 parts, among them J1001 J1001, J1002 J1002, J1003 J1003, J1004 J1004, J1005 J1005, J1006 J1006, J1007 J1007, J1008 J1008, J1009 J1009, J301 SWD/JTAG, J302 USB-C, Q101 SQD50P08-25L, Q102 IPD90N10S4-06, Q103 SQM120P10-10m1L, Q104 SQM120P10-10m1L, Q201 IPD90N10S4-06, Q301 2N7002BK, Q401 DMN15H310SK3, Q402 2N7002BK, Q403 2N7002BK, Q404 2N7002BK, Q405 2N7002BK, Q406 PZTA42-Q, Q407 PMBT3904-Q, Q408 SQM85N15-19, Q409 IPD90N10S4-06, Q410 SQM85N15-19, Q411 IPD90N10S4-06, Q412 SQM85N15-19, Q413 2N7002BK, Q414 SQM85N15-19, Q415 2N7002BK, Q416 SQM85N15-19, Q417 2N7002BK, Q418 PZTA42-Q, Q419 PMBT3904-Q, Q501 IPD90N10S4-06, Q502 2N7002BK, Q503 IPD90N10S4-06, Q504 IPD90N10S4-06, Q505 IPD90N10S4-06, Q506 IPD90N10S4-06, Q507 2N7002BK, Q801 PMBT3904-Q, Q802 PMBT3904-Q, Q803 PMBT3904-Q, Q804 PMBT3904-Q, Q805 PMBT3904-Q, Q806 PMV280ENEA, Q807 PMV280ENEA, U101 TLV3201, U102 UCC27517A, U201 LM5164, U202 TLV76733, U203 TPS48110, U204 TPS7B4253, U205 TPS7B4253, U206 TPS7B4253, U301 STM32G474VETx, U302 TPS3850G33, U303 USBLC6-2SC6, U401 TPS40210, U402 AUIRS2181S, U403 AUIRS2181S, U404 AUIRS2181S, U405 AUIRS2181S, U406 INA181A1, U407 INA181A1, U501 INA181A1, U502 AUIRS2181S, U503 INA181A1, U504 AUIRS2184S, U505 AUIRS2184S, U601 INA592, U602 INA592, U603 INA592, U604 INA592, U605 INA592, U606 MPXHZ6115A, U701 TLV3201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

Commit message: Prototype: board routed, DRC and parity clean
All 625 connections routed: 0 unconnected, 0 DRC errors, parity clean but
for D806's known placeholder footprint.

- Freerouting (run 12) leaves 45 open; finish_router.py, KiCad's DRC the
  arbiter, routes the rest: pin necks of 0.15 mm inside a courtyard, a
  start anywhere on an end's copper island, vias through a pour's
  interior and dear (necks()-judged) bites into its edge, a 50 mm pass
  on a 0.1 mm grid, then rip-up round the ends and along the line
  between them; tidy removes dangling and doubled copper.
- Placement keeps 1 mm round fine-pitch chips and turns R503 180 degrees
  (EGR_AH_G and EGR_HIGH_59 had to cross at 0.6 mm clearance).
- A pour cut by a passing track is repaired in finish().
- Pin escape rule: inside a fine-pitch chip's courtyard a PWR/PWR_LOOM
  track keeps the chip's own 0.2 mm pin gap to its pads (U203 pin 13
  could not be reached at 0.3 mm); the 100 V classes and PWR_HI keep
  theirs.
- widen() reverts a clearance breaker for good, so it converges.
Parts:
- moved U202 33.9 mm to (299.6, 23.8)
- moved C207 32.6 mm to (298.2, 28.1)
- moved C317 32.1 mm to (243.7, 129.8)
- moved U206 31.7 mm to (270.0, 42.3)
- moved C220 31.7 mm to (270.0, 36.0)
- moved R209 29.7 mm to (235.5, 37.3), turned to 180 degrees
- moved J301 27.5 mm to (244.3, 106.2), turned to 0 degrees
- moved TP10 26.4 mm to (298.1, 31.3)
- moved R307 26.1 mm to (208.6, 128.2), turned to 0 degrees
- moved C212 25.5 mm to (239.0, 37.3), turned to 0 degrees
- moved R211 24.3 mm to (235.5, 39.4), turned to 0 degrees
- moved R212 24.3 mm to (239.0, 39.4)
- moved C208 23.0 mm to (243.0, 35.2), turned to 90 degrees
- moved C218 23.0 mm to (243.0, 31.7), turned to -90 degrees
- moved C316 22.5 mm to (201.5, 128.2)
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Routing:
- net /injector/BOOST_100V: track 128.0 -> 190.7 mm, vias 53 -> 57
- net /3V3_MCU: track 771.7 -> 829.2 mm, vias 27 -> 33
- net /injector/HSA_BAT_GATE: track 149.0 -> 204.6 mm, vias 3 -> 10
- net /INJ_A_03: track 45.4 -> 98.5 mm, vias 30 -> 33
- net GND: track 2328.5 -> 2280.8 mm, vias 379 -> 375
- net /SENSOR_5V_MON: track 120.8 -> 166.4 mm, vias 4 -> 3
- net /5V_MAIN: track 673.4 -> 627.9 mm, vias 18 -> 16
- net /mcu_stm32/BOOT0: track 66.8 -> 21.7 mm, vias 3 -> 2
- net /rails/OVC_GATE: track 22.8 -> 61.0 mm, vias 3 -> 5
- net /INJ_LS_2: track 209.3 -> 247.1 mm, vias 4 -> 7
- net /mcu_stm32/USB_CC2: track 51.9 -> 14.2 mm, vias 5 -> 3
- net /INJ_LS_3: track 211.5 -> 248.1 mm, vias 13 -> 4
- net /VBAT_INJ: track 98.9 -> 134.7 mm, vias 75 -> 76
- net /mcu_stm32/USB_CC1: track 50.4 -> 14.8 mm, vias 3 -> 2
- net /injector/RC_BOOST: track 0.00 -> 33.6 mm, vias 0 -> 4
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