File: prototype/prototype.kicad_pcb (KiCad board)
At the start: 4 copper layers, 300 x 200 mm, 433 parts, among them J1001 J1001, J1002 J1002, J1003 J1003, J1004 J1004, J1005 J1005, J1006 J1006, J1007 J1007, J1008 J1008, J1009 J1009, J301 SWD/JTAG, J302 USB-C, Q101 SQD50P08-25L, Q102 IPD90N10S4-06, Q103 SQM120P10-10m1L, Q104 SQM120P10-10m1L, Q201 IPD90N10S4-06, Q301 2N7002BK, Q401 DMN15H310SK3, Q402 2N7002BK, Q403 2N7002BK, Q404 2N7002BK, Q405 2N7002BK, Q406 PZTA42-Q, Q407 PMBT3904-Q, Q408 SQM85N15-19, Q409 IPD90N10S4-06, Q410 SQM85N15-19, Q411 IPD90N10S4-06, Q412 SQM85N15-19, Q413 2N7002BK, Q414 SQM85N15-19, Q415 2N7002BK, Q416 SQM85N15-19, Q417 2N7002BK, Q418 PZTA42-Q, Q419 PMBT3904-Q, Q501 IPD90N10S4-06, Q502 2N7002BK, Q503 IPD90N10S4-06, Q504 IPD90N10S4-06, Q505 IPD90N10S4-06, Q506 IPD90N10S4-06, Q507 2N7002BK, Q801 PMBT3904-Q, Q802 PMBT3904-Q, Q803 PMBT3904-Q, Q804 PMBT3904-Q, Q805 PMBT3904-Q, Q806 PMV280ENEA, Q807 PMV280ENEA, U101 TLV3201, U102 UCC27517A, U201 LM5164, U202 TLV76733, U203 TPS48110, U204 TPS7B4253, U205 TPS7B4253, U206 TPS7B4253, U301 STM32G474VETx, U302 TPS3850G33, U303 USBLC6-2SC6, U401 TPS40210, U402 AUIRS2181S, U403 AUIRS2181S, U404 AUIRS2181S, U405 AUIRS2181S, U406 INA181A1, U407 INA181A1, U501 INA181A1, U502 AUIRS2181S, U503 INA181A1, U504 AUIRS2184S, U505 AUIRS2184S, U601 INA592, U602 INA592, U603 INA592, U604 INA592, U605 INA592, U606 MPXHZ6115A, U701 TLV3201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

Commit message: Prototype review fixes: watchdog kill restored, pour checks that can fail
- D302 (BAT54Q-7-F, anode ~RESET, cathode WDT_FAULT) restores the
  watchdog-to-gate-kill path the 15 Oct supervisor fix removed; production
  and prototype. check_netlist WDO_KILL guards it. WDT_FAULT no longer
  records which trip it was; docs corrected.
- gen_board: sync stage (rename shifted refs, place new parts on a routed
  board), clusters stage, rip_thin, per-net IPC targets in widen, outer-only
  routing for nets In2 cannot carry, finish undoes a pass that necks a pour.
- Tests: pour connectivity read from pcbnew (the DRC list stops at ~500),
  test_no_necks, test_track_power_widths (TRACK_AMPS), test_inputs_committed.
- The 5 V buck's output and switch node now run on the outer layers.
- check_pcb: a parity entry with no items no longer crashes it.
- bring-up guide: probe rating, charged boost caps, 5 A limit, kill FETs.
- Decisions §15, status, handoff traps; fab files and PDF rebuilt.
Parts:
- added D302: BAT54Q-7-F, ecu25kva:SOT-23_Zener_K1_A2, F.Cu at (218.4, 131.3)
- renumbered D302 to D303, D303 to D304
Routing:
- net /mcu_stm32/WDT_FAULT: track 31.7 -> 52.6 mm, vias 3 -> 7
- net /mcu_stm32/~{RESET}: track 68.0 -> 81.0 mm, vias 5 -> 9
- net /rails/SW: track 29.0 -> 33.6 mm, vias 2 -> 0
- net /5V_MAIN: track 627.9 -> 626.4 mm, vias 16 -> 30
